File: KiCAD/Quest_39/Quest_39_blz2.kicad_sch (KiCad schematic)
At the start: 13 parts

Commit message: Edited schematic
Parts:
- removed C?: Cp, symbol Device:C
- added C?: 1uF, symbol Device:C
- added C?: 330uF, symbol Device:C_Polarized
- added R? (x2): 10, symbol Device:R
- added R?: 0R0025, symbol Device:R
- added U?: INA226, Package_SO:VSSOP-10_3x3mm_P0.5mm, symbol Analog_ADC:INA226
- added U?: MCP601T-I/OT, Package_TO_SOT_SMD:SOT-23-5, symbol Amplifier_Operational:MCP601-xOT
- C?: value Cff -> 100pF
Connections:
- net +5V: now also U?.5 (V+), U?.6 (VS)
- net GND: now also C?.2, U?.1 (A1), U?.2 (A0), U?.2 (V-), U?.3 (~{Alert})
- net GND_0: now also U?.1, U?.4 (-), U?.8 (Vbus)
- net RUN: no longer R?.2, U?.A10 (RUN)
- net VIN_0: now also R?.1, R?.1; no longer C?.1, C?.1, C?.1, R?.1, U?.A1 (VIN), U?.A2 (VIN), U?.A3 (VIN), U?.A4 (VIN), U?.A5 (VIN), U?.A6 (VIN), U?.B1 (VIN), U?.B2 (VIN), U?.B3 (VIN), U?.B4 (VIN), U?.B5 (VIN), U?.B6 (VIN), U?.C1 (VIN), U?.C2 (VIN), U?.C3 (VIN), U?.C4 (VIN), U?.C5 (VIN), U?.C6 (VIN)
- new net: C?.2, R?.2, U?.9 (Vin-)
- new net: C?.1, C?.1, C?.1, C?.1, R?.1, R?.1, R?.2, U?.3 (+), U?.A1 (VIN), U?.A2 (VIN), U?.A3 (VIN), U?.A4 (VIN), U?.A5 (VIN), U?.A6 (VIN), U?.B1 (VIN), U?.B2 (VIN), U?.B3 (VIN), U?.B4 (VIN), U?.B5 (VIN), U?.B6 (VIN), U?.C1 (VIN), U?.C2 (VIN), U?.C3 (VIN), U?.C4 (VIN), U?.C5 (VIN), U?.C6 (VIN)
- new net: R?.2, U?.A10 (RUN)
- new net SCL: U?.5 (SCL)
- new net SDA: U?.4 (SDA)
- new net Vin+_0: C?.1, R?.2, U?.10 (Vin+)
Other:
- note added: "Power Measurement"
- moved on the sheet: C?, R?

Commit message: GND van INA226 verbonden, remote sense amplifier in gebruik genomen, labels aangepast en INTVCC not connected gemaakt.
Parts:
- removed C?: 47uF, symbol Device:C
- added C? (x3): 100uF, symbol Device:C_Polarized
- C?: footprint (none) -> OptoDevice:R_LDR_4.9x4.2mm_P2.54mm_Vertical
- C?: value 220uF -> 100uF
Connections:
- net GND: now also U?.7 (GND); no longer C?.2, C?.2, C?.2, C?.2
- net GND_0: now also C?.2, C?.2, C?.2, C?.2, U?.M12 (VOSNS-), C?.2, C?.2, C?.2; no longer U?.J12 (VOSNS+)
- net VOUT_0: now also U?.J12 (VOSNS+), C?.1, C?.1, C?.1; no longer U?.L12 (VOUT_LCL)
- net at U?.K12 (DIFFVOUT): now also U?.L12 (VOUT_LCL)
- removed net INTVCC_0: U?.A7 (INTVCC), U?.D9 (INTVCC), U?.M12 (VOSNS-)
- no-connect marks 15 -> 16
Other:
- moved on the sheet: C?
