File: KiCAD/Quest_39/Quest_39.kicad_sch (KiCad schematic)
At the start: 26 parts

Commit message: Exchanged MCP601 for AD626
Parts:
- added J?: Conn_01x04_Male, symbol Connector:Conn_01x04_Male
Connections:
- net GND: now also J?.1 (Pin_1)
- net SWCLK: now also J?.2 (Pin_2)
- net SWDIO: now also J?.3 (Pin_3)
- new net +3V3: J?.4 (Pin_4)
Changed lines of the file:
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@@
     (stroke (width 0) (type default) (color 0 0 0 0))
   )
-  (wire (pts (xy 181.61 109.22) (xy 195.58 109.22))
+  (wire (pts (xy 181.61 109.22) (xy 204.47 109.22))
     (stroke (width 0) (type default) (color 0 0 0 0))
   )
@@
     (stroke (width 0) (type default) (color 0 0 0 0))
   )
+  (wire (pts (xy 203.2 115.57) (xy 203.2 114.3))
+    (stroke (width 0) (type default) (color 0 0 0 0))
+  )
   (wire (pts (xy 54.61 132.08) (xy 58.42 132.08))
     (stroke (width 0) (type default) (color 0 0 0 0))
@@
     (stroke (width 0) (type default) (color 0 0 0 0))
   )
+  (wire (pts (xy 203.2 114.3) (xy 204.47 114.3))
+    (stroke (width 0) (type default) (color 0 0 0 0))
+  )
   (wire (pts (xy 30.48 113.03) (xy 34.29 113.03))
     (stroke (width 0) (type default) (color 0 0 0 0))
@@
     (stroke (width 0) (type default) (color 0 0 0 0))
   )
+  (wire (pts (xy 203.2 105.41) (xy 203.2 106.68))
+    (stroke (width 0) (type default) (color 0 0 0 0))
+  )
   (wire (pts (xy 30.48 78.74) (xy 34.29 78.74))
     (stroke (width 0) (type default) (color 0 0 0 0))
@@
     (stroke (width 0) (type default) (color 0 0 0 0))
   )
+  (wire (pts (xy 203.2 106.68) (xy 204.47 106.68))
+    (stroke (width 0) (type default) (color 0 0 0 0))
+  )
   (wire (pts (xy 35.56 27.94) (xy 35.56 57.15))
     (stroke (width 0) (type default) (color 0 0 0 0))
@@
     (stroke (width 0) (type default) (color 0 0 0 0))
   )
-  (wire (pts (xy 181.61 111.76) (xy 195.58 111.76))
+  (wire (pts (xy 181.61 111.76) (xy 204.47 111.76))
     (stroke (width 0) (type default) (color 0 0 0 0))
   )
@@
     (pin "1")
     (pin "2")
+  )
+  (symbol (lib_id "power:GND") (at 203.2 115.57 0) (unit 1)
+    (in_bom yes) (on_board yes) (fields_autoplaced)
+    (property "Reference" "#PWR?" (id 0) (at 203.2 121.92 0)
+      (effects (font (size 1.27 1.27)) hide)
+    )
+    (property "Value" "GND" (id 1) (at 203.2 120.65 0))
+    (property "Footprint" "" (id 2) (at 203.2 115.57 0)
+      (effects (font (size 1.27 1.27)) hide)
+    )
+    (property "Datasheet" "" (id 3) (at 203.2 115.57 0)
+      (effects (font (size 1.27 1.27)) hide)
+    )
+    (pin "1")
   )
   (symbol (lib_id "Connector:Screw_Terminal_01x02") (at 246.38 113.03 0) (unit 1)
@@
     (pin "2")
   )
+  (symbol (lib_id "Connector:Conn_01x04_Male") (at 209.55 111.76 180) (unit 1)
+    (in_bom yes) (on_board yes) (fields_autoplaced)
+    (property "Reference" "J?" (id 0) (at 210.82 109.2199 0)
+      (effects (font (size 1.27 1.27)) (justify right))
+    )
+    (property "Value" "Conn_01x04_Male" (id 1) (at 210.82 111.7599 0)
+      (effects (font (size 1.27 1.27)) (justify right))
+    )
+    (property "Footprint" "" (id 2) (at 209.55 111.76 0)
+      (effects (font (size 1.27 1.27)) hide)
+    )
+    (property "Datasheet" "~" (id 3) (at 209.55 111.76 0)
+      (effects (font (size 1.27 1.27)) hide)
+    )
+    (pin "1")
+    (pin "2")
+    (pin "3")
+    (pin "4")
+  )
   (symbol (lib_id "Device:C") (at 147.32 33.02 0) (unit 1)
     (in_bom yes) (on_board yes) (fields_autoplaced)
@@
     (pin "1")
     (pin "2")
+  )
+  (symbol (lib_id "power:+3V3") (at 203.2 105.41 0) (unit 1)
+    (in_bom yes) (on_board yes) (fields_autoplaced)
+    (property "Reference" "#PWR?" (id 0) (at 203.2 109.22 0)
+      (effects (font (size 1.27 1.27)) hide)
+    )
+    (property "Value" "+3V3" (id 1) (at 203.2 100.33 0))
+    (property "Footprint" "" (id 2) (at 203.2 105.41 0)
+      (effects (font (size 1.27 1.27)) hide)
+    )
+    (property "Datasheet" "" (id 3) (at 203.2 105.41 0)
+      (effects (font (size 1.27 1.27)) hide)
+    )
+    (pin "1")
   )
   (symbol (lib_id "Connector:Screw_Terminal_01x02") (at 246.38 82.55 0) (unit 1)
@@
       (reference "#PWR0110") (unit 1) (value "+5V") (footprint "")
     )
-    (path "/8781658c-e5d4-40cc-b0c0-8e95668fb10a/3853d6ba-3ba6-4a80-b248-7b9a71036578"
-      (reference "#PWR0111") (unit 1) (value "+5V") (footprint "")
-    )
-    (path "/8781658c-e5d4-40cc-b0c0-8e95668fb10a/061be5ab-70b7-4ccd-bfd0-b4aa1dee769a"
-      (reference "#PWR0112") (unit 1) (value "GND") (footprint "")
-    )
     (path "/8781658c-e5d4-40cc-b0c0-8e95668fb10a/16f5566b-2033-4cfe-846e-2858efa0d672"
       (reference "#PWR0113") (unit 1) (value "GND") (footprint "")
@@
       (reference "#PWR0179") (unit 1) (value "GND") (footprint "")
     )
+    (path "/8781658c-e5d4-40cc-b0c0-8e95668fb10a/0fde256f-1cf6-4c4c-ba96-b180a83da87a"
+      (reference "#PWR?") (unit 1) (value "GND") (footprint "")
+    )
+    (path "/8781658c-e5d4-40cc-b0c0-8e95668fb10a/54ffa172-1c01-42a1-898a-8972961a1367"
+      (reference "#PWR?") (unit 1) (value "+5V") (footprint "")
+    )
+    (path "/68de5b5c-67ca-40a7-a9c8-801c31bf82ae"
+      (reference "#PWR?") (unit 1) (value "GND") (footprint "")
+    )
+    (path "/8781658c-e5d4-40cc-b0c0-8e95668fb10a/d46b6a1e-2b94-4869-a301-6e02a8642c83"
+      (reference "#PWR?") (unit 1) (value "GND") (footprint "")
+    )
+    (path "/db4c33a8-7a24-4d42-8408-d14930b2b63e"
+      (reference "#PWR?") (unit 1) (value "+3V3") (footprint "")
+    )
+    (path "/8781658c-e5d4-40cc-b0c0-8e95668fb10a/e7099699-d321-4638-abf7-88b93d3f2517"
+      (reference "#PWR?") (unit 1) (value "GND") (footprint "")
+    )
+    (path "/8781658c-e5d4-40cc-b0c0-8e95668fb10a/02caa000-8c59-455e-8e2d-977dd6843e72"
+      (reference "C?") (unit 1) (value "100nF") (footprint "")
+    )
     (path "/b44f6773-e3e8-4e75-9d5c-4dbba7b405cd/035487e2-abe6-4efe-bda0-9e9c984c89ef"
       (reference "C?") (unit 1) (value "22uF") (footprint "")
@@
       (reference "C?") (unit 1) (value "100pF") (footprint "")
     )
+    (path "/8781658c-e5d4-40cc-b0c0-8e95668fb10a/ac0f456a-203c-419f-8cbc-87dedbfc1186"
+      (reference "C?") (unit 1) (value "100nF") (footprint "")
+    )
     (path "/a3821039-2367-4234-b9fc-572f119c5510/ae6741b8-092c-4e64-ba5b-fa8fb8a5b9ab"
       (reference "C?") (unit 1) (value "100uF") (footprint "")
@@
       (reference "C?") (unit 1) (value "330uF") (footprint "")
     )
+    (path "/8781658c-e5d4-40cc-b0c0-8e95668fb10a/bec97cc5-654c-4a5a-ac25-93f43616c62f"
+      (reference "C?") (unit 1) (value "100nF") (footprint "")
+    )
     (path "/84d8ca1d-7213-486c-b202-d20639515304/c55fc249-dd75-4cb9-aa1f-2087cc0b6101"
       (reference "C?") (unit 1) (value "100nF") (footprint "")
@@
       (reference "J?") (unit 1) (value "1x2 Scr. Term.") (footprint "")
     )
+    (path "/a6b0ecbe-69ca-4355-83c8-0390dd315ab8"
+      (reference "J?") (unit 1) (value "Conn_01x04_Male") (footprint "")
+    )
     (path "/b7ec1e0a-09b8-4a1b-a8d2-7b406e266333"
       (reference "J?") (unit 1) (value "1x2 Scr. Term") (footprint "")
@@
       (reference "R?") (unit 1) (value "10") (footprint "")
     )
+    (path "/8781658c-e5d4-40cc-b0c0-8e95668fb10a/1d6403f0-2fa4-4eb2-bc43-fd19969d3b3b"
+      (reference "R?") (unit 1) (value "9K") (footprint "")
+    )
     (path "/a3821039-2367-4234-b9fc-572f119c5510/281441c8-59bf-40a9-ab1c-a8ab520c58fb"
       (reference "R?") (unit 1) (value "10") (footprint "")
@@
       (reference "R?") (unit 1) (value "10") (footprint "")
     )
+    (path "/8781658c-e5d4-40cc-b0c0-8e95668fb10a/5173a47a-a0f4-415b-bb81-5534715cf133"
+      (reference "R?") (unit 1) (value "1K") (footprint "")
+    )
     (path "/8781658c-e5d4-40cc-b0c0-8e95668fb10a/56c1df93-56c8-428b-b8d4-e22b85e8f6df"
       (reference "R?") (unit 1) (value "10") (footprint "")
@@
       (reference "U?") (unit 1) (value "INA226") (footprint "Package_SO:VSSOP-10_3x3mm_P0.5mm")
     )
+    (path "/8781658c-e5d4-40cc-b0c0-8e95668fb10a/8d9d9501-0672-453f-9e1c-8cfccbc06c38"
+      (reference "U?") (unit 1) (value "AD626ANZ") (footprint "N_8_ADI")
+    )
     (path "/b44f6773-e3e8-4e75-9d5c-4dbba7b405cd/9174172e-bc12-4bcf-8f61-493fa29bd79a"
       (reference "U?") (unit 1) (value "MCP601T-I/OT") (footprint "Package_TO_SOT_SMD:SOT-23-5")
@@
       (reference "U?") (unit 1) (value "LTM4611EV-PBF") (footprint "LGA-133_3_LIT")
     )
-    (path "/8781658c-e5d4-40cc-b0c0-8e95668fb10a/950724a2-f2e9-4b4b-8eb8-8328b128358b"
-      (reference "U?") (unit 1) (value "MCP601T-I/OT") (footprint "Package_TO_SOT_SMD:SOT-23-5")
-    )
     (path "/84d8ca1d-7213-486c-b202-d20639515304/9baa1757-0261-4cab-acfe-26d419706fc9"
