File: KiCAD/Quest_39/BUCK_6.kicad_sch (KiCad schematic)
At the start: 21 parts

Commit message: Fixed most ERC errors
Parts:
- gave numbers to parts that had none: 21
Changed lines of the file:
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@@
   (symbol (lib_id "Device:C") (at 55.88 55.88 90) (unit 1)
     (in_bom yes) (on_board yes)
-    (property "Reference" "C?" (id 0) (at 55.88 52.07 90))
+    (property "Reference" "C93" (id 0) (at 55.88 52.07 90))
     (property "Value" "1uF" (id 1) (at 55.88 59.69 90))
     (property "Footprint" "OptoDevice:R_LDR_4.9x4.2mm_P2.54mm_Vertical" (id 2) (at 59.69 54.9148 0)
@@
   (symbol (lib_id "Amplifier_Operational:MCP601-xOT") (at 35.56 66.04 0) (unit 1)
     (in_bom yes) (on_board yes)
-    (property "Reference" "U?" (id 0) (at 38.1 62.23 0))
+    (property "Reference" "U28" (id 0) (at 38.1 62.23 0))
     (property "Value" "MCP601T-I/OT" (id 1) (at 41.91 69.85 0))
     (property "Footprint" "Package_TO_SOT_SMD:SOT-23-5" (id 2) (at 33.02 71.12 0)
@@
   (symbol (lib_id "Device:C") (at 337.82 224.79 0) (unit 1)
     (in_bom yes) (on_board yes) (fields_autoplaced)
-    (property "Reference" "C?" (id 0) (at 341.63 223.5199 0)
+    (property "Reference" "C100" (id 0) (at 341.63 223.5199 0)
       (effects (font (size 1.27 1.27)) (justify left))
     )
@@
   (symbol (lib_id "Device:C_Polarized") (at 368.3 172.72 0) (unit 1)
     (in_bom yes) (on_board yes)
-    (property "Reference" "C?" (id 0) (at 372.0895 171.4075 0)
+    (property "Reference" "C97" (id 0) (at 372.0895 171.4075 0)
       (effects (font (size 1.27 1.27)) (justify left))
     )
@@
   (symbol (lib_id "Device:C") (at 113.03 46.99 0) (unit 1)
     (in_bom yes) (on_board yes) (fields_autoplaced)
-    (property "Reference" "C?" (id 0) (at 116.84 45.7199 0)
+    (property "Reference" "C91" (id 0) (at 116.84 45.7199 0)
       (effects (font (size 1.27 1.27)) (justify left))
     )
@@
   (symbol (lib_id "Analog_ADC:INA226") (at 78.74 73.66 0) (unit 1)
     (in_bom yes) (on_board yes)
-    (property "Reference" "U?" (id 0) (at 83.82 62.23 0)
+    (property "Reference" "U29" (id 0) (at 83.82 62.23 0)
       (effects (font (size 1.27 1.27)) (justify left))
     )
@@
   (symbol (lib_id "Device:R") (at 55.88 41.91 90) (unit 1)
     (in_bom yes) (on_board yes) (fields_autoplaced)
-    (property "Reference" "R?" (id 0) (at 55.88 35.56 90))
+    (property "Reference" "R38" (id 0) (at 55.88 35.56 90))
     (property "Value" "0R0025" (id 1) (at 55.88 38.1 90))
     (property "Footprint" "" (id 2) (at 55.88 43.688 90)
@@
   (symbol (lib_id "Device:C_Polarized") (at 86.36 46.99 0) (unit 1)
     (in_bom yes) (on_board yes) (fields_autoplaced)
-    (property "Reference" "C?" (id 0) (at 90.17 44.8309 0)
+    (property "Reference" "C89" (id 0) (at 90.17 44.8309 0)
       (effects (font (size 1.27 1.27)) (justify left))
     )
@@
   (symbol (lib_id "Device:C") (at 335.28 172.72 0) (unit 1)
     (in_bom yes) (on_board yes) (fields_autoplaced)
-    (property "Reference" "C?" (id 0) (at 339.09 171.4499 0)
+    (property "Reference" "C95" (id 0) (at 339.09 171.4499 0)
       (effects (font (size 1.27 1.27)) (justify left))
     )
@@
   (symbol (lib_id "MCP4151:MCP4151-502E{slash}SN") (at 254 220.98 0) (unit 1)
     (in_bom yes) (on_board yes)
-    (property "Reference" "U?" (id 0) (at 312.42 214.63 0)
+    (property "Reference" "U31" (id 0) (at 312.42 214.63 0)
       (effects (font (size 1.524 1.524)))
     )
@@
   (symbol (lib_id "Device:C_Polarized") (at 393.7 172.72 0) (unit 1)
     (in_bom yes) (on_board yes)
-    (property "Reference" "C?" (id 0) (at 397.4895 171.4075 0)
+    (property "Reference" "C99" (id 0) (at 397.4895 171.4075 0)
       (effects (font (size 1.27 1.27)) (justify left))
     )
@@
   (symbol (lib_id "Device:C") (at 100.33 46.99 0) (unit 1)
     (in_bom yes) (on_board yes) (fields_autoplaced)
-    (property "Reference" "C?" (id 0) (at 104.14 45.7199 0)
+    (property "Reference" "C90" (id 0) (at 104.14 45.7199 0)
       (effects (font (size 1.27 1.27)) (justify left))
     )
@@
   (symbol (lib_id "Device:R") (at 48.26 49.53 0) (unit 1)
     (in_bom yes) (on_board yes) (fields_autoplaced)
-    (property "Reference" "R?" (id 0) (at 50.8 48.2599 0)
+    (property "Reference" "R39" (id 0) (at 50.8 48.2599 0)
       (effects (font (size 1.27 1.27)) (justify left))
     )
@@
   (symbol (lib_id "Device:C") (at 125.73 46.99 0) (unit 1)
     (in_bom yes) (on_board yes) (fields_autoplaced)
-    (property "Reference" "C?" (id 0) (at 129.54 45.7199 0)
+    (property "Reference" "C92" (id 0) (at 129.54 45.7199 0)
       (effects (font (size 1.27 1.27)) (justify left))
     )
@@
   (symbol (lib_id "Device:R") (at 322.58 215.9 0) (unit 1)
     (in_bom yes) (on_board yes) (fields_autoplaced)
-    (property "Reference" "R?" (id 0) (at 325.12 214.6299 0)
+    (property "Reference" "R42" (id 0) (at 325.12 214.6299 0)
       (effects (font (size 1.27 1.27)) (justify left))
     )
@@
   (symbol (lib_id "Device:C_Polarized") (at 354.33 172.72 0) (unit 1)
     (in_bom yes) (on_board yes)
-    (property "Reference" "C?" (id 0) (at 358.1195 171.4075 0)
+    (property "Reference" "C96" (id 0) (at 358.1195 171.4075 0)
       (effects (font (size 1.27 1.27)) (justify left))
     )
@@
   (symbol (lib_id "LTM4611EV:LTM4611EV-PBF") (at 132.08 102.87 0) (unit 1)
     (in_bom yes) (on_board yes)
-    (property "Reference" "U?" (id 0) (at 308.61 50.8 0)
+    (property "Reference" "U30" (id 0) (at 308.61 50.8 0)
       (effects (font (size 1.524 1.524)))
     )
@@
   (symbol (lib_id "Device:R") (at 60.96 49.53 0) (unit 1)
     (in_bom yes) (on_board yes) (fields_autoplaced)
-    (property "Reference" "R?" (id 0) (at 63.5 48.2599 0)
+    (property "Reference" "R40" (id 0) (at 63.5 48.2599 0)
       (effects (font (size 1.27 1.27)) (justify left))
     )
@@
   (symbol (lib_id "Device:R") (at 127 91.44 0) (unit 1)
     (in_bom yes) (on_board yes) (fields_autoplaced)
-    (property "Reference" "R?" (id 0) (at 129.54 90.1699 0)
+    (property "Reference" "R41" (id 0) (at 129.54 90.1699 0)
       (effects (font (size 1.27 1.27)) (justify left))
     )
@@
   (symbol (lib_id "Device:C") (at 128.27 137.16 0) (unit 1)
     (in_bom yes) (on_board yes) (fields_autoplaced)
-    (property "Reference" "C?" (id 0) (at 132.08 135.8899 0)
+    (property "Reference" "C94" (id 0) (at 132.08 135.8899 0)
       (effects (font (size 1.27 1.27)) (justify left))
     )
@@
   (symbol (lib_id "Device:C_Polarized") (at 381 172.72 0) (unit 1)
     (in_bom yes) (on_board yes)
-    (property "Reference" "C?" (id 0) (at 384.7895 171.4075 0)
-      (effects (font (size 1.27 1.27)) (justify left))
-    )
+    (property "Reference" "C98" (id 0) (at 384.7895 171.4075 0)
+      (effects (font (size 1.27 1.27)) (justify left))
+    )

Commit message: Gave all INA226's unique addresses
Parts:
- removed C89: 330uF, symbol Device:C_Polarized
- removed C90, C91, C92: 22uF, symbol Device:C
- removed C93: 1uF, OptoDevice:R_LDR_4.9x4.2mm_P2.54mm_Vertical, symbol Device:C
- removed C94: 100nF, symbol Device:C
- removed C95: 100pF, symbol Device:C
- removed C96, C97, C99: 100uF, symbol Device:C_Polarized
- removed R38: 0R0025, symbol Device:R
- removed R39, R40: 10, symbol Device:R
- removed R41: 10K, symbol Device:R
- removed R42: 20K, symbol Device:R
- removed U28: MCP601T-I/OT, Package_TO_SOT_SMD:SOT-23-5, symbol Amplifier_Operational:MCP601-xOT
- added C101, C99: 22uF, symbol Device:C
- added C102: 1uF, OptoDevice:R_LDR_4.9x4.2mm_P2.54mm_Vertical, symbol Device:C
- added C103, C104, C111: 100nF, symbol Device:C
- added C105: 10nF, symbol Device:C
- added C106, C107, C108, C109: 100uF, symbol Device:C_Polarized
- added C110: 100pF, symbol Device:C
- added R59: 0R0025, symbol Device:R
- added R60, R61: 10R, symbol Device:R
- added R62: 9k, symbol Device:R
- added R63: 1k, symbol Device:R
- added R64: 10k, symbol Device:R
- added R65: 20K, symbol Device:R
- added TP48, TP49, TP50, TP51, TP52, TP53, TP54: TestPoint, symbol Connector:TestPoint
- added U28: AD626ANZ, N_8_ADI, symbol AD626ANZ:AD626ANZ
- C100: value 100nF -> 22uF
- C98: value 100uF -> 330uF
Connections:
- net +5V: now also U29.1 (A1), C104.1, C111.1, U28.6 (+VS); no longer C100.1
- net GND: now also C103.2, C104.2, C111.2, U28.2 (AGND), U28.3 (-VS); no longer C100.2, U29.1 (A1), U29.2 (A0), U29.3 (~{Alert})
- net NEG: now also C100.2, C101.2, C105.1, C106.2, C107.2, C108.2, C109.2, C99.2, R63.2, U28.1 (-IN); no longer U29.8 (Vbus)
- net P0A: now also R65.2
- net POS: now also C106.1, C107.1, C108.1, C109.1, C110.1; no longer C98.1
- net PV_POS: now also C100.1, C98.1, U30.A1 (VIN), U30.A2 (VIN), U30.A3 (VIN), U30.A4 (VIN), U30.A5 (VIN), U30.A6 (VIN), U30.B1 (VIN), U30.B2 (VIN), U30.B3 (VIN), U30.B4 (VIN), U30.B5 (VIN), U30.B6 (VIN), U30.C1 (VIN), U30.C2 (VIN), U30.C3 (VIN), U30.C4 (VIN), U30.C5 (VIN), U30.C6 (VIN), C101.1, C99.1, R59.1, R59.2, R60.1, R61.1, R62.1, R64.1
- net RUN: now also R64.2
- net SDA: now also U29.2 (A0)
- net TRACK/SS: now also C105.2
- net Vfb: now also C110.2, R65.1
- net Vin+: now also C102.1, R60.2
- net Vin-: now also U29.8 (Vbus), U29.9 (Vin-), C102.2, R61.2, TP49.1, U28.5 (OUT)
- net at U30.A11 (COMP): now also TP52.1
- net at U30.A7 (INTVCC): now also U30.D9 (INTVCC), TP48.1
- net at U30.B12 (PLLFLTR/FSET): now also TP51.1
- net at U30.F11 (PGOOD): now also U30.G12 (PGOOD), TP50.1
- net at U30.K12 (DIFFVOUT), U30.L12 (VOUT_LCL): now also TP53.1, TP54.1
- new net: C103.1, U28.4 (FILTER)
- new net +IN: R62.2, R63.1, U28.8 (+IN)
- no-connect marks 16 -> 12
Other:
- note added: "10:1 divider"
- note added: "Addr=0x46"
- note added: "Extra mounting"
- note added: "G=10"
- note added: "Output voltage is set by varying Rfb with a digipot. SPI = 00"
- note added: "the measured voltage is divided and then amplified by 10 as to simulate a follower. This is done to make use of the AD626 (low price and availability)."

Commit message: Assigned all schem. symbols their footprints
Parts:
- removed C106, C107, C108, C109: 100uF, symbol Device:C_Polarized
- added C106, C107, C108, C109: 100uF, Capacitor_SMD:C_1206_3216Metric, symbol Device:C
- C100, C101, C103, C104, C105, C110, C111, C99: footprint (none) -> Capacitor_SMD:C_0805_2012Metric
- C102: footprint OptoDevice:R_LDR_4.9x4.2mm_P2.54mm_Vertical -> Capacitor_SMD:C_0805_2012Metric
- C98: footprint (none) -> Capacitor_SMD:CP_Elec_8x6.9
- R59: footprint (none) -> Resistor_SMD:R_1206_3216Metric
- R60, R61, R62, R63, R64, R65: footprint (none) -> Resistor_SMD:R_0805_2012Metric
- TP48, TP49, TP50, TP51, TP52, TP53, TP54: footprint (none) -> TestPoint:TestPoint_Pad_D2.0mm
- U28: footprint N_8_ADI -> Package_DIP:DIP-8_W7.62mm_Socket_LongPads
- U30: footprint LGA-133_3_LIT -> Package_LGA:Linear_LGA-133_15.0x15.0mm_Layout12x12_P1.27mm
- U31: footprint SOIC8-N_MC_MCH -> Package_SO:MSOP-8_3x3mm_P0.65mm
Connections:
- net NEG: now also C106.2, C107.2, C108.2, C109.2
- net POS: now also C106.1, C107.1, C108.1, C109.1

Commit message: Initial work on layout
Parts:
- C102, C103, C104, C105, C110, C111: footprint Capacitor_SMD:C_0805_2012Metric -> Capacitor_SMD:C_0603_1608Metric
Changed lines of the file:
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@@
       (effects (font (size 1.27 1.27)) (justify left))
     )
-    (property "Footprint" "Capacitor_SMD:C_0805_2012Metric" (id 2) (at 345.1352 168.91 0)
+    (property "Footprint" "Capacitor_SMD:C_0603_1608Metric" (id 2) (at 345.1352 168.91 0)
       (effects (font (size 1.27 1.27)) hide)
     )
@@
     (property "Reference" "C102" (id 0) (at 74.93 57.15 90))
     (property "Value" "1uF" (id 1) (at 74.93 64.77 90))
-    (property "Footprint" "Capacitor_SMD:C_0805_2012Metric" (id 2) (at 78.74 59.9948 0)
+    (property "Footprint" "Capacitor_SMD:C_0603_1608Metric" (id 2) (at 78.74 59.9948 0)
       (effects (font (size 1.27 1.27)) hide)
     )
@@
       (effects (font (size 1.27 1.27)) (justify left))
     )
-    (property "Footprint" "Capacitor_SMD:C_0805_2012Metric" (id 2) (at 106.3752 124.46 0)
+    (property "Footprint" "Capacitor_SMD:C_0603_1608Metric" (id 2) (at 106.3752 124.46 0)
       (effects (font (size 1.27 1.27)) hide)
     )
@@
       (effects (font (size 1.27 1.27)) (justify left))
     )
-    (property "Footprint" "Capacitor_SMD:C_0805_2012Metric" (id 2) (at 26.3652 81.28 0)
+    (property "Footprint" "Capacitor_SMD:C_0603_1608Metric" (id 2) (at 26.3652 81.28 0)
       (effects (font (size 1.27 1.27)) hide)
     )
@@
       (effects (font (size 1.27 1.27)) (justify left))
     )
-    (property "Footprint" "Capacitor_SMD:C_0805_2012Metric" (id 2) (at 64.4652 82.55 0)
+    (property "Footprint" "Capacitor_SMD:C_0603_1608Metric" (id 2) (at 64.4652 82.55 0)
       (effects (font (size 1.27 1.27)) hide)
     )
@@
       (effects (font (size 1.27 1.27)) (justify left))
     )
-    (property "Footprint" "Capacitor_SMD:C_0805_2012Metric" (id 2) (at 341.3252 220.98 0)
-      (effects (font (size 1.27 1.27)) hide)
-    )
+    (property "Footprint" "Capacitor_SMD:C_0603_1608Metric" (id 2) (at 341.3252 220.98 0)
+      (effects (font (size 1.27 1.27)) hide)
+    )
