File: KiCAD/Quest_39/BUCK_8.kicad_sch (KiCad schematic)
At the start: 21 parts

Commit message: Fixed most ERC errors
Parts:
- gave numbers to parts that had none: 21
Changed lines of the file:
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@@
   (symbol (lib_id "Device:C") (at 337.82 224.79 0) (unit 1)
     (in_bom yes) (on_board yes) (fields_autoplaced)
-    (property "Reference" "C?" (id 0) (at 341.63 223.5199 0)
+    (property "Reference" "C124" (id 0) (at 341.63 223.5199 0)
       (effects (font (size 1.27 1.27)) (justify left))
     )
@@
   (symbol (lib_id "Device:R") (at 60.96 49.53 0) (unit 1)
     (in_bom yes) (on_board yes) (fields_autoplaced)
-    (property "Reference" "R?" (id 0) (at 63.5 48.2599 0)
+    (property "Reference" "R50" (id 0) (at 63.5 48.2599 0)
       (effects (font (size 1.27 1.27)) (justify left))
     )
@@
   (symbol (lib_id "Device:C_Polarized") (at 393.7 172.72 0) (unit 1)
     (in_bom yes) (on_board yes)
-    (property "Reference" "C?" (id 0) (at 397.4895 171.4075 0)
+    (property "Reference" "C123" (id 0) (at 397.4895 171.4075 0)
       (effects (font (size 1.27 1.27)) (justify left))
     )
@@
   (symbol (lib_id "Device:C") (at 113.03 46.99 0) (unit 1)
     (in_bom yes) (on_board yes) (fields_autoplaced)
-    (property "Reference" "C?" (id 0) (at 116.84 45.7199 0)
+    (property "Reference" "C115" (id 0) (at 116.84 45.7199 0)
       (effects (font (size 1.27 1.27)) (justify left))
     )
@@
   (symbol (lib_id "Device:C") (at 100.33 46.99 0) (unit 1)
     (in_bom yes) (on_board yes) (fields_autoplaced)
-    (property "Reference" "C?" (id 0) (at 104.14 45.7199 0)
+    (property "Reference" "C114" (id 0) (at 104.14 45.7199 0)
       (effects (font (size 1.27 1.27)) (justify left))
     )
@@
   (symbol (lib_id "Device:C") (at 55.88 55.88 90) (unit 1)
     (in_bom yes) (on_board yes)
-    (property "Reference" "C?" (id 0) (at 55.88 52.07 90))
+    (property "Reference" "C117" (id 0) (at 55.88 52.07 90))
     (property "Value" "1uF" (id 1) (at 55.88 59.69 90))
     (property "Footprint" "OptoDevice:R_LDR_4.9x4.2mm_P2.54mm_Vertical" (id 2) (at 59.69 54.9148 0)
@@
   (symbol (lib_id "Analog_ADC:INA226") (at 78.74 73.66 0) (unit 1)
     (in_bom yes) (on_board yes)
-    (property "Reference" "U?" (id 0) (at 83.82 62.23 0)
+    (property "Reference" "U37" (id 0) (at 83.82 62.23 0)
       (effects (font (size 1.27 1.27)) (justify left))
     )
@@
   (symbol (lib_id "Device:R") (at 48.26 49.53 0) (unit 1)
     (in_bom yes) (on_board yes) (fields_autoplaced)
-    (property "Reference" "R?" (id 0) (at 50.8 48.2599 0)
+    (property "Reference" "R49" (id 0) (at 50.8 48.2599 0)
       (effects (font (size 1.27 1.27)) (justify left))
     )
@@
   (symbol (lib_id "Device:C_Polarized") (at 381 172.72 0) (unit 1)
     (in_bom yes) (on_board yes)
-    (property "Reference" "C?" (id 0) (at 384.7895 171.4075 0)
+    (property "Reference" "C122" (id 0) (at 384.7895 171.4075 0)
       (effects (font (size 1.27 1.27)) (justify left))
     )
@@
   (symbol (lib_id "Device:C") (at 335.28 172.72 0) (unit 1)
     (in_bom yes) (on_board yes) (fields_autoplaced)
-    (property "Reference" "C?" (id 0) (at 339.09 171.4499 0)
+    (property "Reference" "C119" (id 0) (at 339.09 171.4499 0)
       (effects (font (size 1.27 1.27)) (justify left))
     )
@@
   (symbol (lib_id "Device:C") (at 125.73 46.99 0) (unit 1)
     (in_bom yes) (on_board yes) (fields_autoplaced)
-    (property "Reference" "C?" (id 0) (at 129.54 45.7199 0)
+    (property "Reference" "C116" (id 0) (at 129.54 45.7199 0)
       (effects (font (size 1.27 1.27)) (justify left))
     )
@@
   (symbol (lib_id "LTM4611EV:LTM4611EV-PBF") (at 132.08 102.87 0) (unit 1)
     (in_bom yes) (on_board yes)
-    (property "Reference" "U?" (id 0) (at 308.61 50.8 0)
+    (property "Reference" "U38" (id 0) (at 308.61 50.8 0)
       (effects (font (size 1.524 1.524)))
     )
@@
   (symbol (lib_id "Device:C") (at 128.27 137.16 0) (unit 1)
     (in_bom yes) (on_board yes) (fields_autoplaced)
-    (property "Reference" "C?" (id 0) (at 132.08 135.8899 0)
+    (property "Reference" "C118" (id 0) (at 132.08 135.8899 0)
       (effects (font (size 1.27 1.27)) (justify left))
     )
@@
   (symbol (lib_id "Device:C_Polarized") (at 368.3 172.72 0) (unit 1)
     (in_bom yes) (on_board yes)
-    (property "Reference" "C?" (id 0) (at 372.0895 171.4075 0)
+    (property "Reference" "C121" (id 0) (at 372.0895 171.4075 0)
       (effects (font (size 1.27 1.27)) (justify left))
     )
@@
   (symbol (lib_id "Device:C_Polarized") (at 354.33 172.72 0) (unit 1)
     (in_bom yes) (on_board yes)
-    (property "Reference" "C?" (id 0) (at 358.1195 171.4075 0)
+    (property "Reference" "C120" (id 0) (at 358.1195 171.4075 0)
       (effects (font (size 1.27 1.27)) (justify left))
     )
@@
   (symbol (lib_id "Amplifier_Operational:MCP601-xOT") (at 35.56 66.04 0) (unit 1)
     (in_bom yes) (on_board yes)
-    (property "Reference" "U?" (id 0) (at 38.1 62.23 0))
+    (property "Reference" "U36" (id 0) (at 38.1 62.23 0))
     (property "Value" "MCP601T-I/OT" (id 1) (at 41.91 69.85 0))
     (property "Footprint" "Package_TO_SOT_SMD:SOT-23-5" (id 2) (at 33.02 71.12 0)
@@
   (symbol (lib_id "Device:R") (at 322.58 215.9 0) (unit 1)
     (in_bom yes) (on_board yes) (fields_autoplaced)
-    (property "Reference" "R?" (id 0) (at 325.12 214.6299 0)
+    (property "Reference" "R52" (id 0) (at 325.12 214.6299 0)
       (effects (font (size 1.27 1.27)) (justify left))
     )
@@
   (symbol (lib_id "Device:R") (at 127 91.44 0) (unit 1)
     (in_bom yes) (on_board yes) (fields_autoplaced)
-    (property "Reference" "R?" (id 0) (at 129.54 90.1699 0)
+    (property "Reference" "R51" (id 0) (at 129.54 90.1699 0)
       (effects (font (size 1.27 1.27)) (justify left))
     )
@@
   (symbol (lib_id "Device:C_Polarized") (at 86.36 46.99 0) (unit 1)
     (in_bom yes) (on_board yes) (fields_autoplaced)
-    (property "Reference" "C?" (id 0) (at 90.17 44.8309 0)
+    (property "Reference" "C113" (id 0) (at 90.17 44.8309 0)
       (effects (font (size 1.27 1.27)) (justify left))
     )
@@
   (symbol (lib_id "Device:R") (at 55.88 41.91 90) (unit 1)
     (in_bom yes) (on_board yes) (fields_autoplaced)
-    (property "Reference" "R?" (id 0) (at 55.88 35.56 90))
+    (property "Reference" "R48" (id 0) (at 55.88 35.56 90))
     (property "Value" "0R0025" (id 1) (at 55.88 38.1 90))
     (property "Footprint" "" (id 2) (at 55.88 43.688 90)
@@
   (symbol (lib_id "MCP4151:MCP4151-502E{slash}SN") (at 254 220.98 0) (unit 1)
     (in_bom yes) (on_board yes)
-    (property "Reference" "U?" (id 0) (at 312.42 214.63 0)
+    (property "Reference" "U39" (id 0) (at 312.42 214.63 0)
       (effects (font (size 1.524 1.524)))
     )

Commit message: Gave all INA226's unique addresses
Parts:
- removed C113: 330uF, symbol Device:C_Polarized
- removed C114, C115, C116: 22uF, symbol Device:C
- removed C117: 1uF, OptoDevice:R_LDR_4.9x4.2mm_P2.54mm_Vertical, symbol Device:C
- removed C118, C124: 100nF, symbol Device:C
- removed C119: 100pF, symbol Device:C
- removed C120, C121, C122, C123: 100uF, symbol Device:C_Polarized
- removed R48: 0R0025, symbol Device:R
- removed R49, R50: 10, symbol Device:R
- removed R51: 10K, symbol Device:R
- removed R52: 20K, symbol Device:R
- removed U36: MCP601T-I/OT, Package_TO_SOT_SMD:SOT-23-5, symbol Amplifier_Operational:MCP601-xOT
- added C126: 330uF, symbol Device:C_Polarized
- added C127, C128, C129: 22uF, symbol Device:C
- added C130: 1uF, OptoDevice:R_LDR_4.9x4.2mm_P2.54mm_Vertical, symbol Device:C
- added C131, C132, C139: 100nF, symbol Device:C
- added C133: 10nF, symbol Device:C
- added C134, C135, C136, C137: 100uF, symbol Device:C_Polarized
- added C138: 100pF, symbol Device:C
- added R73: 0R0025, symbol Device:R
- added R74, R75: 10R, symbol Device:R
- added R76: 9k, symbol Device:R
- added R77: 1k, symbol Device:R
- added R78: 10k, symbol Device:R
- added R79: 20K, symbol Device:R
- added TP62, TP63, TP64, TP65, TP66, TP67, TP68: TestPoint, symbol Connector:TestPoint
- added U36: AD626ANZ, N_8_ADI, symbol AD626ANZ:AD626ANZ
Connections:
- net +5V: now also C132.1, C139.1, U36.6 (+VS)
- net GND: now also C131.2, C132.2, C139.2, U36.2 (AGND), U36.3 (-VS); no longer U37.1 (A1), U37.3 (~{Alert})
- net NEG: now also C126.2, C127.2, C128.2, C129.2, C133.1, C134.2, C135.2, C136.2, C137.2, R77.2, U36.1 (-IN); no longer U37.8 (Vbus)
- net P0A: now also R79.2
- net POS: now also C134.1, C135.1, C136.1, C137.1, C138.1
- net PV_POS: now also U38.A1 (VIN), U38.A2 (VIN), U38.A3 (VIN), U38.A4 (VIN), U38.A5 (VIN), U38.A6 (VIN), U38.B1 (VIN), U38.B2 (VIN), U38.B3 (VIN), U38.B4 (VIN), U38.B5 (VIN), U38.B6 (VIN), U38.C1 (VIN), U38.C2 (VIN), U38.C3 (VIN), U38.C4 (VIN), U38.C5 (VIN), U38.C6 (VIN), C126.1, C127.1, C128.1, C129.1, R73.1, R73.2, R74.1, R75.1, R76.1, R78.1
- net RUN: now also R78.2
- net SDA: now also U37.1 (A1)
- net TRACK/SS: now also C133.2
- net Vfb: now also C138.2, R79.1
- net Vin+: now also C130.1, R74.2
- net Vin-: now also U37.8 (Vbus), U37.9 (Vin-), C130.2, R75.2, TP63.1, U36.5 (OUT)
- net at U38.A11 (COMP): now also TP66.1
- net at U38.A7 (INTVCC): now also U38.D9 (INTVCC), TP62.1
- net at U38.B12 (PLLFLTR/FSET): now also TP65.1
- net at U38.F11 (PGOOD): now also U38.G12 (PGOOD), TP64.1
- net at U38.K12 (DIFFVOUT), U38.L12 (VOUT_LCL): now also TP67.1, TP68.1
- new net: C131.1, U36.4 (FILTER)
- new net +IN: R76.2, R77.1, U36.8 (+IN)
- no-connect marks 16 -> 12
Other:
- note added: "10:1 divider"
- note added: "Addr=0x48"
- note added: "Extra mounting"
- note added: "G=10"
- note added: "Output voltage is set by varying Rfb with a digipot. SPI = 00"
- note added: "the measured voltage is divided and then amplified by 10 as to simulate a follower. This is done to make use of the AD626 (low price and availability)."

Commit message: Assigned all schem. symbols their footprints
Parts:
- removed C134, C135, C136, C137: 100uF, symbol Device:C_Polarized
- added C134, C135, C136, C137: 100uF, Capacitor_SMD:C_1206_3216Metric, symbol Device:C
- C126: footprint (none) -> Capacitor_SMD:CP_Elec_8x6.9
- C127, C128, C129, C131, C132, C133, C138, C139: footprint (none) -> Capacitor_SMD:C_0805_2012Metric
- C130: footprint OptoDevice:R_LDR_4.9x4.2mm_P2.54mm_Vertical -> Capacitor_SMD:C_0805_2012Metric
- R73: footprint (none) -> Resistor_SMD:R_1206_3216Metric
- R74, R75, R76, R77, R78, R79: footprint (none) -> Resistor_SMD:R_0805_2012Metric
- TP62, TP63, TP64, TP65, TP66, TP67, TP68: footprint (none) -> TestPoint:TestPoint_Pad_D2.0mm
- U36: footprint N_8_ADI -> Package_DIP:DIP-8_W7.62mm_Socket_LongPads
- U38: footprint LGA-133_3_LIT -> Package_LGA:Linear_LGA-133_15.0x15.0mm_Layout12x12_P1.27mm
- U39: footprint SOIC8-N_MC_MCH -> Package_SO:MSOP-8_3x3mm_P0.65mm
Connections:
- net NEG: now also C134.2, C135.2, C136.2, C137.2
- net POS: now also C134.1, C135.1, C136.1, C137.1

Commit message: Initial work on layout
Parts:
- C130, C131, C132, C133, C138, C139: footprint Capacitor_SMD:C_0805_2012Metric -> Capacitor_SMD:C_0603_1608Metric
Changed lines of the file:
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@@
       (effects (font (size 1.27 1.27)) (justify left))
     )
-    (property "Footprint" "Capacitor_SMD:C_0805_2012Metric" (id 2) (at 26.3652 83.82 0)
+    (property "Footprint" "Capacitor_SMD:C_0603_1608Metric" (id 2) (at 26.3652 83.82 0)
       (effects (font (size 1.27 1.27)) hide)
     )
@@
       (effects (font (size 1.27 1.27)) (justify left))
     )
-    (property "Footprint" "Capacitor_SMD:C_0805_2012Metric" (id 2) (at 345.1352 171.45 0)
+    (property "Footprint" "Capacitor_SMD:C_0603_1608Metric" (id 2) (at 345.1352 171.45 0)
       (effects (font (size 1.27 1.27)) hide)
     )
@@
     (property "Reference" "C130" (id 0) (at 74.93 59.69 90))
     (property "Value" "1uF" (id 1) (at 74.93 67.31 90))
-    (property "Footprint" "Capacitor_SMD:C_0805_2012Metric" (id 2) (at 78.74 62.5348 0)
+    (property "Footprint" "Capacitor_SMD:C_0603_1608Metric" (id 2) (at 78.74 62.5348 0)
       (effects (font (size 1.27 1.27)) hide)
     )
@@
       (effects (font (size 1.27 1.27)) (justify left))
     )
-    (property "Footprint" "Capacitor_SMD:C_0805_2012Metric" (id 2) (at 106.3752 127 0)
+    (property "Footprint" "Capacitor_SMD:C_0603_1608Metric" (id 2) (at 106.3752 127 0)
       (effects (font (size 1.27 1.27)) hide)
     )
@@
       (effects (font (size 1.27 1.27)) (justify left))
     )
-    (property "Footprint" "Capacitor_SMD:C_0805_2012Metric" (id 2) (at 64.4652 85.09 0)
+    (property "Footprint" "Capacitor_SMD:C_0603_1608Metric" (id 2) (at 64.4652 85.09 0)
       (effects (font (size 1.27 1.27)) hide)
     )
@@
       (effects (font (size 1.27 1.27)) (justify left))
     )
-    (property "Footprint" "Capacitor_SMD:C_0805_2012Metric" (id 2) (at 341.3252 223.52 0)
-      (effects (font (size 1.27 1.27)) hide)
-    )
+    (property "Footprint" "Capacitor_SMD:C_0603_1608Metric" (id 2) (at 341.3252 223.52 0)
+      (effects (font (size 1.27 1.27)) hide)
+    )
