File: KiCAD/Quest_39/Quest_39.kicad_pcb (KiCad board)
At the start: 2 copper layers, 378 parts, among them J1 1x2 Scr. Term., J10 1x2 Scr. Term., J11 1x2 Scr. Term., J12 Conn_01x05_Male, J2 1x2 Scr. Term., J3 1x2 Scr. Term., J4 1x2 Scr. Term., J5 1x2 Scr. Term., J6 1x2 Scr. Term., J7 1x2 Scr. Term., J8 1x2 Scr. Term., J9 1x2 Scr. Term., U1 AZ1117-3.3, U10 LTM4611EV-PBF, U11 MCP4151-502E/SN, U12 AD626ANZ, U13 INA226, U14 LTM4611EV-PBF, U15 MCP4151-502E/SN, U16 AD626ANZ, U17 INA226, U18 LTM4611EV-PBF, U19 MCP4151-502E/SN, U2 17791063215, U20 AD626ANZ, U21 INA226, U22 LTM4611EV-PBF, U23 MCP4151-502E/SN, U24 AD626ANZ, U25 INA226, U26 LTM4611EV-PBF, U27 MCP4151-502E/SN, U28 AD626ANZ, U29 INA226, U3 STM32F103C8T6, U30 LTM4611EV-PBF, U31 MCP4151-502E/SN, U32 AD626ANZ, U33 INA226, U34 LTM4611EV-PBF, U35 MCP4151-502E/SN, U36 AD626ANZ, U37 INA226, U38 LTM4611EV-PBF, U39 MCP4151-502E/SN, U4 AD626ANZ, U40 AD626ANZ, U41 INA226, U42 LTM4611EV-PBF, U43 MCP4151-502E/SN, U5 INA226, U6 LTM4611EV-PBF, U7 MCP4151-502E/SN, U8 AD626ANZ, U9 INA226, Y1 16MHz

Commit message: Fixed INA226 schem. mistake and further layout work
Parts:
- added C108: 100nF, Capacitor_SMD:C_0603_1608Metric, F.Cu at (48.1, 339.6)
- added C123: 100nF, Capacitor_SMD:C_0603_1608Metric, F.Cu at (40.0, 345.4)
- added C138: 100nF, Capacitor_SMD:C_0603_1608Metric, F.Cu at (56.1, 345.4)
- added C153: 100nF, Capacitor_SMD:C_0603_1608Metric, F.Cu at (48.1, 351.3)
- added C19: 100nF, Capacitor_SMD:C_0603_1608Metric, F.Cu at (48.1, 345.4)
- added C33: 100nF, Capacitor_SMD:C_0603_1608Metric, F.Cu at (40.0, 339.6)
- added C49: 100nF, Capacitor_SMD:C_0603_1608Metric, F.Cu at (56.1, 339.6)
- added C63: 100nF, Capacitor_SMD:C_0603_1608Metric, F.Cu at (64.2, 339.6)
- added C79: 100nF, Capacitor_SMD:C_0603_1608Metric, F.Cu at (40.0, 351.3)
- added C93: 100nF, Capacitor_SMD:C_0603_1608Metric, F.Cu at (56.1, 351.3)
- moved C29 342.6 mm to (217.6, 63.5)
- moved C32 342.6 mm to (235.7, 55.3)
- moved C37 342.6 mm to (240.1, 55.3)
- moved C39 342.6 mm to (226.7, 64.8)
- moved C40 342.6 mm to (230.6, 55.5)
- moved C41 342.6 mm to (242.3, 48.2)
- moved C42 342.6 mm to (247.4, 51.4)
- moved C43 342.6 mm to (231.8, 64.6)
- moved R24 342.6 mm to (242.3, 51.5)
- moved R25 342.6 mm to (253.6, 46.5)
- moved R26 342.6 mm to (236.2, 62.0)
- moved R27 342.6 mm to (243.6, 58.3)
- moved R28 342.6 mm to (244.5, 54.6)
- moved R30 342.6 mm to (236.2, 65.0)
- moved TP13 342.6 mm to (251.6, 50.0)
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- renumbered C94 to C100, C95 to C101, C96 to C102, C97 to C103, C98 to C104, C99 to C105, C100 to C106, C101 to C107, C102 to C109, C103 to C110, C104 to C111, C105 to C112, C106 to C113, C107 to C114, C108 to C115, C109 to C116, C110 to C117, C111 to C118, C112 to C119, C113 to C120, C114 to C121, C115 to C122, C116 to C124, C117 to C125, C118 to C126, C119 to C127, C120 to C128, C121 to C129, C122 to C130, C123 to C131, C124 to C132, C125 to C133, C126 to C134, C127 to C135, C128 to C136, C129 to C137, C130 to C139, C131 to C140, C132 to C141, C133 to C142, C134 to C143, C135 to C144, C136 to C145, C137 to C146, C138 to C147, C139 to C148, C140 to C149, C141 to C150, C142 to C151, C143 to C152, C144 to C154, C145 to C155, C146 to C156, C147 to C157, C148 to C158, C149 to C159, C150 to C160, C151 to C161, C152 to C162, C153 to C163, C19 to C20, C20 to C21, C21 to C22, C22 to C23, C23 to C24, C24 to C25, C25 to C26, C26 to C27, C27 to C28, C28 to C29, C29 to C30, C30 to C31, C31 to C32, C32 to C34, C33 to C35, C34 to C36, C35 to C37, C36 to C38, C37 to C39, C38 to C40, C39 to C41, C40 to C42, C41 to C43, C42 to C44, C43 to C45, C44 to C46, C45 to C47, C46 to C48, C47 to C50, C48 to C51, C49 to C52, C50 to C53, C51 to C54, C52 to C55, C53 to C56, C54 to C57, C55 to C58, C56 to C59, C57 to C60, C58 to C61, C59 to C62, C60 to C64, C61 to C65, C62 to C66, C63 to C67, C64 to C68, C65 to C69, C66 to C70, C67 to C71, C68 to C72, C69 to C73, C70 to C74, C71 to C75, C72 to C76, C73 to C77, C74 to C78, C75 to C80, C76 to C81, C77 to C82, C78 to C83, C79 to C84, C80 to C85, C81 to C86, C82 to C87, C83 to C88, C84 to C89, C85 to C90, C86 to C91, C87 to C92, C88 to C94, C89 to C95, C90 to C96, C91 to C97, C92 to C98, C93 to C99
Connections:
- C104 pad 1: /PV_POS_6 -> /BUCK_6/BUCK_VIN
- C105 pad 1: /PV_POS_6 -> /BUCK_6/BUCK_VIN
- C106 pad 1: /PV_POS_6 -> /BUCK_6/BUCK_VIN
- C107 pad 1: /PV_POS_6 -> /BUCK_6/BUCK_VIN
- C119 pad 1: /PV_POS_7 -> /BUCK_7/BUCK_VIN
- C120 pad 1: /PV_POS_7 -> /BUCK_7/BUCK_VIN
- C121 pad 1: /PV_POS_7 -> /BUCK_7/BUCK_VIN
- C122 pad 1: /PV_POS_7 -> /BUCK_7/BUCK_VIN
- C134 pad 1: /PV_POS_8 -> /BUCK_8/BUCK_VIN
- C135 pad 1: /PV_POS_8 -> /BUCK_8/BUCK_VIN
- C136 pad 1: /PV_POS_8 -> /BUCK_8/BUCK_VIN
- C137 pad 1: /PV_POS_8 -> /BUCK_8/BUCK_VIN
- C14 pad 1: /PV_POS_0 -> /BUCK_0/BUCK_VIN
- C149 pad 1: /PV_POS_9 -> /BUCK_9/BUCK_VIN
- C15 pad 1: /PV_POS_0 -> /BUCK_0/BUCK_VIN
- C150 pad 1: /PV_POS_9 -> /BUCK_9/BUCK_VIN
- C151 pad 1: /PV_POS_9 -> /BUCK_9/BUCK_VIN
- C152 pad 1: /PV_POS_9 -> /BUCK_9/BUCK_VIN
- C16 pad 1: /PV_POS_0 -> /BUCK_0/BUCK_VIN
- C17 pad 1: /PV_POS_0 -> /BUCK_0/BUCK_VIN
- C18 pad 1: /BUCK_0/Vin+ -> /BUCK_0/Vin-
- C18 pad 2: /BUCK_0/Vin- -> /BUCK_0/Vin+
- C29 pad 1: /PV_POS_1 -> /BUCK_1/BUCK_VIN
- C30 pad 1: /PV_POS_1 -> /BUCK_1/BUCK_VIN
- C31 pad 1: /PV_POS_1 -> /BUCK_1/BUCK_VIN
- C32 pad 1: /PV_POS_1 -> /BUCK_1/BUCK_VIN
- C44 pad 1: /PV_POS_2 -> /BUCK_2/BUCK_VIN
- C45 pad 1: /PV_POS_2 -> /BUCK_2/BUCK_VIN
- C46 pad 1: /PV_POS_2 -> /BUCK_2/BUCK_VIN
- C47 pad 1: /PV_POS_2 -> /BUCK_2/BUCK_VIN
- C59 pad 1: /PV_POS_4 -> /BUCK_4/BUCK_VIN
- C60 pad 1: /PV_POS_4 -> /BUCK_4/BUCK_VIN
- C61 pad 1: /PV_POS_4 -> /BUCK_4/BUCK_VIN
- C62 pad 1: /PV_POS_4 -> /BUCK_4/BUCK_VIN
- C74 pad 1: /PV_POS_3 -> /BUCK_3/BUCK_VIN
- C75 pad 1: /PV_POS_3 -> /BUCK_3/BUCK_VIN
- C76 pad 1: /PV_POS_3 -> /BUCK_3/BUCK_VIN
- C77 pad 1: /PV_POS_3 -> /BUCK_3/BUCK_VIN
- C89 pad 1: /PV_POS_5 -> /BUCK_5/BUCK_VIN
- C90 pad 1: /PV_POS_5 -> /BUCK_5/BUCK_VIN
- C91 pad 1: /PV_POS_5 -> /BUCK_5/BUCK_VIN
- C92 pad 1: /PV_POS_5 -> /BUCK_5/BUCK_VIN
- R17 pad 2: /PV_POS_0 -> /BUCK_0/BUCK_VIN
- R19 pad 1: /PV_POS_0 -> /BUCK_0/BUCK_VIN
- R22 pad 1: /PV_POS_0 -> /BUCK_0/BUCK_VIN
- R24 pad 2: /PV_POS_1 -> /BUCK_1/BUCK_VIN
- R26 pad 1: /PV_POS_1 -> /BUCK_1/BUCK_VIN
- R29 pad 1: /PV_POS_1 -> /BUCK_1/BUCK_VIN
- R31 pad 2: /PV_POS_2 -> /BUCK_2/BUCK_VIN
- R33 pad 1: /PV_POS_2 -> /BUCK_2/BUCK_VIN
- R36 pad 1: /PV_POS_2 -> /BUCK_2/BUCK_VIN
- R38 pad 2: /PV_POS_4 -> /BUCK_4/BUCK_VIN
- R40 pad 1: /PV_POS_4 -> /BUCK_4/BUCK_VIN
- R43 pad 1: /PV_POS_4 -> /BUCK_4/BUCK_VIN
- R45 pad 2: /PV_POS_3 -> /BUCK_3/BUCK_VIN
- R47 pad 1: /PV_POS_3 -> /BUCK_3/BUCK_VIN
- R50 pad 1: /PV_POS_3 -> /BUCK_3/BUCK_VIN
- R52 pad 2: /PV_POS_5 -> /BUCK_5/BUCK_VIN
- R54 pad 1: /PV_POS_5 -> /BUCK_5/BUCK_VIN
- R57 pad 1: /PV_POS_5 -> /BUCK_5/BUCK_VIN
- R59 pad 2: /PV_POS_6 -> /BUCK_6/BUCK_VIN
- R61 pad 1: /PV_POS_6 -> /BUCK_6/BUCK_VIN
- R64 pad 1: /PV_POS_6 -> /BUCK_6/BUCK_VIN
- R66 pad 2: /PV_POS_7 -> /BUCK_7/BUCK_VIN
- R68 pad 1: /PV_POS_7 -> /BUCK_7/BUCK_VIN
- R71 pad 1: /PV_POS_7 -> /BUCK_7/BUCK_VIN
- R73 pad 2: /PV_POS_8 -> /BUCK_8/BUCK_VIN
- R75 pad 1: /PV_POS_8 -> /BUCK_8/BUCK_VIN
- R78 pad 1: /PV_POS_8 -> /BUCK_8/BUCK_VIN
- R80 pad 2: /PV_POS_9 -> /BUCK_9/BUCK_VIN
- R82 pad 1: /PV_POS_9 -> /BUCK_9/BUCK_VIN
- R85 pad 1: /PV_POS_9 -> /BUCK_9/BUCK_VIN
- TP14 pad 1: /BUCK_1/Vin- -> Net-(TP14-Pad1)
- TP21 pad 1: /BUCK_2/Vin- -> Net-(TP21-Pad1)
- TP28 pad 1: /BUCK_4/Vin- -> Net-(TP28-Pad1)
- TP35 pad 1: /BUCK_3/Vin- -> Net-(TP35-Pad1)
- TP42 pad 1: /BUCK_5/Vin- -> Net-(TP42-Pad1)
- TP49 pad 1: /BUCK_6/Vin- -> Net-(TP49-Pad1)
- TP56 pad 1: /BUCK_7/Vin- -> Net-(TP56-Pad1)
- TP63 pad 1: /BUCK_8/Vin- -> Net-(TP63-Pad1)
- TP7 pad 1: /BUCK_0/Vin- -> Net-(TP7-Pad1)
- TP70 pad 1: /BUCK_9/Vin- -> Net-(TP70-Pad1)
- U10 pad A1: /PV_POS_1 -> /BUCK_1/BUCK_VIN
- U10 pad A2: /PV_POS_1 -> /BUCK_1/BUCK_VIN
- U10 pad A3: /PV_POS_1 -> /BUCK_1/BUCK_VIN
- U10 pad A4: /PV_POS_1 -> /BUCK_1/BUCK_VIN
- U10 pad A5: /PV_POS_1 -> /BUCK_1/BUCK_VIN
- U10 pad A6: /PV_POS_1 -> /BUCK_1/BUCK_VIN
- U10 pad B1: /PV_POS_1 -> /BUCK_1/BUCK_VIN
- U10 pad B2: /PV_POS_1 -> /BUCK_1/BUCK_VIN
- U10 pad B3: /PV_POS_1 -> /BUCK_1/BUCK_VIN
- U10 pad B4: /PV_POS_1 -> /BUCK_1/BUCK_VIN
- U10 pad B5: /PV_POS_1 -> /BUCK_1/BUCK_VIN
- U10 pad B6: /PV_POS_1 -> /BUCK_1/BUCK_VIN
- U10 pad C1: /PV_POS_1 -> /BUCK_1/BUCK_VIN
- U10 pad C2: /PV_POS_1 -> /BUCK_1/BUCK_VIN
- U10 pad C3: /PV_POS_1 -> /BUCK_1/BUCK_VIN
- U10 pad C4: /PV_POS_1 -> /BUCK_1/BUCK_VIN
- U10 pad C5: /PV_POS_1 -> /BUCK_1/BUCK_VIN
- U10 pad C6: /PV_POS_1 -> /BUCK_1/BUCK_VIN
- U12 pad 5: /BUCK_2/Vin- -> Net-(TP21-Pad1)
- U13 pad 8: /BUCK_2/Vin- -> Net-(TP21-Pad1)
- U14 pad A1: /PV_POS_2 -> /BUCK_2/BUCK_VIN
- U14 pad A2: /PV_POS_2 -> /BUCK_2/BUCK_VIN
- U14 pad A3: /PV_POS_2 -> /BUCK_2/BUCK_VIN
- U14 pad A4: /PV_POS_2 -> /BUCK_2/BUCK_VIN
- U14 pad A5: /PV_POS_2 -> /BUCK_2/BUCK_VIN
- U14 pad A6: /PV_POS_2 -> /BUCK_2/BUCK_VIN
- U14 pad B1: /PV_POS_2 -> /BUCK_2/BUCK_VIN
- U14 pad B2: /PV_POS_2 -> /BUCK_2/BUCK_VIN
- U14 pad B3: /PV_POS_2 -> /BUCK_2/BUCK_VIN
- U14 pad B4: /PV_POS_2 -> /BUCK_2/BUCK_VIN
- U14 pad B5: /PV_POS_2 -> /BUCK_2/BUCK_VIN
- U14 pad B6: /PV_POS_2 -> /BUCK_2/BUCK_VIN
- U14 pad C1: /PV_POS_2 -> /BUCK_2/BUCK_VIN
- U14 pad C2: /PV_POS_2 -> /BUCK_2/BUCK_VIN
- U14 pad C3: /PV_POS_2 -> /BUCK_2/BUCK_VIN
- U14 pad C4: /PV_POS_2 -> /BUCK_2/BUCK_VIN
- U14 pad C5: /PV_POS_2 -> /BUCK_2/BUCK_VIN
- U14 pad C6: /PV_POS_2 -> /BUCK_2/BUCK_VIN
- U16 pad 5: /BUCK_4/Vin- -> Net-(TP28-Pad1)
- U17 pad 8: /BUCK_4/Vin- -> Net-(TP28-Pad1)
- U18 pad A1: /PV_POS_4 -> /BUCK_4/BUCK_VIN
- U18 pad A2: /PV_POS_4 -> /BUCK_4/BUCK_VIN
- U18 pad A3: /PV_POS_4 -> /BUCK_4/BUCK_VIN
- U18 pad A4: /PV_POS_4 -> /BUCK_4/BUCK_VIN
- U18 pad A5: /PV_POS_4 -> /BUCK_4/BUCK_VIN
- U18 pad A6: /PV_POS_4 -> /BUCK_4/BUCK_VIN
- U18 pad B1: /PV_POS_4 -> /BUCK_4/BUCK_VIN
- U18 pad B2: /PV_POS_4 -> /BUCK_4/BUCK_VIN
- U18 pad B3: /PV_POS_4 -> /BUCK_4/BUCK_VIN
- U18 pad B4: /PV_POS_4 -> /BUCK_4/BUCK_VIN
- U18 pad B5: /PV_POS_4 -> /BUCK_4/BUCK_VIN
- U18 pad B6: /PV_POS_4 -> /BUCK_4/BUCK_VIN
- U18 pad C1: /PV_POS_4 -> /BUCK_4/BUCK_VIN
- U18 pad C2: /PV_POS_4 -> /BUCK_4/BUCK_VIN
- U18 pad C3: /PV_POS_4 -> /BUCK_4/BUCK_VIN
- U18 pad C4: /PV_POS_4 -> /BUCK_4/BUCK_VIN
- U18 pad C5: /PV_POS_4 -> /BUCK_4/BUCK_VIN
- U18 pad C6: /PV_POS_4 -> /BUCK_4/BUCK_VIN
- U20 pad 5: /BUCK_3/Vin- -> Net-(TP35-Pad1)
- U21 pad 8: /BUCK_3/Vin- -> Net-(TP35-Pad1)
- U22 pad A1: /PV_POS_3 -> /BUCK_3/BUCK_VIN
- U22 pad A2: /PV_POS_3 -> /BUCK_3/BUCK_VIN
- U22 pad A3: /PV_POS_3 -> /BUCK_3/BUCK_VIN
- U22 pad A4: /PV_POS_3 -> /BUCK_3/BUCK_VIN
- U22 pad A5: /PV_POS_3 -> /BUCK_3/BUCK_VIN
- U22 pad A6: /PV_POS_3 -> /BUCK_3/BUCK_VIN
- U22 pad B1: /PV_POS_3 -> /BUCK_3/BUCK_VIN
- U22 pad B2: /PV_POS_3 -> /BUCK_3/BUCK_VIN
- U22 pad B3: /PV_POS_3 -> /BUCK_3/BUCK_VIN
- U22 pad B4: /PV_POS_3 -> /BUCK_3/BUCK_VIN
- U22 pad B5: /PV_POS_3 -> /BUCK_3/BUCK_VIN
- U22 pad B6: /PV_POS_3 -> /BUCK_3/BUCK_VIN
- U22 pad C1: /PV_POS_3 -> /BUCK_3/BUCK_VIN
- U22 pad C2: /PV_POS_3 -> /BUCK_3/BUCK_VIN
- U22 pad C3: /PV_POS_3 -> /BUCK_3/BUCK_VIN
- U22 pad C4: /PV_POS_3 -> /BUCK_3/BUCK_VIN
- U22 pad C5: /PV_POS_3 -> /BUCK_3/BUCK_VIN
- U22 pad C6: /PV_POS_3 -> /BUCK_3/BUCK_VIN
- U24 pad 5: /BUCK_5/Vin- -> Net-(TP42-Pad1)
- U25 pad 8: /BUCK_5/Vin- -> Net-(TP42-Pad1)
- U26 pad A1: /PV_POS_5 -> /BUCK_5/BUCK_VIN
- U26 pad A2: /PV_POS_5 -> /BUCK_5/BUCK_VIN
- U26 pad A3: /PV_POS_5 -> /BUCK_5/BUCK_VIN
- U26 pad A4: /PV_POS_5 -> /BUCK_5/BUCK_VIN
- U26 pad A5: /PV_POS_5 -> /BUCK_5/BUCK_VIN
- U26 pad A6: /PV_POS_5 -> /BUCK_5/BUCK_VIN
- U26 pad B1: /PV_POS_5 -> /BUCK_5/BUCK_VIN
- U26 pad B2: /PV_POS_5 -> /BUCK_5/BUCK_VIN
- U26 pad B3: /PV_POS_5 -> /BUCK_5/BUCK_VIN
- U26 pad B4: /PV_POS_5 -> /BUCK_5/BUCK_VIN
- U26 pad B5: /PV_POS_5 -> /BUCK_5/BUCK_VIN
- U26 pad B6: /PV_POS_5 -> /BUCK_5/BUCK_VIN
- U26 pad C1: /PV_POS_5 -> /BUCK_5/BUCK_VIN
- U26 pad C2: /PV_POS_5 -> /BUCK_5/BUCK_VIN
- U26 pad C3: /PV_POS_5 -> /BUCK_5/BUCK_VIN
- U26 pad C4: /PV_POS_5 -> /BUCK_5/BUCK_VIN
- U26 pad C5: /PV_POS_5 -> /BUCK_5/BUCK_VIN
- U26 pad C6: /PV_POS_5 -> /BUCK_5/BUCK_VIN
- U28 pad 5: /BUCK_6/Vin- -> Net-(TP49-Pad1)
- U29 pad 8: /BUCK_6/Vin- -> Net-(TP49-Pad1)
- U30 pad A1: /PV_POS_6 -> /BUCK_6/BUCK_VIN
- U30 pad A2: /PV_POS_6 -> /BUCK_6/BUCK_VIN
- U30 pad A3: /PV_POS_6 -> /BUCK_6/BUCK_VIN
- U30 pad A4: /PV_POS_6 -> /BUCK_6/BUCK_VIN
- U30 pad A5: /PV_POS_6 -> /BUCK_6/BUCK_VIN
- U30 pad A6: /PV_POS_6 -> /BUCK_6/BUCK_VIN
- U30 pad B1: /PV_POS_6 -> /BUCK_6/BUCK_VIN
- U30 pad B2: /PV_POS_6 -> /BUCK_6/BUCK_VIN
- U30 pad B3: /PV_POS_6 -> /BUCK_6/BUCK_VIN
- U30 pad B4: /PV_POS_6 -> /BUCK_6/BUCK_VIN
- U30 pad B5: /PV_POS_6 -> /BUCK_6/BUCK_VIN
- U30 pad B6: /PV_POS_6 -> /BUCK_6/BUCK_VIN
- U30 pad C1: /PV_POS_6 -> /BUCK_6/BUCK_VIN
- U30 pad C2: /PV_POS_6 -> /BUCK_6/BUCK_VIN
- U30 pad C3: /PV_POS_6 -> /BUCK_6/BUCK_VIN
- U30 pad C4: /PV_POS_6 -> /BUCK_6/BUCK_VIN
- U30 pad C5: /PV_POS_6 -> /BUCK_6/BUCK_VIN
- U30 pad C6: /PV_POS_6 -> /BUCK_6/BUCK_VIN
- U32 pad 5: /BUCK_7/Vin- -> Net-(TP56-Pad1)
- U33 pad 8: /BUCK_7/Vin- -> Net-(TP56-Pad1)
- U34 pad A1: /PV_POS_7 -> /BUCK_7/BUCK_VIN
- U34 pad A2: /PV_POS_7 -> /BUCK_7/BUCK_VIN
- U34 pad A3: /PV_POS_7 -> /BUCK_7/BUCK_VIN
- U34 pad A4: /PV_POS_7 -> /BUCK_7/BUCK_VIN
- U34 pad A5: /PV_POS_7 -> /BUCK_7/BUCK_VIN
- U34 pad A6: /PV_POS_7 -> /BUCK_7/BUCK_VIN
- U34 pad B1: /PV_POS_7 -> /BUCK_7/BUCK_VIN
- U34 pad B2: /PV_POS_7 -> /BUCK_7/BUCK_VIN
- U34 pad B3: /PV_POS_7 -> /BUCK_7/BUCK_VIN
- U34 pad B4: /PV_POS_7 -> /BUCK_7/BUCK_VIN
- U34 pad B5: /PV_POS_7 -> /BUCK_7/BUCK_VIN
- U34 pad B6: /PV_POS_7 -> /BUCK_7/BUCK_VIN
- U34 pad C1: /PV_POS_7 -> /BUCK_7/BUCK_VIN
- U34 pad C2: /PV_POS_7 -> /BUCK_7/BUCK_VIN
- U34 pad C3: /PV_POS_7 -> /BUCK_7/BUCK_VIN
- U34 pad C4: /PV_POS_7 -> /BUCK_7/BUCK_VIN
- U34 pad C5: /PV_POS_7 -> /BUCK_7/BUCK_VIN
- U34 pad C6: /PV_POS_7 -> /BUCK_7/BUCK_VIN
- U36 pad 5: /BUCK_8/Vin- -> Net-(TP63-Pad1)
- U37 pad 8: /BUCK_8/Vin- -> Net-(TP63-Pad1)
- U38 pad A1: /PV_POS_8 -> /BUCK_8/BUCK_VIN
- U38 pad A2: /PV_POS_8 -> /BUCK_8/BUCK_VIN
- U38 pad A3: /PV_POS_8 -> /BUCK_8/BUCK_VIN
- U38 pad A4: /PV_POS_8 -> /BUCK_8/BUCK_VIN
- U38 pad A5: /PV_POS_8 -> /BUCK_8/BUCK_VIN
- U38 pad A6: /PV_POS_8 -> /BUCK_8/BUCK_VIN
- U38 pad B1: /PV_POS_8 -> /BUCK_8/BUCK_VIN
- U38 pad B2: /PV_POS_8 -> /BUCK_8/BUCK_VIN
- U38 pad B3: /PV_POS_8 -> /BUCK_8/BUCK_VIN
- U38 pad B4: /PV_POS_8 -> /BUCK_8/BUCK_VIN
- U38 pad B5: /PV_POS_8 -> /BUCK_8/BUCK_VIN
- U38 pad B6: /PV_POS_8 -> /BUCK_8/BUCK_VIN
- U38 pad C1: /PV_POS_8 -> /BUCK_8/BUCK_VIN
- U38 pad C2: /PV_POS_8 -> /BUCK_8/BUCK_VIN
- U38 pad C3: /PV_POS_8 -> /BUCK_8/BUCK_VIN
- U38 pad C4: /PV_POS_8 -> /BUCK_8/BUCK_VIN
- U38 pad C5: /PV_POS_8 -> /BUCK_8/BUCK_VIN
- U38 pad C6: /PV_POS_8 -> /BUCK_8/BUCK_VIN
- U4 pad 5: /BUCK_0/Vin- -> Net-(TP7-Pad1)
- U40 pad 5: /BUCK_9/Vin- -> Net-(TP70-Pad1)
- U41 pad 8: /BUCK_9/Vin- -> Net-(TP70-Pad1)
- U42 pad A1: /PV_POS_9 -> /BUCK_9/BUCK_VIN
- U42 pad A2: /PV_POS_9 -> /BUCK_9/BUCK_VIN
- U42 pad A3: /PV_POS_9 -> /BUCK_9/BUCK_VIN
- U42 pad A4: /PV_POS_9 -> /BUCK_9/BUCK_VIN
- U42 pad A5: /PV_POS_9 -> /BUCK_9/BUCK_VIN
- U42 pad A6: /PV_POS_9 -> /BUCK_9/BUCK_VIN
- U42 pad B1: /PV_POS_9 -> /BUCK_9/BUCK_VIN
- U42 pad B2: /PV_POS_9 -> /BUCK_9/BUCK_VIN
- U42 pad B3: /PV_POS_9 -> /BUCK_9/BUCK_VIN
- U42 pad B4: /PV_POS_9 -> /BUCK_9/BUCK_VIN
- U42 pad B5: /PV_POS_9 -> /BUCK_9/BUCK_VIN
- U42 pad B6: /PV_POS_9 -> /BUCK_9/BUCK_VIN
- U42 pad C1: /PV_POS_9 -> /BUCK_9/BUCK_VIN
- U42 pad C2: /PV_POS_9 -> /BUCK_9/BUCK_VIN
- U42 pad C3: /PV_POS_9 -> /BUCK_9/BUCK_VIN
- U42 pad C4: /PV_POS_9 -> /BUCK_9/BUCK_VIN
- U42 pad C5: /PV_POS_9 -> /BUCK_9/BUCK_VIN
- U42 pad C6: /PV_POS_9 -> /BUCK_9/BUCK_VIN
- U5 pad 8: /BUCK_0/Vin- -> Net-(TP7-Pad1)
- U6 pad A1: /PV_POS_0 -> /BUCK_0/BUCK_VIN
- U6 pad A2: /PV_POS_0 -> /BUCK_0/BUCK_VIN
- U6 pad A3: /PV_POS_0 -> /BUCK_0/BUCK_VIN
- U6 pad A4: /PV_POS_0 -> /BUCK_0/BUCK_VIN
- U6 pad A5: /PV_POS_0 -> /BUCK_0/BUCK_VIN
- U6 pad A6: /PV_POS_0 -> /BUCK_0/BUCK_VIN
- U6 pad B1: /PV_POS_0 -> /BUCK_0/BUCK_VIN
- U6 pad B2: /PV_POS_0 -> /BUCK_0/BUCK_VIN
- U6 pad B3: /PV_POS_0 -> /BUCK_0/BUCK_VIN
- U6 pad B4: /PV_POS_0 -> /BUCK_0/BUCK_VIN
- U6 pad B5: /PV_POS_0 -> /BUCK_0/BUCK_VIN
- U6 pad B6: /PV_POS_0 -> /BUCK_0/BUCK_VIN
- U6 pad C1: /PV_POS_0 -> /BUCK_0/BUCK_VIN
- U6 pad C2: /PV_POS_0 -> /BUCK_0/BUCK_VIN
- U6 pad C3: /PV_POS_0 -> /BUCK_0/BUCK_VIN
- U6 pad C4: /PV_POS_0 -> /BUCK_0/BUCK_VIN
- U6 pad C5: /PV_POS_0 -> /BUCK_0/BUCK_VIN
- U6 pad C6: /PV_POS_0 -> /BUCK_0/BUCK_VIN
- U8 pad 5: /BUCK_1/Vin- -> Net-(TP14-Pad1)
- U9 pad 8: /BUCK_1/Vin- -> Net-(TP14-Pad1)
Routing:
- net /NEG_0: track 0.00 -> 17.7 mm
- net /PV_POS_0: track 0.00 -> 10.3 mm
- net /BUCK_0/Vin+: track 0.00 -> 8.33 mm, vias 0 -> 2
- net /BUCK_0/Vin-: track 0.00 -> 8.19 mm
- net /BUCK_0/BUCK_VIN: track 0.00 -> 7.82 mm

Commit message: Completed first buck converter section PCB layout
Parts:
- moved C19 322.2 mm to (95.2, 26.7), turned to 90 degrees
- moved R21 79.2 mm to (82.4, 34.5)
- moved C21 77.5 mm to (88.8, 26.4), turned to 90 degrees
- moved TP7 75.0 mm to (96.9, 30.6), turned to 90 degrees
- moved C20 75.0 mm to (88.8, 23.5), turned to -90 degrees
- moved R20 61.1 mm to (81.5, 37.2), turned to 90 degrees
- moved U4 60.2 mm to (86.3, 30.5), turned to 180 degrees
- moved R22 57.7 mm to (125.3, 33.8)
- moved TP6 55.6 mm to (120.5, 34.7), turned to 90 degrees
- moved J1 52.6 mm to (74.4, 40.0), turned to -90 degrees
- moved C26 47.1 mm to (106.3, 47.1), turned to 90 degrees
- moved C25 45.7 mm to (108.7, 47.0), turned to 90 degrees
- moved U5 45.6 mm to (92.7, 26.7), turned to -90 degrees
- moved C24 45.2 mm to (111.1, 47.0), turned to 90 degrees
- moved TP10 45.0 mm to (133.0, 34.2), turned to 90 degrees
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Routing:
- net /NEG_0: track 17.7 -> 0.00 mm
- net /PV_POS_0: track 10.3 -> 0.00 mm
- net /BUCK_0/Vin+: track 8.33 -> 0.00 mm, vias 2 -> 0
- net /BUCK_0/Vin-: track 8.19 -> 0.00 mm
- net /BUCK_0/BUCK_VIN: track 7.82 -> 0.00 mm

Commit message: Partial wiring of first buck converter section PCB layout
Parts:
- added TP13: TestPoint, TestPoint:TestPoint_Pad_D2.0mm, F.Cu at (130.9, 242.3)
- added TP20: TestPoint, TestPoint:TestPoint_Pad_D2.0mm, F.Cu at (141.6, 249.7)
- added TP27: TestPoint, TestPoint:TestPoint_Pad_D2.0mm, F.Cu at (152.4, 249.7)
- added TP34: TestPoint, TestPoint:TestPoint_Pad_D2.0mm, F.Cu at (130.9, 257.0)
- added TP41: TestPoint, TestPoint:TestPoint_Pad_D2.0mm, F.Cu at (152.4, 257.0)
- added TP48: TestPoint, TestPoint:TestPoint_Pad_D2.0mm, F.Cu at (141.6, 242.3)
- added TP55: TestPoint, TestPoint:TestPoint_Pad_D2.0mm, F.Cu at (130.9, 249.7)
- added TP62: TestPoint, TestPoint:TestPoint_Pad_D2.0mm, F.Cu at (141.6, 257.0)
- added TP69: TestPoint, TestPoint:TestPoint_Pad_D2.0mm, F.Cu at (152.4, 242.3)
- moved TP7 23.6 mm to (74.4, 23.4)
- moved TP11 3.62 mm to (124.4, 54.1)
- moved TP12 3.62 mm to (128.5, 54.1)
- moved TP8 3.43 mm to (132.6, 54.1)
- moved C14 2.29 mm to (99.4, 43.4)
- moved R17 1.52 mm to (92.6, 39.9)
- moved U4 0.72 mm to (85.8, 31.0)
- moved C19 0.72 mm to (94.7, 27.2)
- moved C20 0.72 mm to (88.3, 24.0)
- moved C21 0.72 mm to (88.3, 26.9)
- moved U5 0.72 mm to (92.2, 27.2)
- moved R20 0.36 mm to (81.5, 37.6)
- moved C18 0.13 mm to (92.7, 32.4)
- moved R18 0.13 mm to (91.7, 35.1)
- moved R19 0.13 mm to (93.7, 35.1)
Connections:
- TP6 pad 1: Net-(TP6-Pad1) -> Net-(U6-PadA7)
- U10 pad A7: Net-(TP13-Pad1) -> Net-(U10-PadA7)
- U10 pad D9: Net-(TP13-Pad1) -> unconnected-(U10-PadD9)
- U14 pad A7: Net-(TP20-Pad1) -> Net-(U14-PadA7)
- U14 pad D9: Net-(TP20-Pad1) -> unconnected-(U14-PadD9)
- U18 pad A7: Net-(TP27-Pad1) -> Net-(U18-PadA7)
- U18 pad D9: Net-(TP27-Pad1) -> unconnected-(U18-PadD9)
- U22 pad A7: Net-(TP34-Pad1) -> Net-(U22-PadA7)
- U22 pad D9: Net-(TP34-Pad1) -> unconnected-(U22-PadD9)
- U26 pad A7: Net-(TP41-Pad1) -> Net-(U26-PadA7)
- U26 pad D9: Net-(TP41-Pad1) -> unconnected-(U26-PadD9)
- U30 pad A7: Net-(TP48-Pad1) -> Net-(U30-PadA7)
- U30 pad D9: Net-(TP48-Pad1) -> unconnected-(U30-PadD9)
- U34 pad A7: Net-(TP55-Pad1) -> Net-(U34-PadA7)
- U34 pad D9: Net-(TP55-Pad1) -> unconnected-(U34-PadD9)
- U38 pad A7: Net-(TP62-Pad1) -> Net-(U38-PadA7)
- U38 pad D9: Net-(TP62-Pad1) -> unconnected-(U38-PadD9)
- U42 pad A7: Net-(TP69-Pad1) -> Net-(U42-PadA7)
- U42 pad D9: Net-(TP69-Pad1) -> unconnected-(U42-PadD9)
- U6 pad A7: Net-(TP6-Pad1) -> Net-(U6-PadA7)
- U6 pad D9: Net-(TP6-Pad1) -> unconnected-(U6-PadD9)
Routing:
- net Net-(TP7-Pad1): track 0.00 -> 21.7 mm
- net Net-(TP11-Pad1): track 0.00 -> 17.9 mm
- net Net-(TP8-Pad1): track 0.00 -> 12.2 mm
- net /BUCK_0/BUCK_VIN: track 0.00 -> 9.41 mm
- net /BUCK_0/+IN: track 0.00 -> 8.11 mm
- net +5V: track 0.00 -> 7.45 mm
- net /NEG_0: track 0.00 -> 6.93 mm
- net Net-(TP10-Pad1): track 0.00 -> 6.66 mm
- net /BUCK_0/Vin+: track 0.00 -> 5.89 mm, vias 0 -> 2
- net /BUCK_0/Vin-: track 0.00 -> 5.30 mm
- net Net-(U6-PadA7): track 0.00 -> 5.20 mm, vias 0 -> 2
- net /PV_POS_0: track 0.00 -> 4.60 mm
- net /BUCK_0/RUN: track 0.00 -> 3.91 mm
- net Net-(TP9-Pad1): track 0.00 -> 3.77 mm
- net /BUCK_0/Vfb: track 0.00 -> 3.35 mm
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- added copper zone on F.Cu, net /BUCK_0/BUCK_VIN
- added copper zone on F.Cu, net /NEG_0
- added copper zone on F.Cu, net /NEG_1
- added copper zone on F.Cu, net /PV_POS_0

Commit message: Added second buck converter section PCB layout
Parts:
- removed the TP13 at (130.9, 242.3)
- removed the TP20 at (141.6, 249.7)
- removed the TP27 at (152.4, 249.7)
- removed the TP34 at (130.9, 257.0)
- removed the TP41 at (152.4, 257.0)
- removed the TP48 at (141.6, 242.3)
- removed the TP55 at (130.9, 249.7)
- removed the TP62 at (141.6, 257.0)
- removed the TP69 at (152.4, 242.3)
- moved C33 279.1 mm to (93.9, 65.7), turned to 90 degrees
- moved J2 169.1 mm to (74.3, 78.5), turned to -90 degrees
- moved TP14 167.1 mm to (73.3, 61.4)
- moved R25 165.1 mm to (90.9, 74.6), turned to 90 degrees
- moved C35 162.9 mm to (87.2, 63.8), turned to -90 degrees
- moved R28 162.8 mm to (82.8, 73.2)
- moved R27 162.7 mm to (81.8, 76.3), turned to 90 degrees
- moved R24 152.7 mm to (92.1, 78.5)
- moved TP19 148.1 mm to (119.4, 96.8)
- moved C34 147.8 mm to (92.0, 72.0)
- moved U8 147.3 mm to (84.7, 69.0), turned to 180 degrees
- moved C30 146.6 mm to (112.3, 82.3), turned to -90 degrees
- moved C31 144.6 mm to (109.8, 82.3), turned to -90 degrees
- moved R26 143.7 mm to (93.1, 74.6), turned to 90 degrees
- moved C41 143.5 mm to (104.6, 88.7), turned to 90 degrees
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Connections:
- TP6 pad 1: Net-(U6-PadA7) -> Net-(TP6-Pad1)
- U10 pad A7: Net-(U10-PadA7) -> Net-(TP13-Pad1)
- U10 pad D9: unconnected-(U10-PadD9) -> Net-(TP13-Pad1)
- U14 pad A7: Net-(U14-PadA7) -> Net-(TP20-Pad1)
- U14 pad D9: unconnected-(U14-PadD9) -> Net-(TP20-Pad1)
- U18 pad A7: Net-(U18-PadA7) -> Net-(TP27-Pad1)
- U18 pad D9: unconnected-(U18-PadD9) -> Net-(TP27-Pad1)
- U22 pad A7: Net-(U22-PadA7) -> Net-(TP34-Pad1)
- U22 pad D9: unconnected-(U22-PadD9) -> Net-(TP34-Pad1)
- U26 pad A7: Net-(U26-PadA7) -> Net-(TP41-Pad1)
- U26 pad D9: unconnected-(U26-PadD9) -> Net-(TP41-Pad1)
- U30 pad A7: Net-(U30-PadA7) -> Net-(TP48-Pad1)
- U30 pad D9: unconnected-(U30-PadD9) -> Net-(TP48-Pad1)
- U34 pad A7: Net-(U34-PadA7) -> Net-(TP55-Pad1)
- U34 pad D9: unconnected-(U34-PadD9) -> Net-(TP55-Pad1)
- U38 pad A7: Net-(U38-PadA7) -> Net-(TP62-Pad1)
- U38 pad D9: unconnected-(U38-PadD9) -> Net-(TP62-Pad1)
- U42 pad A7: Net-(U42-PadA7) -> Net-(TP69-Pad1)
- U42 pad D9: unconnected-(U42-PadD9) -> Net-(TP69-Pad1)
- U6 pad A7: Net-(U6-PadA7) -> Net-(TP6-Pad1)
- U6 pad D9: unconnected-(U6-PadD9) -> Net-(TP6-Pad1)
Routing:
- net GND: track 1.37 -> 192.2 mm, vias 0 -> 6
- net +5V: track 7.45 -> 192.9 mm
- net Net-(TP14-Pad1): track 0.00 -> 29.2 mm, vias 0 -> 1
- net Net-(TP18-Pad1): track 0.00 -> 27.2 mm, vias 0 -> 4
- net /NEG_1: track 0.00 -> 26.5 mm, vias 0 -> 2
- net /NEG_0: track 6.93 -> 23.6 mm, vias 0 -> 2
- net Net-(TP15-Pad1): track 0.00 -> 15.2 mm, vias 0 -> 2
- net Net-(TP11-Pad1): track 17.9 -> 30.3 mm, vias 0 -> 4
- net /BUCK_1/+IN: track 0.00 -> 8.65 mm
- net /BUCK_1/BUCK_VIN: track 0.00 -> 8.50 mm
- net Net-(TP7-Pad1): track 21.7 -> 28.7 mm, vias 0 -> 1
- net Net-(TP10-Pad1): track 6.66 -> 0.00 mm
- net /BUCK_1/Vin-: track 0.00 -> 6.38 mm, vias 0 -> 2
- net /BUCK_1/Vin+: track 0.00 -> 6.25 mm
- net Net-(TP13-Pad1): track 0.00 -> 5.50 mm, vias 0 -> 2
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- added copper zone on F.Cu, net /BUCK_1/BUCK_VIN
- added copper zone on F.Cu, net /PV_POS_1

Commit message: Added 3rd buck converter section
Parts:
- added JP1: SolderJumper_2_Bridged, Jumper:SolderJumper-2_P1.3mm_Bridged_RoundedPad1.0x1.5mm, F.Cu at (130.9, 61.3)
- added JP10: SolderJumper_2_Bridged, Jumper:SolderJumper-2_P1.3mm_Bridged_RoundedPad1.0x1.5mm, F.Cu at (167.1, 343.2)
- added JP2: SolderJumper_2_Bridged, Jumper:SolderJumper-2_P1.3mm_Bridged_RoundedPad1.0x1.5mm, F.Cu at (130.6, 102.6)
- added JP3: SolderJumper_2_Bridged, Jumper:SolderJumper-2_P1.3mm_Bridged_RoundedPad1.0x1.5mm, F.Cu at (130.6, 144.4)
- added JP4: SolderJumper_2_Bridged, Jumper:SolderJumper-2_P1.3mm_Bridged_RoundedPad1.0x1.5mm, F.Cu at (167.1, 351.3)
- added JP5: SolderJumper_2_Bridged, Jumper:SolderJumper-2_P1.3mm_Bridged_RoundedPad1.0x1.5mm, F.Cu at (143.1, 359.4)
- added JP6: SolderJumper_2_Bridged, Jumper:SolderJumper-2_P1.3mm_Bridged_RoundedPad1.0x1.5mm, F.Cu at (179.2, 343.2)
- added JP7: SolderJumper_2_Bridged, Jumper:SolderJumper-2_P1.3mm_Bridged_RoundedPad1.0x1.5mm, F.Cu at (155.1, 343.2)
- added JP8: SolderJumper_2_Bridged, Jumper:SolderJumper-2_P1.3mm_Bridged_RoundedPad1.0x1.5mm, F.Cu at (143.1, 351.3)
- added JP9: SolderJumper_2_Bridged, Jumper:SolderJumper-2_P1.3mm_Bridged_RoundedPad1.0x1.5mm, F.Cu at (155.1, 359.4)
- added TP27: TestPoint, TestPoint:TestPoint_Pad_D2.0mm, F.Cu at (171.3, 351.6)
- added TP34: TestPoint, TestPoint:TestPoint_Pad_D2.0mm, F.Cu at (147.3, 359.6)
- added TP41: TestPoint, TestPoint:TestPoint_Pad_D2.0mm, F.Cu at (183.4, 343.5)
- added TP48: TestPoint, TestPoint:TestPoint_Pad_D2.0mm, F.Cu at (159.3, 343.5)
- added TP55: TestPoint, TestPoint:TestPoint_Pad_D2.0mm, F.Cu at (147.3, 351.6)
- added TP62: TestPoint, TestPoint:TestPoint_Pad_D2.0mm, F.Cu at (159.3, 359.6)
- added TP69: TestPoint, TestPoint:TestPoint_Pad_D2.0mm, F.Cu at (171.3, 343.5)
- moved TP21 265.3 mm to (73.8, 103.1)
- moved C48 247.3 mm to (92.0, 113.3)
- moved U13 246.8 mm to (91.2, 107.3), turned to -90 degrees
- moved R35 244.4 mm to (83.0, 115.1)
- moved R33 244.2 mm to (93.1, 116.0), turned to 90 degrees
- moved R32 242.0 mm to (90.9, 116.0), turned to 90 degrees
- moved C50 240.0 mm to (87.2, 105.5), turned to -90 degrees
- moved C51 240.0 mm to (87.2, 108.6), turned to 90 degrees
- moved R36 237.8 mm to (123.8, 117.5)
- moved C49 235.4 mm to (93.9, 107.2), turned to 90 degrees
- moved R34 235.1 mm to (82.1, 117.9), turned to 90 degrees
- moved TP20 234.6 mm to (118.8, 118.2)
- moved TP24 232.3 mm to (130.7, 117.5)
- moved TP23 231.6 mm to (130.8, 122.3)
- moved C45 231.1 mm to (108.0, 124.1), turned to -90 degrees
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Connections:
- TP11 pad 1: Net-(TP11-Pad1) -> Net-(U6-PadL12)
- TP12 pad 1: Net-(TP11-Pad1) -> Net-(U6-PadK12)
- TP18 pad 1: Net-(TP18-Pad1) -> Net-(U10-PadL12)
- TP19 pad 1: Net-(TP18-Pad1) -> Net-(TP19-Pad1)
- TP25 pad 1: Net-(TP25-Pad1) -> Net-(U14-PadL12)
- TP26 pad 1: Net-(TP25-Pad1) -> Net-(U14-PadK12)
- TP32 pad 1: Net-(TP32-Pad1) -> Net-(U18-PadL12)
- TP33 pad 1: Net-(TP32-Pad1) -> Net-(TP33-Pad1)
- TP39 pad 1: Net-(TP39-Pad1) -> Net-(U22-PadL12)
- TP40 pad 1: Net-(TP39-Pad1) -> Net-(U22-PadK12)
- TP46 pad 1: Net-(TP46-Pad1) -> Net-(U26-PadL12)
- TP47 pad 1: Net-(TP46-Pad1) -> Net-(U26-PadK12)
- TP53 pad 1: Net-(TP53-Pad1) -> Net-(U30-PadL12)
- TP54 pad 1: Net-(TP53-Pad1) -> Net-(U30-PadK12)
- TP61 pad 1: Net-(TP60-Pad1) -> Net-(TP61-Pad1)
- TP67 pad 1: Net-(TP67-Pad1) -> Net-(U38-PadL12)
- TP68 pad 1: Net-(TP67-Pad1) -> Net-(U38-PadK12)
- TP74 pad 1: Net-(TP74-Pad1) -> Net-(U42-PadL12)
- TP75 pad 1: Net-(TP74-Pad1) -> Net-(U42-PadK12)
- U10 pad D9: Net-(TP13-Pad1) -> unconnected-(U10-PadD9)
- U10 pad K12: Net-(TP18-Pad1) -> Net-(TP19-Pad1)
- U10 pad L12: Net-(TP18-Pad1) -> Net-(U10-PadL12)
- U14 pad D9: Net-(TP20-Pad1) -> unconnected-(U14-PadD9)
- U14 pad K12: Net-(TP25-Pad1) -> Net-(U14-PadK12)
- U14 pad L12: Net-(TP25-Pad1) -> Net-(U14-PadL12)
- U18 pad D9: Net-(TP27-Pad1) -> unconnected-(U18-PadD9)
- U18 pad K12: Net-(TP32-Pad1) -> Net-(TP33-Pad1)
- U18 pad L12: Net-(TP32-Pad1) -> Net-(U18-PadL12)
- U22 pad D9: Net-(TP34-Pad1) -> unconnected-(U22-PadD9)
- U22 pad K12: Net-(TP39-Pad1) -> Net-(U22-PadK12)
- U22 pad L12: Net-(TP39-Pad1) -> Net-(U22-PadL12)
- U26 pad D9: Net-(TP41-Pad1) -> unconnected-(U26-PadD9)
- U26 pad K12: Net-(TP46-Pad1) -> Net-(U26-PadK12)
- U26 pad L12: Net-(TP46-Pad1) -> Net-(U26-PadL12)
- U30 pad D9: Net-(TP48-Pad1) -> unconnected-(U30-PadD9)
- U30 pad K12: Net-(TP53-Pad1) -> Net-(U30-PadK12)
- U30 pad L12: Net-(TP53-Pad1) -> Net-(U30-PadL12)
- U34 pad D9: Net-(TP55-Pad1) -> unconnected-(U34-PadD9)
- U34 pad K12: Net-(TP60-Pad1) -> Net-(TP61-Pad1)
- U38 pad D9: Net-(TP62-Pad1) -> unconnected-(U38-PadD9)
- U38 pad K12: Net-(TP67-Pad1) -> Net-(U38-PadK12)
- U38 pad L12: Net-(TP67-Pad1) -> Net-(U38-PadL12)
- U42 pad D9: Net-(TP69-Pad1) -> unconnected-(U42-PadD9)
- U42 pad K12: Net-(TP74-Pad1) -> Net-(U42-PadK12)
- U42 pad L12: Net-(TP74-Pad1) -> Net-(U42-PadL12)
- U6 pad D9: Net-(TP6-Pad1) -> unconnected-(U6-PadD9)
- U6 pad K12: Net-(TP11-Pad1) -> Net-(U6-PadK12)
- U6 pad L12: Net-(TP11-Pad1) -> Net-(U6-PadL12)
Routing:
- net +5V: track 192.9 -> 301.2 mm
- net GND: track 192.2 -> 298.5 mm, vias 6 -> 10
- net Net-(TP11-Pad1): track 30.3 -> 0.00 mm, vias 4 -> 0
- net Net-(TP21-Pad1): track 0.00 -> 27.4 mm, vias 0 -> 1
- net Net-(TP18-Pad1): track 27.2 -> 0.00 mm, vias 4 -> 0
- net /NEG_2: track 2.92 -> 26.5 mm, vias 0 -> 2
- net Net-(U6-PadL12): track 0.00 -> 18.5 mm, vias 0 -> 2
- net Net-(U10-PadL12): track 0.00 -> 18.0 mm, vias 0 -> 2
- net Net-(U14-PadL12): track 0.00 -> 15.6 mm, vias 0 -> 2
- net Net-(U6-PadK12): track 0.00 -> 14.2 mm, vias 0 -> 2
- net Net-(TP22-Pad1): track 0.00 -> 13.1 mm, vias 0 -> 2
- net Net-(TP19-Pad1): track 0.00 -> 12.9 mm, vias 0 -> 2
- net Net-(U14-PadK12): track 0.00 -> 10.1 mm, vias 0 -> 2
- net /BUCK_2/BUCK_VIN: track 0.00 -> 9.26 mm
- net /BUCK_2/+IN: track 0.00 -> 8.69 mm
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- added copper zone on F.Cu, net /BUCK_2/BUCK_VIN
- added copper zone on F.Cu, net /NEG_2
- added copper zone on F.Cu, net /PV_POS_2

Commit message: Placed 4th buck converter, started 5th.
Parts:
- removed the TP34 at (112.8, 352.4)
- U16: footprint Package_DIP:DIP-8_W8.89mm_SMDSocket_LongPads -> Package_DIP:DIP-8_W7.62mm_Socket_LongPads
- moved C79 209.1 mm to (94.1, 149.3), turned to 90 degrees
- moved C81 207.5 mm to (87.3, 151.3), turned to 90 degrees
- moved C80 204.0 mm to (87.2, 146.4), turned to -90 degrees
- moved TP35 201.8 mm to (73.7, 145.2)
- moved TP34 201.3 mm to (118.9, 160.3)
- moved R46 200.4 mm to (90.6, 158.5), turned to 90 degrees
- moved R47 197.6 mm to (93.5, 158.5), turned to 90 degrees
- moved TP37 193.1 mm to (131.2, 164.3)
- moved R50 189.7 mm to (123.9, 159.3)
- moved R48 188.6 mm to (81.6, 159.9), turned to 90 degrees
- moved C78 188.4 mm to (92.0, 155.5)
- moved C74 188.0 mm to (98.9, 166.2), turned to -90 degrees
- moved U21 187.2 mm to (91.5, 149.2), turned to -90 degrees
- moved R49 184.8 mm to (82.5, 157.4)
- moved R51 183.8 mm to (132.0, 170.3), turned to -90 degrees
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Routing:
- net GND: track 298.5 -> 457.9 mm, vias 10 -> 14
- net +5V: track 301.2 -> 453.8 mm
- net /NEG_3: track 2.97 -> 28.3 mm, vias 0 -> 2
- net Net-(TP35-Pad1): track 0.00 -> 22.0 mm, vias 0 -> 2
- net Net-(JP5-Pad2): track 0.00 -> 19.7 mm, vias 0 -> 2
- net Net-(JP4-Pad2): track 0.00 -> 17.6 mm, vias 0 -> 2
- net Net-(TP29-Pad1): track 0.00 -> 14.6 mm, vias 0 -> 2
- net Net-(JP5-Pad1): track 0.00 -> 14.6 mm, vias 0 -> 2
- net Net-(TP36-Pad1): track 0.00 -> 13.9 mm, vias 0 -> 2
- net Net-(JP4-Pad1): track 0.00 -> 12.1 mm, vias 0 -> 2
- net /NEG_4: track 0.00 -> 11.0 mm
- net /BUCK_3/BUCK_VIN: track 0.00 -> 8.95 mm
- net /BUCK_3/+IN: track 0.00 -> 8.08 mm
- net /BUCK_3/Vin-: track 0.00 -> 7.17 mm, vias 0 -> 2
- net /BUCK_3/Vin+: track 0.00 -> 6.96 mm
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- added copper zone on F.Cu, net /BUCK_3/BUCK_VIN
- added copper zone on F.Cu, net /BUCK_4/BUCK_VIN
- added copper zone on F.Cu, net /NEG_3
- added copper zone on F.Cu, net /NEG_4
- added copper zone on F.Cu, net /PV_POS_3
- added copper zone on F.Cu, net /PV_POS_4
