File: KiCAD/Quest_39/Quest_39.kicad_pcb (KiCad board)
At the start: 2 copper layers, 404 parts, among them J1 1x2 Scr. Term., J10 1x2 Scr. Term., J11 1x2 Scr. Term., J12 Conn_01x05_Male, J2 1x2 Scr. Term., J3 1x2 Scr. Term., J4 1x2 Scr. Term., J5 1x2 Scr. Term., J6 1x2 Scr. Term., J7 1x2 Scr. Term., J8 1x2 Scr. Term., J9 1x2 Scr. Term., U1 AZ1117-3.3, U10 LTM4611EV-PBF, U11 MCP4151-502E/SN, U12 AD626ANZ, U13 INA226, U14 LTM4611EV-PBF, U15 MCP4151-502E/SN, U16 AD626ANZ, U17 INA226, U18 LTM4611EV-PBF, U19 MCP4151-502E/SN, U2 17791063215, U20 AD626ANZ, U21 INA226, U22 LTM4611EV-PBF, U23 MCP4151-502E/SN, U24 AD626ANZ, U25 INA226, U26 LTM4611EV-PBF, U27 MCP4151-502E/SN, U28 AD626ANZ, U29 INA226, U3 STM32F103C8T6, U30 LTM4611EV-PBF, U31 MCP4151-502E/SN, U32 AD626ANZ, U33 INA226, U34 LTM4611EV-PBF, U35 MCP4151-502E/SN, U36 AD626ANZ, U37 INA226, U38 LTM4611EV-PBF, U39 MCP4151-502E/SN, U4 AD626ANZ, U40 AD626ANZ, U41 INA226, U42 LTM4611EV-PBF, U43 MCP4151-502E/SN, U5 INA226, U6 LTM4611EV-PBF, U7 MCP4151-502E/SN, U8 AD626ANZ, U9 INA226, Y1 16MHz

Commit message: Finished placing 5th buck converter, started 6th
Parts:
- removed the TP27 at (171.3, 351.6)
- removed the TP41 at (232.3, 334.8)
- moved TP46 331.1 mm to (189.8, 21.1)
- moved TP47 320.4 mm to (189.8, 28.1)
- moved JP6 318.8 mm to (189.8, 24.6), turned to 90 degrees
- moved TP43 316.6 mm to (189.7, 31.5)
- moved C101 310.3 mm to (215.3, 39.2), turned to -90 degrees
- moved U27 307.7 mm to (185.3, 38.7)
- moved C103 306.2 mm to (185.3, 35.9), turned to 180 degrees
- moved C99 304.4 mm to (210.5, 39.2), turned to -90 degrees
- moved C89 302.7 mm to (221.2, 46.3), turned to 90 degrees
- moved C102 302.2 mm to (189.6, 42.4), turned to -90 degrees
- moved C98 301.0 mm to (208.2, 39.2), turned to -90 degrees
- moved TP45 300.6 mm to (191.2, 53.5)
- moved R58 299.5 mm to (187.4, 42.3), turned to 90 degrees
- moved R57 297.2 mm to (196.5, 53.1), turned to 180 degrees
- moved C100 293.9 mm to (212.9, 39.2), turned to -90 degrees
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Routing:
- net +5V: track 453.8 -> 567.6 mm, vias 0 -> 4
- net GND: track 457.9 -> 567.5 mm, vias 14 -> 18
- net Net-(TP28-Pad1): track 0.00 -> 22.0 mm, vias 0 -> 2
- net /NEG_4: track 11.0 -> 31.6 mm, vias 0 -> 4
- net Net-(JP6-Pad2): track 0.00 -> 18.0 mm, vias 0 -> 2
- net /NEG_5: track 4.78 -> 19.8 mm, vias 0 -> 2
- net Net-(TP43-Pad1): track 0.00 -> 14.4 mm, vias 0 -> 2
- net Net-(JP6-Pad1): track 0.00 -> 12.1 mm, vias 0 -> 2
- net /NEG_0: track 17.5 -> 26.2 mm, vias 2 -> 4
- net /BUCK_4/BUCK_VIN: track 0.00 -> 8.24 mm
- net /BUCK_4/+IN: track 0.00 -> 8.15 mm
- net /BUCK_4/Vin-: track 0.00 -> 7.41 mm, vias 0 -> 2
- net /BUCK_4/Vin+: track 0.00 -> 7.31 mm
- net /NEG_6: track 0.00 -> 5.19 mm
- net Net-(TP45-Pad1): track 0.00 -> 4.86 mm
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- added copper zone on F.Cu, net /BUCK_5/BUCK_VIN
- added copper zone on F.Cu, net /NEG_5
- added copper zone on F.Cu, net /PV_POS_5
Other:
- board text added: "Moeten we wel de diff. amp. gebruiken?"

Commit message: Finished placing all LTM4611EV buck-converters
Parts:
- removed C138: 100nF, Capacitor_SMD:C_0603_1608Metric
- removed the TP48 at (194.5, 265.5)
- removed the TP48 at (159.3, 343.5)
- removed the TP55 at (147.3, 351.6)
- removed the TP55 at (124.5, 308.6)
- removed the TP62 at (159.3, 359.6)
- removed the TP62 at (238.6, 297.1)
- removed the TP69 at (66.8, 314.5)
- removed the TP69 at (171.3, 343.5)
- removed the U37 at (223.9, 297.4)
- added TP48: TestPoint, TestPoint:TestPoint_Pad_D2.0mm, F.Cu at (199.6, 100.0)
- added TP55: TestPoint, TestPoint:TestPoint_Pad_D2.0mm, F.Cu at (199.6, 146.2)
- added TP62: TestPoint, TestPoint:TestPoint_Pad_D2.0mm, F.Cu at (199.7, 192.5)
- added TP69: TestPoint, TestPoint:TestPoint_Pad_D2.0mm, F.Cu at (199.7, 238.5)
- added U37: 100nF, Capacitor_SMD:C_0603_1608Metric, F.Cu at (226.7, 202.9)
- added U37: INA226, Package_SO:VSSOP-10_3x3mm_P0.5mm, F.Cu at (229.4, 202.6)
- U40: footprint Package_DIP:DIP-8_W8.89mm_SMDSocket_LongPads -> Package_DIP:DIP-8_W7.62mm_Socket_LongPads
- moved C93 333.8 mm to (226.5, 64.2), turned to 90 degrees
- moved H3 326.1 mm to (252.2, 18.5)
- moved C108 290.5 mm to (226.5, 110.5), turned to 90 degrees
- moved JP7 274.6 mm to (189.9, 70.8), turned to 90 degrees
- moved C123 265.4 mm to (226.6, 156.7), turned to 90 degrees
- moved H4 260.5 mm to (68.3, 18.3)
- moved JP8 238.9 mm to (189.9, 117.0), turned to 90 degrees
- moved C119 225.2 mm to (221.3, 138.8), turned to 90 degrees
- moved C130 222.8 mm to (213.1, 131.7), turned to -90 degrees
- moved R69 220.2 mm to (238.0, 145.0), turned to -90 degrees
- moved R67 220.2 mm to (229.7, 146.2), turned to -90 degrees
- moved TP57 219.1 mm to (189.8, 124.0)
- moved TP54 216.4 mm to (189.9, 74.3)
- moved TP53 216.2 mm to (189.8, 67.3)
- moved U40 214.2 mm to (235.4, 243.7)
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Connections:
- C104 pad 1: /BUCK_6/BUCK_VIN -> /BUCK_5/BUCK_VIN
- C104 pad 2: /NEG_6 -> /NEG_5
- C105 pad 1: /BUCK_6/BUCK_VIN -> /BUCK_5/BUCK_VIN
- C105 pad 2: /NEG_6 -> /NEG_5
- C106 pad 1: /BUCK_6/BUCK_VIN -> /BUCK_5/BUCK_VIN
- C106 pad 2: /NEG_6 -> /NEG_5
- C107 pad 1: /BUCK_6/BUCK_VIN -> /BUCK_5/BUCK_VIN
- C107 pad 2: /NEG_6 -> /NEG_5
- C109 pad 1: /BUCK_6/Vin+ -> /BUCK_5/Vin+
- C109 pad 2: /BUCK_6/Vin- -> /BUCK_5/Vin-
- C110 pad 1: Net-(C110-Pad1) -> Net-(C95-Pad1)
- C112 pad 1: /NEG_6 -> /NEG_5
- C112 pad 2: /BUCK_6/TRACK/SS -> /BUCK_5/TRACK/SS
- C113 pad 1: /NEG_7 -> /NEG_6
- C113 pad 2: /NEG_6 -> /NEG_5
- C114 pad 1: /NEG_7 -> /NEG_6
- C114 pad 2: /NEG_6 -> /NEG_5
- C115 pad 1: /NEG_7 -> /NEG_6
- C115 pad 2: /NEG_6 -> /NEG_5
- C116 pad 1: /NEG_7 -> /NEG_6
- C116 pad 2: /NEG_6 -> /NEG_5
- C117 pad 1: /NEG_7 -> /NEG_6
- C117 pad 2: /BUCK_6/Vfb -> /BUCK_5/Vfb
- C119 pad 1: /BUCK_7/BUCK_VIN -> /BUCK_5/BUCK_VIN
- C119 pad 2: /NEG_7 -> /NEG_5
- C120 pad 1: /BUCK_7/BUCK_VIN -> /BUCK_5/BUCK_VIN
- C120 pad 2: /NEG_7 -> /NEG_5
- C121 pad 1: /BUCK_7/BUCK_VIN -> /BUCK_5/BUCK_VIN
- C121 pad 2: /NEG_7 -> /NEG_5
- C122 pad 1: /BUCK_7/BUCK_VIN -> /BUCK_5/BUCK_VIN
- C122 pad 2: /NEG_7 -> /NEG_5
- C124 pad 1: /BUCK_7/Vin+ -> /BUCK_5/Vin+
- C124 pad 2: /BUCK_7/Vin- -> /BUCK_5/Vin-
- C125 pad 1: Net-(C125-Pad1) -> Net-(C95-Pad1)
- C127 pad 1: /NEG_7 -> /NEG_5
- C127 pad 2: /BUCK_7/TRACK/SS -> /BUCK_5/TRACK/SS
- C128 pad 1: /NEG_8 -> /NEG_6
- C128 pad 2: /NEG_7 -> /NEG_5
- C129 pad 1: /NEG_8 -> /NEG_6
- C129 pad 2: /NEG_7 -> /NEG_5
- C130 pad 1: /NEG_8 -> /NEG_6
- C130 pad 2: /NEG_7 -> /NEG_5
- C131 pad 1: /NEG_8 -> /NEG_6
- C131 pad 2: /NEG_7 -> /NEG_5
- C132 pad 1: /NEG_8 -> /NEG_6
- C132 pad 2: /BUCK_7/Vfb -> /BUCK_5/Vfb
- C134 pad 1: /BUCK_8/BUCK_VIN -> /BUCK_5/BUCK_VIN
- C134 pad 2: /NEG_8 -> /NEG_5
- C135 pad 1: /BUCK_8/BUCK_VIN -> /BUCK_5/BUCK_VIN
- C135 pad 2: /NEG_8 -> /NEG_5
- C136 pad 1: /BUCK_8/BUCK_VIN -> /BUCK_5/BUCK_VIN
- C136 pad 2: /NEG_8 -> /NEG_5
- C137 pad 1: /BUCK_8/BUCK_VIN -> /BUCK_5/BUCK_VIN
- C137 pad 2: /NEG_8 -> /NEG_5
- C139 pad 1: /BUCK_8/Vin+ -> /BUCK_5/Vin+
- C139 pad 2: /BUCK_8/Vin- -> /BUCK_5/Vin-
- C140 pad 1: Net-(C140-Pad1) -> Net-(C95-Pad1)
- C142 pad 1: /NEG_8 -> /NEG_5
- C142 pad 2: /BUCK_8/TRACK/SS -> /BUCK_5/TRACK/SS
- C143 pad 1: /NEG_9 -> /NEG_6
- C143 pad 2: /NEG_8 -> /NEG_5
- C144 pad 1: /NEG_9 -> /NEG_6
- C144 pad 2: /NEG_8 -> /NEG_5
- C145 pad 1: /NEG_9 -> /NEG_6
- C145 pad 2: /NEG_8 -> /NEG_5
- C146 pad 1: /NEG_9 -> /NEG_6
- C146 pad 2: /NEG_8 -> /NEG_5
- C147 pad 1: /NEG_9 -> /NEG_6
- C147 pad 2: /BUCK_8/Vfb -> /BUCK_5/Vfb
- C149 pad 1: /BUCK_9/BUCK_VIN -> /BUCK_5/BUCK_VIN
- C149 pad 2: /NEG_9 -> /NEG_5
- C150 pad 1: /BUCK_9/BUCK_VIN -> /BUCK_5/BUCK_VIN
- C150 pad 2: /NEG_9 -> /NEG_5
- C151 pad 1: /BUCK_9/BUCK_VIN -> /BUCK_5/BUCK_VIN
- C151 pad 2: /NEG_9 -> /NEG_5
- C152 pad 1: /BUCK_9/BUCK_VIN -> /BUCK_5/BUCK_VIN
- C152 pad 2: /NEG_9 -> /NEG_5
- C154 pad 1: /BUCK_9/Vin+ -> /BUCK_5/Vin+
- C154 pad 2: /BUCK_9/Vin- -> /BUCK_5/Vin-
- C155 pad 1: Net-(C155-Pad1) -> Net-(C95-Pad1)
- C157 pad 1: /NEG_9 -> /NEG_5
- C157 pad 2: /BUCK_9/TRACK/SS -> /BUCK_5/TRACK/SS
- C158 pad 1: /POS_9 -> /NEG_6
- C158 pad 2: /NEG_9 -> /NEG_5
- C159 pad 1: /POS_9 -> /NEG_6
- C159 pad 2: /NEG_9 -> /NEG_5
- C160 pad 1: /POS_9 -> /NEG_6
- C160 pad 2: /NEG_9 -> /NEG_5
- C161 pad 1: /POS_9 -> /NEG_6
- C161 pad 2: /NEG_9 -> /NEG_5
- C162 pad 1: /POS_9 -> /NEG_6
- C162 pad 2: /BUCK_9/Vfb -> /BUCK_5/Vfb
- J10 pad 1: /PV_POS_8 -> /PV_POS_5
- J10 pad 2: /NEG_8 -> /NEG_5
- J11 pad 1: /PV_POS_9 -> /PV_POS_5
- J11 pad 2: /NEG_9 -> /NEG_5
- J8 pad 1: /PV_POS_6 -> /PV_POS_5
- J8 pad 2: /NEG_6 -> /NEG_5
- J9 pad 1: /PV_POS_7 -> /PV_POS_5
- J9 pad 2: /NEG_7 -> /NEG_5
- JP10 pad 1: Net-(JP10-Pad1) -> Net-(JP6-Pad1)
- JP10 pad 2: Net-(JP10-Pad2) -> Net-(JP6-Pad2)
- JP7 pad 1: Net-(JP7-Pad1) -> Net-(JP6-Pad1)
- JP7 pad 2: Net-(JP7-Pad2) -> Net-(JP6-Pad2)
- JP8 pad 1: Net-(JP8-Pad1) -> Net-(JP6-Pad1)
- JP8 pad 2: Net-(JP8-Pad2) -> Net-(JP6-Pad2)
- JP9 pad 1: Net-(JP9-Pad1) -> Net-(JP6-Pad1)
- JP9 pad 2: Net-(JP9-Pad2) -> Net-(JP6-Pad2)
- R59 pad 1: /PV_POS_6 -> /PV_POS_5
- R59 pad 2: /BUCK_6/BUCK_VIN -> /BUCK_5/BUCK_VIN
- R60 pad 1: /PV_POS_6 -> /PV_POS_5
- R60 pad 2: /BUCK_6/Vin+ -> /BUCK_5/Vin+
- R61 pad 1: /BUCK_6/BUCK_VIN -> /BUCK_5/BUCK_VIN
- R61 pad 2: /BUCK_6/Vin- -> /BUCK_5/Vin-
- R62 pad 1: /PV_POS_6 -> /PV_POS_5
- R62 pad 2: /BUCK_6/+IN -> /BUCK_5/+IN
- R63 pad 1: /BUCK_6/+IN -> /BUCK_5/+IN
- R63 pad 2: /NEG_6 -> /NEG_5
- R64 pad 1: /BUCK_6/BUCK_VIN -> /BUCK_5/BUCK_VIN
- R64 pad 2: /BUCK_6/RUN -> /BUCK_5/RUN
- R65 pad 1: /BUCK_6/Vfb -> /BUCK_5/Vfb
- R65 pad 2: /BUCK_6/P0A -> /BUCK_5/P0A
- R66 pad 1: /PV_POS_7 -> /PV_POS_5
- R66 pad 2: /BUCK_7/BUCK_VIN -> /BUCK_5/BUCK_VIN
- R67 pad 1: /PV_POS_7 -> /PV_POS_5
- R67 pad 2: /BUCK_7/Vin+ -> /BUCK_5/Vin+
- R68 pad 1: /BUCK_7/BUCK_VIN -> /BUCK_5/BUCK_VIN
- R68 pad 2: /BUCK_7/Vin- -> /BUCK_5/Vin-
- R69 pad 1: /PV_POS_7 -> /PV_POS_5
- R69 pad 2: /BUCK_7/+IN -> /BUCK_5/+IN
- R70 pad 1: /BUCK_7/+IN -> /BUCK_5/+IN
- R70 pad 2: /NEG_7 -> /NEG_5
- R71 pad 1: /BUCK_7/BUCK_VIN -> /BUCK_5/BUCK_VIN
- R71 pad 2: /BUCK_7/RUN -> /BUCK_5/RUN
- R72 pad 1: /BUCK_7/Vfb -> /BUCK_5/Vfb
- R72 pad 2: /BUCK_7/P0A -> /BUCK_5/P0A
- R73 pad 1: /PV_POS_8 -> /PV_POS_5
- R73 pad 2: /BUCK_8/BUCK_VIN -> /BUCK_5/BUCK_VIN
- R74 pad 1: /PV_POS_8 -> /PV_POS_5
- R74 pad 2: /BUCK_8/Vin+ -> /BUCK_5/Vin+
- R75 pad 1: /BUCK_8/BUCK_VIN -> /BUCK_5/BUCK_VIN
- R75 pad 2: /BUCK_8/Vin- -> /BUCK_5/Vin-
- R76 pad 1: /PV_POS_8 -> /PV_POS_5
- R76 pad 2: /BUCK_8/+IN -> /BUCK_5/+IN
- R77 pad 1: /BUCK_8/+IN -> /BUCK_5/+IN
- R77 pad 2: /NEG_8 -> /NEG_5
- R78 pad 1: /BUCK_8/BUCK_VIN -> /BUCK_5/BUCK_VIN
- R78 pad 2: /BUCK_8/RUN -> /BUCK_5/RUN
- R79 pad 1: /BUCK_8/Vfb -> /BUCK_5/Vfb
- R79 pad 2: /BUCK_8/P0A -> /BUCK_5/P0A
- R80 pad 1: /PV_POS_9 -> /PV_POS_5
- R80 pad 2: /BUCK_9/BUCK_VIN -> /BUCK_5/BUCK_VIN
- R81 pad 1: /PV_POS_9 -> /PV_POS_5
- R81 pad 2: /BUCK_9/Vin+ -> /BUCK_5/Vin+
- R82 pad 1: /BUCK_9/BUCK_VIN -> /BUCK_5/BUCK_VIN
- R82 pad 2: /BUCK_9/Vin- -> /BUCK_5/Vin-
- R83 pad 1: /PV_POS_9 -> /PV_POS_5
- R83 pad 2: /BUCK_9/+IN -> /BUCK_5/+IN
- R84 pad 1: /BUCK_9/+IN -> /BUCK_5/+IN
- R84 pad 2: /NEG_9 -> /NEG_5
- R85 pad 1: /BUCK_9/BUCK_VIN -> /BUCK_5/BUCK_VIN
- R85 pad 2: /BUCK_9/RUN -> /BUCK_5/RUN
- R86 pad 1: /BUCK_9/Vfb -> /BUCK_5/Vfb
- R86 pad 2: /BUCK_9/P0A -> /BUCK_5/P0A
- TP49 pad 1: Net-(TP49-Pad1) -> Net-(TP42-Pad1)
- TP50 pad 1: Net-(TP50-Pad1) -> Net-(TP43-Pad1)
- TP51 pad 1: Net-(TP51-Pad1) -> Net-(TP44-Pad1)
- TP52 pad 1: Net-(TP52-Pad1) -> Net-(TP45-Pad1)
- TP53 pad 1: Net-(JP7-Pad2) -> Net-(JP6-Pad2)
- TP54 pad 1: Net-(JP7-Pad1) -> Net-(JP6-Pad1)
- TP56 pad 1: Net-(TP56-Pad1) -> Net-(TP42-Pad1)
- TP57 pad 1: Net-(TP57-Pad1) -> Net-(TP43-Pad1)
- TP58 pad 1: Net-(TP58-Pad1) -> Net-(TP44-Pad1)
- TP59 pad 1: Net-(TP59-Pad1) -> Net-(TP45-Pad1)
- TP60 pad 1: Net-(JP8-Pad2) -> Net-(JP6-Pad2)
- TP61 pad 1: Net-(JP8-Pad1) -> Net-(JP6-Pad1)
- TP63 pad 1: Net-(TP63-Pad1) -> Net-(TP42-Pad1)
- TP64 pad 1: Net-(TP64-Pad1) -> Net-(TP43-Pad1)
- TP65 pad 1: Net-(TP65-Pad1) -> Net-(TP44-Pad1)
- TP66 pad 1: Net-(TP66-Pad1) -> Net-(TP45-Pad1)
- TP67 pad 1: Net-(JP9-Pad2) -> Net-(JP6-Pad2)
- TP68 pad 1: Net-(JP9-Pad1) -> Net-(JP6-Pad1)
- TP70 pad 1: Net-(TP70-Pad1) -> Net-(TP42-Pad1)
- TP71 pad 1: Net-(TP71-Pad1) -> Net-(TP43-Pad1)
- TP72 pad 1: Net-(TP72-Pad1) -> Net-(TP44-Pad1)
- TP73 pad 1: Net-(TP73-Pad1) -> Net-(TP45-Pad1)
- TP74 pad 1: Net-(JP10-Pad2) -> Net-(JP6-Pad2)
- TP75 pad 1: Net-(JP10-Pad1) -> Net-(JP6-Pad1)
- U28 pad 1: /NEG_6 -> /NEG_5
- U28 pad 4: Net-(C110-Pad1) -> Net-(C95-Pad1)
- U28 pad 5: Net-(TP49-Pad1) -> Net-(TP42-Pad1)
- U28 pad 7: unconnected-(U28-Pad7) -> unconnected-(U24-Pad7)
- U28 pad 8: /BUCK_6/+IN -> /BUCK_5/+IN
- U29 pad 10: /BUCK_6/Vin+ -> /BUCK_5/Vin+
- U29 pad 2: /SDA -> +5V
- U29 pad 3: unconnected-(U29-Pad3) -> unconnected-(U25-Pad3)
- U29 pad 8: Net-(TP49-Pad1) -> Net-(TP42-Pad1)
- U29 pad 9: /BUCK_6/Vin- -> /BUCK_5/Vin-
- U30 pad A1: /BUCK_6/BUCK_VIN -> /BUCK_5/BUCK_VIN
- U30 pad A10: /BUCK_6/RUN -> /BUCK_5/RUN
- U30 pad A11: Net-(TP52-Pad1) -> Net-(TP45-Pad1)
- U30 pad A12: unconnected-(U30-PadA12) -> unconnected-(U26-PadA12)
- U30 pad A2: /BUCK_6/BUCK_VIN -> /BUCK_5/BUCK_VIN
- U30 pad A3: /BUCK_6/BUCK_VIN -> /BUCK_5/BUCK_VIN
- U30 pad A4: /BUCK_6/BUCK_VIN -> /BUCK_5/BUCK_VIN
- U30 pad A5: /BUCK_6/BUCK_VIN -> /BUCK_5/BUCK_VIN
- U30 pad A6: /BUCK_6/BUCK_VIN -> /BUCK_5/BUCK_VIN
- U30 pad A7: Net-(TP48-Pad1) -> Net-(TP41-Pad1)
- U30 pad A8: /NEG_6 -> /NEG_5
- U30 pad A9: /BUCK_6/TRACK/SS -> /BUCK_5/TRACK/SS
- U30 pad B1: /BUCK_6/BUCK_VIN -> /BUCK_5/BUCK_VIN
- U30 pad B11: unconnected-(U30-PadB11) -> unconnected-(U26-PadB11)
- U30 pad B12: Net-(TP51-Pad1) -> Net-(TP44-Pad1)
- U30 pad B2: /BUCK_6/BUCK_VIN -> /BUCK_5/BUCK_VIN
- U30 pad B3: /BUCK_6/BUCK_VIN -> /BUCK_5/BUCK_VIN
- U30 pad B4: /BUCK_6/BUCK_VIN -> /BUCK_5/BUCK_VIN
- U30 pad B5: /BUCK_6/BUCK_VIN -> /BUCK_5/BUCK_VIN
- U30 pad B6: /BUCK_6/BUCK_VIN -> /BUCK_5/BUCK_VIN
- U30 pad B7: /NEG_6 -> /NEG_5
- U30 pad B9: /NEG_6 -> /NEG_5
- U30 pad C1: /BUCK_6/BUCK_VIN -> /BUCK_5/BUCK_VIN
- U30 pad C10: unconnected-(U30-PadC10) -> unconnected-(U26-PadC10)
- U30 pad C11: unconnected-(U30-PadC11) -> unconnected-(U26-PadC11)
- U30 pad C12: unconnected-(U30-PadC12) -> unconnected-(U26-PadC12)
- U30 pad C2: /BUCK_6/BUCK_VIN -> /BUCK_5/BUCK_VIN
- U30 pad C3: /BUCK_6/BUCK_VIN -> /BUCK_5/BUCK_VIN
- U30 pad C4: /BUCK_6/BUCK_VIN -> /BUCK_5/BUCK_VIN
- U30 pad C5: /BUCK_6/BUCK_VIN -> /BUCK_5/BUCK_VIN
- U30 pad C6: /BUCK_6/BUCK_VIN -> /BUCK_5/BUCK_VIN
- U30 pad C7: /NEG_6 -> /NEG_5
- U30 pad C9: /NEG_6 -> /NEG_5
- U30 pad D1: /NEG_6 -> /NEG_5
- U30 pad D10: unconnected-(U30-PadD10) -> unconnected-(U26-PadD10)
- U30 pad D11: unconnected-(U30-PadD11) -> unconnected-(U26-PadD11)
- U30 pad D12: unconnected-(U30-PadD12) -> unconnected-(U26-PadD12)
- U30 pad D2: /NEG_6 -> /NEG_5
- U30 pad D3: /NEG_6 -> /NEG_5
- U30 pad D4: /NEG_6 -> /NEG_5
- U30 pad D5: /NEG_6 -> /NEG_5
- U30 pad D6: /NEG_6 -> /NEG_5
- U30 pad D8: /NEG_6 -> /NEG_5
- U30 pad D9: unconnected-(U30-PadD9) -> unconnected-(U26-PadD9)
- U30 pad E1: /NEG_6 -> /NEG_5
- U30 pad E12: unconnected-(U30-PadE12) -> unconnected-(U26-PadE12)
- U30 pad E2: /NEG_6 -> /NEG_5
- U30 pad E3: /NEG_6 -> /NEG_5
- U30 pad E4: /NEG_6 -> /NEG_5
- U30 pad E5: /NEG_6 -> /NEG_5
- U30 pad E6: /NEG_6 -> /NEG_5
- U30 pad E7: /NEG_6 -> /NEG_5
- U30 pad E9: /NEG_6 -> /NEG_5
- U30 pad F1: /NEG_6 -> /NEG_5
- U30 pad F11: Net-(TP50-Pad1) -> Net-(TP43-Pad1)
- U30 pad F12: /BUCK_6/Vfb -> /BUCK_5/Vfb
- U30 pad F2: /NEG_6 -> /NEG_5
- U30 pad F3: /NEG_6 -> /NEG_5
- U30 pad F4: /NEG_6 -> /NEG_5
- U30 pad F5: /NEG_6 -> /NEG_5
- U30 pad F6: /NEG_6 -> /NEG_5
- U30 pad F7: /NEG_6 -> /NEG_5
- U30 pad F8: /NEG_6 -> /NEG_5
- U30 pad F9: /NEG_6 -> /NEG_5
- U30 pad G1: /NEG_6 -> /NEG_5
- U30 pad G11: /NEG_6 -> /NEG_5
- U30 pad G12: Net-(TP50-Pad1) -> Net-(TP43-Pad1)
- U30 pad G2: /NEG_6 -> /NEG_5
- U30 pad G3: /NEG_6 -> /NEG_5
- U30 pad G4: /NEG_6 -> /NEG_5
- U30 pad G5: /NEG_6 -> /NEG_5
- U30 pad G6: /NEG_6 -> /NEG_5
- U30 pad G7: /NEG_6 -> /NEG_5
- U30 pad G8: /NEG_6 -> /NEG_5
- U30 pad G9: /NEG_6 -> /NEG_5
- U30 pad H1: /NEG_6 -> /NEG_5
- U30 pad H11: /NEG_6 -> /NEG_5
- U30 pad H12: /NEG_6 -> /NEG_5
- U30 pad H2: /NEG_6 -> /NEG_5
- U30 pad H3: /NEG_6 -> /NEG_5
- U30 pad H4: /NEG_6 -> /NEG_5
- U30 pad H5: /NEG_6 -> /NEG_5
- U30 pad H6: /NEG_6 -> /NEG_5
- U30 pad H7: /NEG_6 -> /NEG_5
- U30 pad H8: /NEG_6 -> /NEG_5
- U30 pad H9: /NEG_6 -> /NEG_5
- U30 pad J1: /NEG_7 -> /NEG_6
- U30 pad J10: /NEG_7 -> /NEG_6
- U30 pad J12: /NEG_7 -> /NEG_6
- U30 pad J2: /NEG_7 -> /NEG_6
- U30 pad J3: /NEG_7 -> /NEG_6
- U30 pad J4: /NEG_7 -> /NEG_6
- U30 pad J5: /NEG_7 -> /NEG_6
- U30 pad J6: /NEG_7 -> /NEG_6
- U30 pad J7: /NEG_7 -> /NEG_6
- U30 pad J8: /NEG_7 -> /NEG_6
- U30 pad J9: /NEG_7 -> /NEG_6
- U30 pad K1: /NEG_7 -> /NEG_6
- U30 pad K10: /NEG_7 -> /NEG_6
- U30 pad K11: /NEG_7 -> /NEG_6
- U30 pad K12: Net-(JP7-Pad1) -> Net-(JP6-Pad1)
- U30 pad K2: /NEG_7 -> /NEG_6
- U30 pad K3: /NEG_7 -> /NEG_6
- U30 pad K4: /NEG_7 -> /NEG_6
- U30 pad K5: /NEG_7 -> /NEG_6
- U30 pad K6: /NEG_7 -> /NEG_6
- U30 pad K7: /NEG_7 -> /NEG_6
- U30 pad K8: /NEG_7 -> /NEG_6
- U30 pad K9: /NEG_7 -> /NEG_6
- U30 pad L1: /NEG_7 -> /NEG_6
- U30 pad L10: /NEG_7 -> /NEG_6
- U30 pad L11: /NEG_7 -> /NEG_6
- U30 pad L12: Net-(JP7-Pad2) -> Net-(JP6-Pad2)
- U30 pad L2: /NEG_7 -> /NEG_6
- U30 pad L3: /NEG_7 -> /NEG_6
- U30 pad L4: /NEG_7 -> /NEG_6
- U30 pad L5: /NEG_7 -> /NEG_6
- U30 pad L6: /NEG_7 -> /NEG_6
- U30 pad L7: /NEG_7 -> /NEG_6
- U30 pad L8: /NEG_7 -> /NEG_6
- U30 pad L9: /NEG_7 -> /NEG_6
- U30 pad M1: /NEG_7 -> /NEG_6
- U30 pad M10: /NEG_7 -> /NEG_6
- U30 pad M11: /NEG_7 -> /NEG_6
- U30 pad M12: /NEG_6 -> /NEG_5
- U30 pad M2: /NEG_7 -> /NEG_6
- U30 pad M3: /NEG_7 -> /NEG_6
- U30 pad M4: /NEG_7 -> /NEG_6
- U30 pad M5: /NEG_7 -> /NEG_6
- U30 pad M6: /NEG_7 -> /NEG_6
- U30 pad M7: /NEG_7 -> /NEG_6
- U30 pad M8: /NEG_7 -> /NEG_6
- U30 pad M9: /NEG_7 -> /NEG_6
- U31 pad 1: /CS6 -> /CS5
- U31 pad 5: /BUCK_6/P0A -> /BUCK_5/P0A
- U31 pad 6: /NEG_6 -> /NEG_5
- U31 pad 7: unconnected-(U31-Pad7) -> unconnected-(U27-Pad7)
- U32 pad 1: /NEG_7 -> /NEG_5
- U32 pad 4: Net-(C125-Pad1) -> Net-(C95-Pad1)
- U32 pad 5: Net-(TP56-Pad1) -> Net-(TP42-Pad1)
- U32 pad 7: unconnected-(U32-Pad7) -> unconnected-(U24-Pad7)
- U32 pad 8: /BUCK_7/+IN -> /BUCK_5/+IN
- U33 pad 10: /BUCK_7/Vin+ -> /BUCK_5/Vin+
- U33 pad 2: /SCL -> +5V
- U33 pad 3: unconnected-(U33-Pad3) -> unconnected-(U25-Pad3)
- U33 pad 8: Net-(TP56-Pad1) -> Net-(TP42-Pad1)
- U33 pad 9: /BUCK_7/Vin- -> /BUCK_5/Vin-
- U34 pad A1: /BUCK_7/BUCK_VIN -> /BUCK_5/BUCK_VIN
- U34 pad A10: /BUCK_7/RUN -> /BUCK_5/RUN
- U34 pad A11: Net-(TP59-Pad1) -> Net-(TP45-Pad1)
- U34 pad A12: unconnected-(U34-PadA12) -> unconnected-(U26-PadA12)
- U34 pad A2: /BUCK_7/BUCK_VIN -> /BUCK_5/BUCK_VIN
- U34 pad A3: /BUCK_7/BUCK_VIN -> /BUCK_5/BUCK_VIN
- U34 pad A4: /BUCK_7/BUCK_VIN -> /BUCK_5/BUCK_VIN
- U34 pad A5: /BUCK_7/BUCK_VIN -> /BUCK_5/BUCK_VIN
- U34 pad A6: /BUCK_7/BUCK_VIN -> /BUCK_5/BUCK_VIN
- U34 pad A7: Net-(TP55-Pad1) -> Net-(TP41-Pad1)
- U34 pad A8: /NEG_7 -> /NEG_5
- U34 pad A9: /BUCK_7/TRACK/SS -> /BUCK_5/TRACK/SS
- U34 pad B1: /BUCK_7/BUCK_VIN -> /BUCK_5/BUCK_VIN
- U34 pad B11: unconnected-(U34-PadB11) -> unconnected-(U26-PadB11)
- U34 pad B12: Net-(TP58-Pad1) -> Net-(TP44-Pad1)
- U34 pad B2: /BUCK_7/BUCK_VIN -> /BUCK_5/BUCK_VIN
- U34 pad B3: /BUCK_7/BUCK_VIN -> /BUCK_5/BUCK_VIN
- U34 pad B4: /BUCK_7/BUCK_VIN -> /BUCK_5/BUCK_VIN
- U34 pad B5: /BUCK_7/BUCK_VIN -> /BUCK_5/BUCK_VIN
- U34 pad B6: /BUCK_7/BUCK_VIN -> /BUCK_5/BUCK_VIN
- U34 pad B7: /NEG_7 -> /NEG_5
- U34 pad B9: /NEG_7 -> /NEG_5
- U34 pad C1: /BUCK_7/BUCK_VIN -> /BUCK_5/BUCK_VIN
- U34 pad C10: unconnected-(U34-PadC10) -> unconnected-(U26-PadC10)
- U34 pad C11: unconnected-(U34-PadC11) -> unconnected-(U26-PadC11)
- U34 pad C12: unconnected-(U34-PadC12) -> unconnected-(U26-PadC12)
- U34 pad C2: /BUCK_7/BUCK_VIN -> /BUCK_5/BUCK_VIN
- U34 pad C3: /BUCK_7/BUCK_VIN -> /BUCK_5/BUCK_VIN
- U34 pad C4: /BUCK_7/BUCK_VIN -> /BUCK_5/BUCK_VIN
- U34 pad C5: /BUCK_7/BUCK_VIN -> /BUCK_5/BUCK_VIN
- U34 pad C6: /BUCK_7/BUCK_VIN -> /BUCK_5/BUCK_VIN
- U34 pad C7: /NEG_7 -> /NEG_5
- U34 pad C9: /NEG_7 -> /NEG_5
- U34 pad D1: /NEG_7 -> /NEG_5
- U34 pad D10: unconnected-(U34-PadD10) -> unconnected-(U26-PadD10)
- U34 pad D11: unconnected-(U34-PadD11) -> unconnected-(U26-PadD11)
- U34 pad D12: unconnected-(U34-PadD12) -> unconnected-(U26-PadD12)
- U34 pad D2: /NEG_7 -> /NEG_5
- U34 pad D3: /NEG_7 -> /NEG_5
- U34 pad D4: /NEG_7 -> /NEG_5
- U34 pad D5: /NEG_7 -> /NEG_5
- U34 pad D6: /NEG_7 -> /NEG_5
- U34 pad D8: /NEG_7 -> /NEG_5
- U34 pad D9: unconnected-(U34-PadD9) -> unconnected-(U26-PadD9)
- U34 pad E1: /NEG_7 -> /NEG_5
- U34 pad E12: unconnected-(U34-PadE12) -> unconnected-(U26-PadE12)
- U34 pad E2: /NEG_7 -> /NEG_5
- U34 pad E3: /NEG_7 -> /NEG_5
- U34 pad E4: /NEG_7 -> /NEG_5
- U34 pad E5: /NEG_7 -> /NEG_5
- U34 pad E6: /NEG_7 -> /NEG_5
- U34 pad E7: /NEG_7 -> /NEG_5
- U34 pad E9: /NEG_7 -> /NEG_5
- U34 pad F1: /NEG_7 -> /NEG_5
- U34 pad F11: Net-(TP57-Pad1) -> Net-(TP43-Pad1)
- U34 pad F12: /BUCK_7/Vfb -> /BUCK_5/Vfb
- U34 pad F2: /NEG_7 -> /NEG_5
- U34 pad F3: /NEG_7 -> /NEG_5
- U34 pad F4: /NEG_7 -> /NEG_5
- U34 pad F5: /NEG_7 -> /NEG_5
- U34 pad F6: /NEG_7 -> /NEG_5
- U34 pad F7: /NEG_7 -> /NEG_5
- U34 pad F8: /NEG_7 -> /NEG_5
- U34 pad F9: /NEG_7 -> /NEG_5
- U34 pad G1: /NEG_7 -> /NEG_5
- U34 pad G11: /NEG_7 -> /NEG_5
- U34 pad G12: Net-(TP57-Pad1) -> Net-(TP43-Pad1)
- U34 pad G2: /NEG_7 -> /NEG_5
- U34 pad G3: /NEG_7 -> /NEG_5
- U34 pad G4: /NEG_7 -> /NEG_5
- U34 pad G5: /NEG_7 -> /NEG_5
- U34 pad G6: /NEG_7 -> /NEG_5
- U34 pad G7: /NEG_7 -> /NEG_5
- U34 pad G8: /NEG_7 -> /NEG_5
- U34 pad G9: /NEG_7 -> /NEG_5
- U34 pad H1: /NEG_7 -> /NEG_5
- U34 pad H11: /NEG_7 -> /NEG_5
- U34 pad H12: /NEG_7 -> /NEG_5
- U34 pad H2: /NEG_7 -> /NEG_5
- U34 pad H3: /NEG_7 -> /NEG_5
- U34 pad H4: /NEG_7 -> /NEG_5
- U34 pad H5: /NEG_7 -> /NEG_5
- U34 pad H6: /NEG_7 -> /NEG_5
- U34 pad H7: /NEG_7 -> /NEG_5
- U34 pad H8: /NEG_7 -> /NEG_5
- U34 pad H9: /NEG_7 -> /NEG_5
- U34 pad J1: /NEG_8 -> /NEG_6
- U34 pad J10: /NEG_8 -> /NEG_6
- U34 pad J12: /NEG_8 -> /NEG_6
- U34 pad J2: /NEG_8 -> /NEG_6
- U34 pad J3: /NEG_8 -> /NEG_6
- U34 pad J4: /NEG_8 -> /NEG_6
- U34 pad J5: /NEG_8 -> /NEG_6
- U34 pad J6: /NEG_8 -> /NEG_6
- U34 pad J7: /NEG_8 -> /NEG_6
- U34 pad J8: /NEG_8 -> /NEG_6
- U34 pad J9: /NEG_8 -> /NEG_6
- U34 pad K1: /NEG_8 -> /NEG_6
- U34 pad K10: /NEG_8 -> /NEG_6
- U34 pad K11: /NEG_8 -> /NEG_6
- U34 pad K12: Net-(JP8-Pad1) -> Net-(JP6-Pad1)
- U34 pad K2: /NEG_8 -> /NEG_6
- U34 pad K3: /NEG_8 -> /NEG_6
- U34 pad K4: /NEG_8 -> /NEG_6
- U34 pad K5: /NEG_8 -> /NEG_6
- U34 pad K6: /NEG_8 -> /NEG_6
- U34 pad K7: /NEG_8 -> /NEG_6
- U34 pad K8: /NEG_8 -> /NEG_6
- U34 pad K9: /NEG_8 -> /NEG_6
- U34 pad L1: /NEG_8 -> /NEG_6
- U34 pad L10: /NEG_8 -> /NEG_6
- U34 pad L11: /NEG_8 -> /NEG_6
- U34 pad L12: Net-(JP8-Pad2) -> Net-(JP6-Pad2)
- U34 pad L2: /NEG_8 -> /NEG_6
- U34 pad L3: /NEG_8 -> /NEG_6
- U34 pad L4: /NEG_8 -> /NEG_6
- U34 pad L5: /NEG_8 -> /NEG_6
- U34 pad L6: /NEG_8 -> /NEG_6
- U34 pad L7: /NEG_8 -> /NEG_6
- U34 pad L8: /NEG_8 -> /NEG_6
- U34 pad L9: /NEG_8 -> /NEG_6
- U34 pad M1: /NEG_8 -> /NEG_6
- U34 pad M10: /NEG_8 -> /NEG_6
- U34 pad M11: /NEG_8 -> /NEG_6
- U34 pad M12: /NEG_7 -> /NEG_5
- U34 pad M2: /NEG_8 -> /NEG_6
- U34 pad M3: /NEG_8 -> /NEG_6
- U34 pad M4: /NEG_8 -> /NEG_6
- U34 pad M5: /NEG_8 -> /NEG_6
- U34 pad M6: /NEG_8 -> /NEG_6
- U34 pad M7: /NEG_8 -> /NEG_6
- U34 pad M8: /NEG_8 -> /NEG_6
- U34 pad M9: /NEG_8 -> /NEG_6
- U35 pad 1: /CS7 -> /CS5
- U35 pad 5: /BUCK_7/P0A -> /BUCK_5/P0A
- U35 pad 6: /NEG_7 -> /NEG_5
- U35 pad 7: unconnected-(U35-Pad7) -> unconnected-(U27-Pad7)
- U36 pad 1: /NEG_8 -> /NEG_5
- U36 pad 4: Net-(C140-Pad1) -> Net-(C95-Pad1)
- U36 pad 5: Net-(TP63-Pad1) -> Net-(TP42-Pad1)
- U36 pad 7: unconnected-(U36-Pad7) -> unconnected-(U24-Pad7)
- U36 pad 8: /BUCK_8/+IN -> /BUCK_5/+IN
- U38 pad A1: /BUCK_8/BUCK_VIN -> /BUCK_5/BUCK_VIN
- U38 pad A10: /BUCK_8/RUN -> /BUCK_5/RUN
- U38 pad A11: Net-(TP66-Pad1) -> Net-(TP45-Pad1)
- U38 pad A12: unconnected-(U38-PadA12) -> unconnected-(U26-PadA12)
- U38 pad A2: /BUCK_8/BUCK_VIN -> /BUCK_5/BUCK_VIN
- U38 pad A3: /BUCK_8/BUCK_VIN -> /BUCK_5/BUCK_VIN
- U38 pad A4: /BUCK_8/BUCK_VIN -> /BUCK_5/BUCK_VIN
- U38 pad A5: /BUCK_8/BUCK_VIN -> /BUCK_5/BUCK_VIN
- U38 pad A6: /BUCK_8/BUCK_VIN -> /BUCK_5/BUCK_VIN
- U38 pad A7: Net-(TP62-Pad1) -> Net-(TP41-Pad1)
- U38 pad A8: /NEG_8 -> /NEG_5
- U38 pad A9: /BUCK_8/TRACK/SS -> /BUCK_5/TRACK/SS
- U38 pad B1: /BUCK_8/BUCK_VIN -> /BUCK_5/BUCK_VIN
- U38 pad B11: unconnected-(U38-PadB11) -> unconnected-(U26-PadB11)
- U38 pad B12: Net-(TP65-Pad1) -> Net-(TP44-Pad1)
- U38 pad B2: /BUCK_8/BUCK_VIN -> /BUCK_5/BUCK_VIN
- U38 pad B3: /BUCK_8/BUCK_VIN -> /BUCK_5/BUCK_VIN
- U38 pad B4: /BUCK_8/BUCK_VIN -> /BUCK_5/BUCK_VIN
- U38 pad B5: /BUCK_8/BUCK_VIN -> /BUCK_5/BUCK_VIN
- U38 pad B6: /BUCK_8/BUCK_VIN -> /BUCK_5/BUCK_VIN
- U38 pad B7: /NEG_8 -> /NEG_5
- U38 pad B9: /NEG_8 -> /NEG_5
- U38 pad C1: /BUCK_8/BUCK_VIN -> /BUCK_5/BUCK_VIN
- U38 pad C10: unconnected-(U38-PadC10) -> unconnected-(U26-PadC10)
- U38 pad C11: unconnected-(U38-PadC11) -> unconnected-(U26-PadC11)
- U38 pad C12: unconnected-(U38-PadC12) -> unconnected-(U26-PadC12)
- U38 pad C2: /BUCK_8/BUCK_VIN -> /BUCK_5/BUCK_VIN
- U38 pad C3: /BUCK_8/BUCK_VIN -> /BUCK_5/BUCK_VIN
- U38 pad C4: /BUCK_8/BUCK_VIN -> /BUCK_5/BUCK_VIN
- U38 pad C5: /BUCK_8/BUCK_VIN -> /BUCK_5/BUCK_VIN
- U38 pad C6: /BUCK_8/BUCK_VIN -> /BUCK_5/BUCK_VIN
- U38 pad C7: /NEG_8 -> /NEG_5
- U38 pad C9: /NEG_8 -> /NEG_5
- U38 pad D1: /NEG_8 -> /NEG_5
- U38 pad D10: unconnected-(U38-PadD10) -> unconnected-(U26-PadD10)
- U38 pad D11: unconnected-(U38-PadD11) -> unconnected-(U26-PadD11)
- U38 pad D12: unconnected-(U38-PadD12) -> unconnected-(U26-PadD12)
- U38 pad D2: /NEG_8 -> /NEG_5
- U38 pad D3: /NEG_8 -> /NEG_5
- U38 pad D4: /NEG_8 -> /NEG_5
- U38 pad D5: /NEG_8 -> /NEG_5
- U38 pad D6: /NEG_8 -> /NEG_5
- U38 pad D8: /NEG_8 -> /NEG_5
- U38 pad D9: unconnected-(U38-PadD9) -> unconnected-(U26-PadD9)
- U38 pad E1: /NEG_8 -> /NEG_5
- U38 pad E12: unconnected-(U38-PadE12) -> unconnected-(U26-PadE12)
- U38 pad E2: /NEG_8 -> /NEG_5
- U38 pad E3: /NEG_8 -> /NEG_5
- U38 pad E4: /NEG_8 -> /NEG_5
- U38 pad E5: /NEG_8 -> /NEG_5
- U38 pad E6: /NEG_8 -> /NEG_5
- U38 pad E7: /NEG_8 -> /NEG_5
- U38 pad E9: /NEG_8 -> /NEG_5
- U38 pad F1: /NEG_8 -> /NEG_5
- U38 pad F11: Net-(TP64-Pad1) -> Net-(TP43-Pad1)
- U38 pad F12: /BUCK_8/Vfb -> /BUCK_5/Vfb
- U38 pad F2: /NEG_8 -> /NEG_5
- U38 pad F3: /NEG_8 -> /NEG_5
- U38 pad F4: /NEG_8 -> /NEG_5
- U38 pad F5: /NEG_8 -> /NEG_5
- U38 pad F6: /NEG_8 -> /NEG_5
- U38 pad F7: /NEG_8 -> /NEG_5
- U38 pad F8: /NEG_8 -> /NEG_5
- U38 pad F9: /NEG_8 -> /NEG_5
- U38 pad G1: /NEG_8 -> /NEG_5
- U38 pad G11: /NEG_8 -> /NEG_5
- U38 pad G12: Net-(TP64-Pad1) -> Net-(TP43-Pad1)
- U38 pad G2: /NEG_8 -> /NEG_5
- U38 pad G3: /NEG_8 -> /NEG_5
- U38 pad G4: /NEG_8 -> /NEG_5
- U38 pad G5: /NEG_8 -> /NEG_5
- U38 pad G6: /NEG_8 -> /NEG_5
- U38 pad G7: /NEG_8 -> /NEG_5
- U38 pad G8: /NEG_8 -> /NEG_5
- U38 pad G9: /NEG_8 -> /NEG_5
- U38 pad H1: /NEG_8 -> /NEG_5
- U38 pad H11: /NEG_8 -> /NEG_5
- U38 pad H12: /NEG_8 -> /NEG_5
- U38 pad H2: /NEG_8 -> /NEG_5
- U38 pad H3: /NEG_8 -> /NEG_5
- U38 pad H4: /NEG_8 -> /NEG_5
- U38 pad H5: /NEG_8 -> /NEG_5
- U38 pad H6: /NEG_8 -> /NEG_5
- U38 pad H7: /NEG_8 -> /NEG_5
- U38 pad H8: /NEG_8 -> /NEG_5
- U38 pad H9: /NEG_8 -> /NEG_5
- U38 pad J1: /NEG_9 -> /NEG_6
- U38 pad J10: /NEG_9 -> /NEG_6
- U38 pad J12: /NEG_9 -> /NEG_6
- U38 pad J2: /NEG_9 -> /NEG_6
- U38 pad J3: /NEG_9 -> /NEG_6
- U38 pad J4: /NEG_9 -> /NEG_6
- U38 pad J5: /NEG_9 -> /NEG_6
- U38 pad J6: /NEG_9 -> /NEG_6
- U38 pad J7: /NEG_9 -> /NEG_6
- U38 pad J8: /NEG_9 -> /NEG_6
- U38 pad J9: /NEG_9 -> /NEG_6
- U38 pad K1: /NEG_9 -> /NEG_6
- U38 pad K10: /NEG_9 -> /NEG_6
- U38 pad K11: /NEG_9 -> /NEG_6
- U38 pad K12: Net-(JP9-Pad1) -> Net-(JP6-Pad1)
- U38 pad K2: /NEG_9 -> /NEG_6
- U38 pad K3: /NEG_9 -> /NEG_6
- U38 pad K4: /NEG_9 -> /NEG_6
- U38 pad K5: /NEG_9 -> /NEG_6
- U38 pad K6: /NEG_9 -> /NEG_6
- U38 pad K7: /NEG_9 -> /NEG_6
- U38 pad K8: /NEG_9 -> /NEG_6
- U38 pad K9: /NEG_9 -> /NEG_6
- U38 pad L1: /NEG_9 -> /NEG_6
- U38 pad L10: /NEG_9 -> /NEG_6
- U38 pad L11: /NEG_9 -> /NEG_6
- U38 pad L12: Net-(JP9-Pad2) -> Net-(JP6-Pad2)
- U38 pad L2: /NEG_9 -> /NEG_6
- U38 pad L3: /NEG_9 -> /NEG_6
- U38 pad L4: /NEG_9 -> /NEG_6
- U38 pad L5: /NEG_9 -> /NEG_6
- U38 pad L6: /NEG_9 -> /NEG_6
- U38 pad L7: /NEG_9 -> /NEG_6
- U38 pad L8: /NEG_9 -> /NEG_6
- U38 pad L9: /NEG_9 -> /NEG_6
- U38 pad M1: /NEG_9 -> /NEG_6
- U38 pad M10: /NEG_9 -> /NEG_6
- U38 pad M11: /NEG_9 -> /NEG_6
- U38 pad M12: /NEG_8 -> /NEG_5
- U38 pad M2: /NEG_9 -> /NEG_6
- U38 pad M3: /NEG_9 -> /NEG_6
- U38 pad M4: /NEG_9 -> /NEG_6
- U38 pad M5: /NEG_9 -> /NEG_6
- U38 pad M6: /NEG_9 -> /NEG_6
- U38 pad M7: /NEG_9 -> /NEG_6
- U38 pad M8: /NEG_9 -> /NEG_6
- U38 pad M9: /NEG_9 -> /NEG_6
- U39 pad 1: /CS8 -> /CS5
- U39 pad 5: /BUCK_8/P0A -> /BUCK_5/P0A
- U39 pad 6: /NEG_8 -> /NEG_5
- U39 pad 7: unconnected-(U39-Pad7) -> unconnected-(U27-Pad7)
- U40 pad 1: /NEG_9 -> /NEG_5
- U40 pad 4: Net-(C155-Pad1) -> Net-(C95-Pad1)
- U40 pad 5: Net-(TP70-Pad1) -> Net-(TP42-Pad1)
- U40 pad 7: unconnected-(U40-Pad7) -> unconnected-(U24-Pad7)
- U40 pad 8: /BUCK_9/+IN -> /BUCK_5/+IN
- U41 pad 1: /SDA -> +5V
- U41 pad 10: /BUCK_9/Vin+ -> /BUCK_5/Vin+
- U41 pad 3: unconnected-(U41-Pad3) -> unconnected-(U25-Pad3)
- U41 pad 8: Net-(TP70-Pad1) -> Net-(TP42-Pad1)
- U41 pad 9: /BUCK_9/Vin- -> /BUCK_5/Vin-
- U42 pad A1: /BUCK_9/BUCK_VIN -> /BUCK_5/BUCK_VIN
- U42 pad A10: /BUCK_9/RUN -> /BUCK_5/RUN
- U42 pad A11: Net-(TP73-Pad1) -> Net-(TP45-Pad1)
- U42 pad A12: unconnected-(U42-PadA12) -> unconnected-(U26-PadA12)
- U42 pad A2: /BUCK_9/BUCK_VIN -> /BUCK_5/BUCK_VIN
- U42 pad A3: /BUCK_9/BUCK_VIN -> /BUCK_5/BUCK_VIN
- U42 pad A4: /BUCK_9/BUCK_VIN -> /BUCK_5/BUCK_VIN
- U42 pad A5: /BUCK_9/BUCK_VIN -> /BUCK_5/BUCK_VIN
- U42 pad A6: /BUCK_9/BUCK_VIN -> /BUCK_5/BUCK_VIN
- U42 pad A7: Net-(TP69-Pad1) -> Net-(TP41-Pad1)
- U42 pad A8: /NEG_9 -> /NEG_5
- U42 pad A9: /BUCK_9/TRACK/SS -> /BUCK_5/TRACK/SS
- U42 pad B1: /BUCK_9/BUCK_VIN -> /BUCK_5/BUCK_VIN
- U42 pad B11: unconnected-(U42-PadB11) -> unconnected-(U26-PadB11)
- U42 pad B12: Net-(TP72-Pad1) -> Net-(TP44-Pad1)
- U42 pad B2: /BUCK_9/BUCK_VIN -> /BUCK_5/BUCK_VIN
- U42 pad B3: /BUCK_9/BUCK_VIN -> /BUCK_5/BUCK_VIN
- U42 pad B4: /BUCK_9/BUCK_VIN -> /BUCK_5/BUCK_VIN
- U42 pad B5: /BUCK_9/BUCK_VIN -> /BUCK_5/BUCK_VIN
- U42 pad B6: /BUCK_9/BUCK_VIN -> /BUCK_5/BUCK_VIN
- U42 pad B7: /NEG_9 -> /NEG_5
- U42 pad B9: /NEG_9 -> /NEG_5
- U42 pad C1: /BUCK_9/BUCK_VIN -> /BUCK_5/BUCK_VIN
- U42 pad C10: unconnected-(U42-PadC10) -> unconnected-(U26-PadC10)
- U42 pad C11: unconnected-(U42-PadC11) -> unconnected-(U26-PadC11)
- U42 pad C12: unconnected-(U42-PadC12) -> unconnected-(U26-PadC12)
- U42 pad C2: /BUCK_9/BUCK_VIN -> /BUCK_5/BUCK_VIN
- U42 pad C3: /BUCK_9/BUCK_VIN -> /BUCK_5/BUCK_VIN
- U42 pad C4: /BUCK_9/BUCK_VIN -> /BUCK_5/BUCK_VIN
- U42 pad C5: /BUCK_9/BUCK_VIN -> /BUCK_5/BUCK_VIN
- U42 pad C6: /BUCK_9/BUCK_VIN -> /BUCK_5/BUCK_VIN
- U42 pad C7: /NEG_9 -> /NEG_5
- U42 pad C9: /NEG_9 -> /NEG_5
- U42 pad D1: /NEG_9 -> /NEG_5
- U42 pad D10: unconnected-(U42-PadD10) -> unconnected-(U26-PadD10)
- U42 pad D11: unconnected-(U42-PadD11) -> unconnected-(U26-PadD11)
- U42 pad D12: unconnected-(U42-PadD12) -> unconnected-(U26-PadD12)
- U42 pad D2: /NEG_9 -> /NEG_5
- U42 pad D3: /NEG_9 -> /NEG_5
- U42 pad D4: /NEG_9 -> /NEG_5
- U42 pad D5: /NEG_9 -> /NEG_5
- U42 pad D6: /NEG_9 -> /NEG_5
- U42 pad D8: /NEG_9 -> /NEG_5
- U42 pad D9: unconnected-(U42-PadD9) -> unconnected-(U26-PadD9)
- U42 pad E1: /NEG_9 -> /NEG_5
- U42 pad E12: unconnected-(U42-PadE12) -> unconnected-(U26-PadE12)
- U42 pad E2: /NEG_9 -> /NEG_5
- U42 pad E3: /NEG_9 -> /NEG_5
- U42 pad E4: /NEG_9 -> /NEG_5
- U42 pad E5: /NEG_9 -> /NEG_5
- U42 pad E6: /NEG_9 -> /NEG_5
- U42 pad E7: /NEG_9 -> /NEG_5
- U42 pad E9: /NEG_9 -> /NEG_5
- U42 pad F1: /NEG_9 -> /NEG_5
- U42 pad F11: Net-(TP71-Pad1) -> Net-(TP43-Pad1)
- U42 pad F12: /BUCK_9/Vfb -> /BUCK_5/Vfb
- U42 pad F2: /NEG_9 -> /NEG_5
- U42 pad F3: /NEG_9 -> /NEG_5
- U42 pad F4: /NEG_9 -> /NEG_5
- U42 pad F5: /NEG_9 -> /NEG_5
- U42 pad F6: /NEG_9 -> /NEG_5
- U42 pad F7: /NEG_9 -> /NEG_5
- U42 pad F8: /NEG_9 -> /NEG_5
- U42 pad F9: /NEG_9 -> /NEG_5
- U42 pad G1: /NEG_9 -> /NEG_5
- U42 pad G11: /NEG_9 -> /NEG_5
- U42 pad G12: Net-(TP71-Pad1) -> Net-(TP43-Pad1)
- U42 pad G2: /NEG_9 -> /NEG_5
- U42 pad G3: /NEG_9 -> /NEG_5
- U42 pad G4: /NEG_9 -> /NEG_5
- U42 pad G5: /NEG_9 -> /NEG_5
- U42 pad G6: /NEG_9 -> /NEG_5
- U42 pad G7: /NEG_9 -> /NEG_5
- U42 pad G8: /NEG_9 -> /NEG_5
- U42 pad G9: /NEG_9 -> /NEG_5
- U42 pad H1: /NEG_9 -> /NEG_5
- U42 pad H11: /NEG_9 -> /NEG_5
- U42 pad H12: /NEG_9 -> /NEG_5
- U42 pad H2: /NEG_9 -> /NEG_5
- U42 pad H3: /NEG_9 -> /NEG_5
- U42 pad H4: /NEG_9 -> /NEG_5
- U42 pad H5: /NEG_9 -> /NEG_5
- U42 pad H6: /NEG_9 -> /NEG_5
- U42 pad H7: /NEG_9 -> /NEG_5
- U42 pad H8: /NEG_9 -> /NEG_5
- U42 pad H9: /NEG_9 -> /NEG_5
- U42 pad J1: /POS_9 -> /NEG_6
- U42 pad J10: /POS_9 -> /NEG_6
- U42 pad J12: /POS_9 -> /NEG_6
- U42 pad J2: /POS_9 -> /NEG_6
- U42 pad J3: /POS_9 -> /NEG_6
- U42 pad J4: /POS_9 -> /NEG_6
- U42 pad J5: /POS_9 -> /NEG_6
- U42 pad J6: /POS_9 -> /NEG_6
- U42 pad J7: /POS_9 -> /NEG_6
- U42 pad J8: /POS_9 -> /NEG_6
- U42 pad J9: /POS_9 -> /NEG_6
- U42 pad K1: /POS_9 -> /NEG_6
- U42 pad K10: /POS_9 -> /NEG_6
- U42 pad K11: /POS_9 -> /NEG_6
- U42 pad K12: Net-(JP10-Pad1) -> Net-(JP6-Pad1)
- U42 pad K2: /POS_9 -> /NEG_6
- U42 pad K3: /POS_9 -> /NEG_6
- U42 pad K4: /POS_9 -> /NEG_6
- U42 pad K5: /POS_9 -> /NEG_6
- U42 pad K6: /POS_9 -> /NEG_6
- U42 pad K7: /POS_9 -> /NEG_6
- U42 pad K8: /POS_9 -> /NEG_6
- U42 pad K9: /POS_9 -> /NEG_6
- U42 pad L1: /POS_9 -> /NEG_6
- U42 pad L10: /POS_9 -> /NEG_6
- U42 pad L11: /POS_9 -> /NEG_6
- U42 pad L12: Net-(JP10-Pad2) -> Net-(JP6-Pad2)
- U42 pad L2: /POS_9 -> /NEG_6
- U42 pad L3: /POS_9 -> /NEG_6
- U42 pad L4: /POS_9 -> /NEG_6
- U42 pad L5: /POS_9 -> /NEG_6
- U42 pad L6: /POS_9 -> /NEG_6
- U42 pad L7: /POS_9 -> /NEG_6
- U42 pad L8: /POS_9 -> /NEG_6
- U42 pad L9: /POS_9 -> /NEG_6
- U42 pad M1: /POS_9 -> /NEG_6
- U42 pad M10: /POS_9 -> /NEG_6
- U42 pad M11: /POS_9 -> /NEG_6
- U42 pad M12: /NEG_9 -> /NEG_5
- U42 pad M2: /POS_9 -> /NEG_6
- U42 pad M3: /POS_9 -> /NEG_6
- U42 pad M4: /POS_9 -> /NEG_6
- U42 pad M5: /POS_9 -> /NEG_6
- U42 pad M6: /POS_9 -> /NEG_6
- U42 pad M7: /POS_9 -> /NEG_6
- U42 pad M8: /POS_9 -> /NEG_6
- U42 pad M9: /POS_9 -> /NEG_6
- U43 pad 1: /CS9 -> /CS5
- U43 pad 5: /BUCK_9/P0A -> /BUCK_5/P0A
- U43 pad 6: /NEG_9 -> /NEG_5
- U43 pad 7: unconnected-(U43-Pad7) -> unconnected-(U27-Pad7)
Routing:
- net +5V: track 567.6 -> 1073.0 mm, vias 4 -> 0
- net GND: track 567.5 -> 186.9 mm, vias 18 -> 34
- net /NEG_5: track 19.8 -> 154.2 mm, vias 2 -> 20
- net Net-(TP42-Pad1): track 3.50 -> 130.9 mm, vias 0 -> 5
- net Net-(JP6-Pad2): track 18.0 -> 90.2 mm, vias 2 -> 10
- net Net-(TP43-Pad1): track 14.4 -> 71.9 mm, vias 2 -> 10
- net /BUCK_5/Vin-: track 0.00 -> 52.2 mm
- net Net-(JP6-Pad1): track 12.1 -> 60.6 mm, vias 2 -> 10
- net /BUCK_5/+IN: track 0.00 -> 46.1 mm
- net /BUCK_5/Vin+: track 0.00 -> 38.1 mm
- net /BUCK_5/BUCK_VIN: track 4.54 -> 42.0 mm
- net /NEG_6: track 5.19 -> 25.9 mm
- net Net-(TP45-Pad1): track 4.86 -> 24.3 mm
- net Net-(TP41-Pad1): track 4.75 -> 23.7 mm, vias 2 -> 10
- net /PV_POS_5: track 0.00 -> 18.9 mm
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- added copper zone on In1.Cu, net GND
Other:
- copper layers 2 -> 4
- board text removed: "Moeten we wel de diff. amp. gebruiken?"
