File: KiCAD/Quest_39/Quest_39.kicad_pcb (KiCad board)
At the start: 4 copper layers, 398 parts, among them J1 1x2 Scr. Term., J10 1x2 Scr. Term., J11 1x2 Scr. Term., J12 Conn_01x05_Male, J2 1x2 Scr. Term., J3 1x2 Scr. Term., J4 1x2 Scr. Term., J5 1x2 Scr. Term., J6 1x2 Scr. Term., J7 1x2 Scr. Term., J8 1x2 Scr. Term., J9 1x2 Scr. Term., U1 AZ1117-3.3, U10 LTM4611EV-PBF, U11 MCP4151-502E/SN, U12 AD626ANZ, U13 INA226, U14 LTM4611EV-PBF, U15 MCP4151-502E/SN, U16 AD626ANZ, U17 INA226, U18 LTM4611EV-PBF, U19 MCP4151-502E/SN, U2 17791063215, U20 AD626ANZ, U21 INA226, U22 LTM4611EV-PBF, U23 MCP4151-502E/SN, U24 AD626ANZ, U25 INA226, U26 LTM4611EV-PBF, U27 MCP4151-502E/SN, U28 AD626ANZ, U29 INA226, U3 STM32F103C8T6, U30 LTM4611EV-PBF, U31 MCP4151-502E/SN, U32 AD626ANZ, U33 INA226, U34 LTM4611EV-PBF, U35 MCP4151-502E/SN, U36 AD626ANZ, U37 100nF, U37 INA226, U38 LTM4611EV-PBF, U39 MCP4151-502E/SN, U4 AD626ANZ, U40 AD626ANZ, U41 INA226, U42 LTM4611EV-PBF, U43 MCP4151-502E/SN, U5 INA226, U6 LTM4611EV-PBF, U7 MCP4151-502E/SN, U8 AD626ANZ, U9 INA226, Y1 16MHz

Commit message: Routed I2C SDA/SCL
Parts:
- moved U1 97.6 mm to (96.3, 146.1)
- moved R6 84.5 mm to (83.9, 108.1)
- moved R5 84.3 mm to (86.8, 108.1)
- moved U2 73.3 mm to (74.5, 230.2)
- moved C2 73.0 mm to (97.4, 131.5)
- moved C4 73.0 mm to (92.4, 119.0)
- moved C12 73.0 mm to (86.5, 124.5)
- moved C13 73.0 mm to (86.5, 128.0)
- moved C5 73.0 mm to (89.0, 121.5)
- moved C7 73.0 mm to (89.5, 131.0)
- moved C8 73.0 mm to (89.5, 133.0)
- moved D2 73.0 mm to (82.0, 135.7)
- moved FB1 73.0 mm to (92.0, 132.0)
- moved R4 73.0 mm to (82.0, 132.6)
- moved Y1 73.0 mm to (84.0, 126.1)
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Routing:
- net /SDA: track 2.86 -> 832.1 mm, vias 0 -> 10
- net /SCL: track 0.00 -> 526.8 mm, vias 0 -> 10
- net /SWDIO: track 0.00 -> 19.4 mm
- net /SWO: track 0.00 -> 13.3 mm
- net /SWCLK: track 0.00 -> 11.8 mm
- net /HSE_IN: track 0.00 -> 9.06 mm
- net /HSE_OUT: track 0.00 -> 7.24 mm
- net Net-(D2-Pad2): track 0.00 -> 3.07 mm
- net /BUCK_4/BUCK_VIN: track 8.24 -> 5.23 mm
- net /BUCK_1/Vin-: track 6.38 -> 9.27 mm, vias 2 -> 0
- net /BUCK_2/Vin-: track 6.70 -> 9.48 mm, vias 2 -> 0
- net /BUCK_0/Vin-: track 7.23 -> 9.94 mm, vias 2 -> 0
- net /BUCK_3/Vin-: track 7.17 -> 9.55 mm, vias 2 -> 0
- net /BUCK_4/Vin-: track 7.41 -> 9.73 mm, vias 2 -> 0
- net Net-(TP27-Pad1): track 4.41 -> 6.37 mm
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- added copper zone on In2.Cu, net GND

Commit message: Switched to 4-layer stack-up w/ dedicated +5V and GND planes to improve EMI and make routing for PWR-traces easier
Routing:
- net +5V: track 1073.0 -> 106.7 mm, vias 0 -> 43
- net /SCL: track 526.8 -> 889.4 mm, vias 10 -> 0
- net Net-(TP42-Pad1): track 130.9 -> 139.2 mm, vias 5 -> 1
- net /SDA: track 832.1 -> 830.6 mm
- added copper zone on In2.Cu, net +5V
- removed copper zone on In2.Cu, net GND
Other:
- board text added: "misschien een fout: wrm willen de LTM4611's aan de rechterkant allemaal NEG_5?"

Commit message: Redid layout for the LTM4611EV Buck-converters (Issues with net-assignment to IC pads)
Parts:
- removed the J11 at (180.3, 218.8)
- removed the U37 at (160.9, 186.9)
- removed the U37 at (163.7, 186.6)
- added C138: 100nF, Capacitor_SMD:C_0603_1608Metric, F.Cu at (160.0, 107.5)
- added J7: 1x2 Scr. Term., TB005:TB005-762-02BE, F.Cu at (180.1, 168.6)
- added U37: INA226, Package_SO:VSSOP-10_3x3mm_P0.5mm, F.Cu at (162.6, 107.3)
- moved C102 172.8 mm to (124.0, 199.3)
- moved C103 172.8 mm to (119.7, 192.8)
- moved C89 172.8 mm to (155.5, 203.2)
- moved C90 172.8 mm to (146.2, 203.3)
- moved C91 172.8 mm to (144.3, 203.3)
- moved C93 172.8 mm to (160.8, 221.1)
- moved C95 172.8 mm to (167.3, 222.4)
- moved C97 172.8 mm to (130.8, 208.1)
- moved J6 172.8 mm to (180.2, 207.0)
- moved JP6 172.8 mm to (124.1, 181.5)
- moved R53 172.8 mm to (164.0, 210.6)
- moved R56 172.8 mm to (171.3, 212.0)
- moved R58 172.8 mm to (121.8, 199.1)
- moved TP41 172.8 mm to (133.9, 210.6)
- moved TP44 172.8 mm to (122.8, 206.1)
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- renumbered J6 to J11, J7 to J6
Connections:
- C104 pad 1: /BUCK_5/BUCK_VIN -> /BUCK_6/BUCK_VIN
- C104 pad 2: /NEG_5 -> /NEG_6
- C105 pad 1: /BUCK_5/BUCK_VIN -> /BUCK_6/BUCK_VIN
- C105 pad 2: /NEG_5 -> /NEG_6
- C106 pad 1: /BUCK_5/BUCK_VIN -> /BUCK_6/BUCK_VIN
- C106 pad 2: /NEG_5 -> /NEG_6
- C107 pad 1: /BUCK_5/BUCK_VIN -> /BUCK_6/BUCK_VIN
- C107 pad 2: /NEG_5 -> /NEG_6
- C109 pad 1: /BUCK_5/Vin+ -> /BUCK_6/Vin+
- C109 pad 2: /BUCK_5/Vin- -> /BUCK_6/Vin-
- C110 pad 1: Net-(C95-Pad1) -> Net-(C110-Pad1)
- C112 pad 1: /NEG_5 -> /NEG_6
- C112 pad 2: /BUCK_5/TRACK/SS -> /BUCK_6/TRACK/SS
- C113 pad 1: /NEG_6 -> /NEG_7
- C113 pad 2: /NEG_5 -> /NEG_6
- C114 pad 1: /NEG_6 -> /NEG_7
- C114 pad 2: /NEG_5 -> /NEG_6
- C115 pad 1: /NEG_6 -> /NEG_7
- C115 pad 2: /NEG_5 -> /NEG_6
- C116 pad 1: /NEG_6 -> /NEG_7
- C116 pad 2: /NEG_5 -> /NEG_6
- C117 pad 1: /NEG_6 -> /NEG_7
- C117 pad 2: /BUCK_5/Vfb -> /BUCK_6/Vfb
- C119 pad 1: /BUCK_5/BUCK_VIN -> /BUCK_7/BUCK_VIN
- C119 pad 2: /NEG_5 -> /NEG_7
- C120 pad 1: /BUCK_5/BUCK_VIN -> /BUCK_7/BUCK_VIN
- C120 pad 2: /NEG_5 -> /NEG_7
- C121 pad 1: /BUCK_5/BUCK_VIN -> /BUCK_7/BUCK_VIN
- C121 pad 2: /NEG_5 -> /NEG_7
- C122 pad 1: /BUCK_5/BUCK_VIN -> /BUCK_7/BUCK_VIN
- C122 pad 2: /NEG_5 -> /NEG_7
- C124 pad 1: /BUCK_5/Vin+ -> /BUCK_7/Vin+
- C124 pad 2: /BUCK_5/Vin- -> /BUCK_7/Vin-
- C125 pad 1: Net-(C95-Pad1) -> Net-(C125-Pad1)
- C127 pad 1: /NEG_5 -> /NEG_7
- C127 pad 2: /BUCK_5/TRACK/SS -> /BUCK_7/TRACK/SS
- C128 pad 1: /NEG_6 -> /NEG_8
- C128 pad 2: /NEG_5 -> /NEG_7
- C129 pad 1: /NEG_6 -> /NEG_8
- C129 pad 2: /NEG_5 -> /NEG_7
- C130 pad 1: /NEG_6 -> /NEG_8
- C130 pad 2: /NEG_5 -> /NEG_7
- C131 pad 1: /NEG_6 -> /NEG_8
- C131 pad 2: /NEG_5 -> /NEG_7
- C132 pad 1: /NEG_6 -> /NEG_8
- C132 pad 2: /BUCK_5/Vfb -> /BUCK_7/Vfb
- C134 pad 1: /BUCK_5/BUCK_VIN -> /BUCK_8/BUCK_VIN
- C134 pad 2: /NEG_5 -> /NEG_8
- C135 pad 1: /BUCK_5/BUCK_VIN -> /BUCK_8/BUCK_VIN
- C135 pad 2: /NEG_5 -> /NEG_8
- C136 pad 1: /BUCK_5/BUCK_VIN -> /BUCK_8/BUCK_VIN
- C136 pad 2: /NEG_5 -> /NEG_8
- C137 pad 1: /BUCK_5/BUCK_VIN -> /BUCK_8/BUCK_VIN
- C137 pad 2: /NEG_5 -> /NEG_8
- C139 pad 1: /BUCK_5/Vin+ -> /BUCK_8/Vin+
- C139 pad 2: /BUCK_5/Vin- -> /BUCK_8/Vin-
- C140 pad 1: Net-(C95-Pad1) -> Net-(C140-Pad1)
- C142 pad 1: /NEG_5 -> /NEG_8
- C142 pad 2: /BUCK_5/TRACK/SS -> /BUCK_8/TRACK/SS
- C143 pad 1: /NEG_6 -> /NEG_9
- C143 pad 2: /NEG_5 -> /NEG_8
- C144 pad 1: /NEG_6 -> /NEG_9
- C144 pad 2: /NEG_5 -> /NEG_8
- C145 pad 1: /NEG_6 -> /NEG_9
- C145 pad 2: /NEG_5 -> /NEG_8
- C146 pad 1: /NEG_6 -> /NEG_9
- C146 pad 2: /NEG_5 -> /NEG_8
- C147 pad 1: /NEG_6 -> /NEG_9
- C147 pad 2: /BUCK_5/Vfb -> /BUCK_8/Vfb
- C149 pad 1: /BUCK_5/BUCK_VIN -> /BUCK_9/BUCK_VIN
- C149 pad 2: /NEG_5 -> /NEG_9
- C150 pad 1: /BUCK_5/BUCK_VIN -> /BUCK_9/BUCK_VIN
- C150 pad 2: /NEG_5 -> /NEG_9
- C151 pad 1: /BUCK_5/BUCK_VIN -> /BUCK_9/BUCK_VIN
- C151 pad 2: /NEG_5 -> /NEG_9
- C152 pad 1: /BUCK_5/BUCK_VIN -> /BUCK_9/BUCK_VIN
- C152 pad 2: /NEG_5 -> /NEG_9
- C154 pad 1: /BUCK_5/Vin+ -> /BUCK_9/Vin+
- C154 pad 2: /BUCK_5/Vin- -> /BUCK_9/Vin-
- C155 pad 1: Net-(C95-Pad1) -> Net-(C155-Pad1)
- C157 pad 1: /NEG_5 -> /NEG_9
- C157 pad 2: /BUCK_5/TRACK/SS -> /BUCK_9/TRACK/SS
- C158 pad 1: /NEG_6 -> /POS_9
- C158 pad 2: /NEG_5 -> /NEG_9
- C159 pad 1: /NEG_6 -> /POS_9
- C159 pad 2: /NEG_5 -> /NEG_9
- C160 pad 1: /NEG_6 -> /POS_9
- C160 pad 2: /NEG_5 -> /NEG_9
- C161 pad 1: /NEG_6 -> /POS_9
- C161 pad 2: /NEG_5 -> /NEG_9
- C162 pad 1: /NEG_6 -> /POS_9
- C162 pad 2: /BUCK_5/Vfb -> /BUCK_9/Vfb
- J10 pad 1: /PV_POS_5 -> /PV_POS_9
- J10 pad 2: /NEG_5 -> /NEG_9
- J8 pad 1: /PV_POS_5 -> /PV_POS_7
- J8 pad 2: /NEG_5 -> /NEG_7
- J9 pad 1: /PV_POS_5 -> /PV_POS_8
- J9 pad 2: /NEG_5 -> /NEG_8
- JP10 pad 1: Net-(JP6-Pad1) -> Net-(JP10-Pad1)
- JP10 pad 2: Net-(JP6-Pad2) -> Net-(JP10-Pad2)
- JP7 pad 1: Net-(JP6-Pad1) -> Net-(JP7-Pad1)
- JP7 pad 2: Net-(JP6-Pad2) -> Net-(JP7-Pad2)
- JP8 pad 1: Net-(JP6-Pad1) -> Net-(JP8-Pad1)
- JP8 pad 2: Net-(JP6-Pad2) -> Net-(JP8-Pad2)
- JP9 pad 1: Net-(JP6-Pad1) -> Net-(JP9-Pad1)
- JP9 pad 2: Net-(JP6-Pad2) -> Net-(JP9-Pad2)
- R59 pad 1: /PV_POS_5 -> /PV_POS_6
- R59 pad 2: /BUCK_5/BUCK_VIN -> /BUCK_6/BUCK_VIN
- R60 pad 1: /PV_POS_5 -> /PV_POS_6
- R60 pad 2: /BUCK_5/Vin+ -> /BUCK_6/Vin+
- R61 pad 1: /BUCK_5/BUCK_VIN -> /BUCK_6/BUCK_VIN
- R61 pad 2: /BUCK_5/Vin- -> /BUCK_6/Vin-
- R62 pad 1: /PV_POS_5 -> /PV_POS_6
- R62 pad 2: /BUCK_5/+IN -> /BUCK_6/+IN
- R63 pad 1: /BUCK_5/+IN -> /BUCK_6/+IN
- R63 pad 2: /NEG_5 -> /NEG_6
- R64 pad 1: /BUCK_5/BUCK_VIN -> /BUCK_6/BUCK_VIN
- R64 pad 2: /BUCK_5/RUN -> /BUCK_6/RUN
- R65 pad 1: /BUCK_5/Vfb -> /BUCK_6/Vfb
- R65 pad 2: /BUCK_5/P0A -> /BUCK_6/P0A
- R66 pad 1: /PV_POS_5 -> /PV_POS_7
- R66 pad 2: /BUCK_5/BUCK_VIN -> /BUCK_7/BUCK_VIN
- R67 pad 1: /PV_POS_5 -> /PV_POS_7
- R67 pad 2: /BUCK_5/Vin+ -> /BUCK_7/Vin+
- R68 pad 1: /BUCK_5/BUCK_VIN -> /BUCK_7/BUCK_VIN
- R68 pad 2: /BUCK_5/Vin- -> /BUCK_7/Vin-
- R69 pad 1: /PV_POS_5 -> /PV_POS_7
- R69 pad 2: /BUCK_5/+IN -> /BUCK_7/+IN
- R70 pad 1: /BUCK_5/+IN -> /BUCK_7/+IN
- R70 pad 2: /NEG_5 -> /NEG_7
- R71 pad 1: /BUCK_5/BUCK_VIN -> /BUCK_7/BUCK_VIN
- R71 pad 2: /BUCK_5/RUN -> /BUCK_7/RUN
- R72 pad 1: /BUCK_5/Vfb -> /BUCK_7/Vfb
- R72 pad 2: /BUCK_5/P0A -> /BUCK_7/P0A
- R73 pad 1: /PV_POS_5 -> /PV_POS_8
- R73 pad 2: /BUCK_5/BUCK_VIN -> /BUCK_8/BUCK_VIN
- R74 pad 1: /PV_POS_5 -> /PV_POS_8
- R74 pad 2: /BUCK_5/Vin+ -> /BUCK_8/Vin+
- R75 pad 1: /BUCK_5/BUCK_VIN -> /BUCK_8/BUCK_VIN
- R75 pad 2: /BUCK_5/Vin- -> /BUCK_8/Vin-
- R76 pad 1: /PV_POS_5 -> /PV_POS_8
- R76 pad 2: /BUCK_5/+IN -> /BUCK_8/+IN
- R77 pad 1: /BUCK_5/+IN -> /BUCK_8/+IN
- R77 pad 2: /NEG_5 -> /NEG_8
- R78 pad 1: /BUCK_5/BUCK_VIN -> /BUCK_8/BUCK_VIN
- R78 pad 2: /BUCK_5/RUN -> /BUCK_8/RUN
- R79 pad 1: /BUCK_5/Vfb -> /BUCK_8/Vfb
- R79 pad 2: /BUCK_5/P0A -> /BUCK_8/P0A
- R80 pad 1: /PV_POS_5 -> /PV_POS_9
- R80 pad 2: /BUCK_5/BUCK_VIN -> /BUCK_9/BUCK_VIN
- R81 pad 1: /PV_POS_5 -> /PV_POS_9
- R81 pad 2: /BUCK_5/Vin+ -> /BUCK_9/Vin+
- R82 pad 1: /BUCK_5/BUCK_VIN -> /BUCK_9/BUCK_VIN
- R82 pad 2: /BUCK_5/Vin- -> /BUCK_9/Vin-
- R83 pad 1: /PV_POS_5 -> /PV_POS_9
- R83 pad 2: /BUCK_5/+IN -> /BUCK_9/+IN
- R84 pad 1: /BUCK_5/+IN -> /BUCK_9/+IN
- R84 pad 2: /NEG_5 -> /NEG_9
- R85 pad 1: /BUCK_5/BUCK_VIN -> /BUCK_9/BUCK_VIN
- R85 pad 2: /BUCK_5/RUN -> /BUCK_9/RUN
- R86 pad 1: /BUCK_5/Vfb -> /BUCK_9/Vfb
- R86 pad 2: /BUCK_5/P0A -> /BUCK_9/P0A
- TP48 pad 1: Net-(TP41-Pad1) -> Net-(TP48-Pad1)
- TP49 pad 1: Net-(TP42-Pad1) -> Net-(TP49-Pad1)
- TP50 pad 1: Net-(TP43-Pad1) -> Net-(TP50-Pad1)
- TP51 pad 1: Net-(TP44-Pad1) -> Net-(TP51-Pad1)
- TP52 pad 1: Net-(TP45-Pad1) -> Net-(TP52-Pad1)
- TP53 pad 1: Net-(JP6-Pad2) -> Net-(JP7-Pad2)
- TP54 pad 1: Net-(JP6-Pad1) -> Net-(JP7-Pad1)
- TP55 pad 1: Net-(TP41-Pad1) -> Net-(TP55-Pad1)
- TP56 pad 1: Net-(TP42-Pad1) -> Net-(TP56-Pad1)
- TP57 pad 1: Net-(TP43-Pad1) -> Net-(TP57-Pad1)
- TP58 pad 1: Net-(TP44-Pad1) -> Net-(TP58-Pad1)
- TP59 pad 1: Net-(TP45-Pad1) -> Net-(TP59-Pad1)
- TP60 pad 1: Net-(JP6-Pad2) -> Net-(JP8-Pad2)
- TP61 pad 1: Net-(JP6-Pad1) -> Net-(JP8-Pad1)
- TP62 pad 1: Net-(TP41-Pad1) -> Net-(TP62-Pad1)
- TP63 pad 1: Net-(TP42-Pad1) -> Net-(TP63-Pad1)
- TP64 pad 1: Net-(TP43-Pad1) -> Net-(TP64-Pad1)
- TP65 pad 1: Net-(TP44-Pad1) -> Net-(TP65-Pad1)
- TP66 pad 1: Net-(TP45-Pad1) -> Net-(TP66-Pad1)
- TP67 pad 1: Net-(JP6-Pad2) -> Net-(JP9-Pad2)
- TP68 pad 1: Net-(JP6-Pad1) -> Net-(JP9-Pad1)
- TP69 pad 1: Net-(TP41-Pad1) -> Net-(TP69-Pad1)
- TP70 pad 1: Net-(TP42-Pad1) -> Net-(TP70-Pad1)
- TP71 pad 1: Net-(TP43-Pad1) -> Net-(TP71-Pad1)
- TP72 pad 1: Net-(TP44-Pad1) -> Net-(TP72-Pad1)
- TP73 pad 1: Net-(TP45-Pad1) -> Net-(TP73-Pad1)
- TP74 pad 1: Net-(JP6-Pad2) -> Net-(JP10-Pad2)
- TP75 pad 1: Net-(JP6-Pad1) -> Net-(JP10-Pad1)
- U28 pad 1: /NEG_5 -> /NEG_6
- U28 pad 4: Net-(C95-Pad1) -> Net-(C110-Pad1)
- U28 pad 5: Net-(TP42-Pad1) -> Net-(TP49-Pad1)
- U28 pad 7: unconnected-(U24-Pad7) -> unconnected-(U28-Pad7)
- U28 pad 8: /BUCK_5/+IN -> /BUCK_6/+IN
- U29 pad 10: /BUCK_5/Vin+ -> /BUCK_6/Vin+
- U29 pad 2: +5V -> /SDA
- U29 pad 3: unconnected-(U25-Pad3) -> unconnected-(U29-Pad3)
- U29 pad 8: Net-(TP42-Pad1) -> Net-(TP49-Pad1)
- U29 pad 9: /BUCK_5/Vin- -> /BUCK_6/Vin-
- U30 pad A1: /BUCK_5/BUCK_VIN -> /BUCK_6/BUCK_VIN
- U30 pad A10: /BUCK_5/RUN -> /BUCK_6/RUN
- U30 pad A11: Net-(TP45-Pad1) -> Net-(TP52-Pad1)
- U30 pad A12: unconnected-(U26-PadA12) -> unconnected-(U30-PadA12)
- U30 pad A2: /BUCK_5/BUCK_VIN -> /BUCK_6/BUCK_VIN
- U30 pad A3: /BUCK_5/BUCK_VIN -> /BUCK_6/BUCK_VIN
- U30 pad A4: /BUCK_5/BUCK_VIN -> /BUCK_6/BUCK_VIN
- U30 pad A5: /BUCK_5/BUCK_VIN -> /BUCK_6/BUCK_VIN
- U30 pad A6: /BUCK_5/BUCK_VIN -> /BUCK_6/BUCK_VIN
- U30 pad A7: Net-(TP41-Pad1) -> Net-(TP48-Pad1)
- U30 pad A8: /NEG_5 -> /NEG_6
- U30 pad A9: /BUCK_5/TRACK/SS -> /BUCK_6/TRACK/SS
- U30 pad B1: /BUCK_5/BUCK_VIN -> /BUCK_6/BUCK_VIN
- U30 pad B11: unconnected-(U26-PadB11) -> unconnected-(U30-PadB11)
- U30 pad B12: Net-(TP44-Pad1) -> Net-(TP51-Pad1)
- U30 pad B2: /BUCK_5/BUCK_VIN -> /BUCK_6/BUCK_VIN
- U30 pad B3: /BUCK_5/BUCK_VIN -> /BUCK_6/BUCK_VIN
- U30 pad B4: /BUCK_5/BUCK_VIN -> /BUCK_6/BUCK_VIN
- U30 pad B5: /BUCK_5/BUCK_VIN -> /BUCK_6/BUCK_VIN
- U30 pad B6: /BUCK_5/BUCK_VIN -> /BUCK_6/BUCK_VIN
- U30 pad B7: /NEG_5 -> /NEG_6
- U30 pad B9: /NEG_5 -> /NEG_6
- U30 pad C1: /BUCK_5/BUCK_VIN -> /BUCK_6/BUCK_VIN
- U30 pad C10: unconnected-(U26-PadC10) -> unconnected-(U30-PadC10)
- U30 pad C11: unconnected-(U26-PadC11) -> unconnected-(U30-PadC11)
- U30 pad C12: unconnected-(U26-PadC12) -> unconnected-(U30-PadC12)
- U30 pad C2: /BUCK_5/BUCK_VIN -> /BUCK_6/BUCK_VIN
- U30 pad C3: /BUCK_5/BUCK_VIN -> /BUCK_6/BUCK_VIN
- U30 pad C4: /BUCK_5/BUCK_VIN -> /BUCK_6/BUCK_VIN
- U30 pad C5: /BUCK_5/BUCK_VIN -> /BUCK_6/BUCK_VIN
- U30 pad C6: /BUCK_5/BUCK_VIN -> /BUCK_6/BUCK_VIN
- U30 pad C7: /NEG_5 -> /NEG_6
- U30 pad C9: /NEG_5 -> /NEG_6
- U30 pad D1: /NEG_5 -> /NEG_6
- U30 pad D10: unconnected-(U26-PadD10) -> unconnected-(U30-PadD10)
- U30 pad D11: unconnected-(U26-PadD11) -> unconnected-(U30-PadD11)
- U30 pad D12: unconnected-(U26-PadD12) -> unconnected-(U30-PadD12)
- U30 pad D2: /NEG_5 -> /NEG_6
- U30 pad D3: /NEG_5 -> /NEG_6
- U30 pad D4: /NEG_5 -> /NEG_6
- U30 pad D5: /NEG_5 -> /NEG_6
- U30 pad D6: /NEG_5 -> /NEG_6
- U30 pad D8: /NEG_5 -> /NEG_6
- U30 pad D9: unconnected-(U26-PadD9) -> unconnected-(U30-PadD9)
- U30 pad E1: /NEG_5 -> /NEG_6
- U30 pad E12: unconnected-(U26-PadE12) -> unconnected-(U30-PadE12)
- U30 pad E2: /NEG_5 -> /NEG_6
- U30 pad E3: /NEG_5 -> /NEG_6
- U30 pad E4: /NEG_5 -> /NEG_6
- U30 pad E5: /NEG_5 -> /NEG_6
- U30 pad E6: /NEG_5 -> /NEG_6
- U30 pad E7: /NEG_5 -> /NEG_6
- U30 pad E9: /NEG_5 -> /NEG_6
- U30 pad F1: /NEG_5 -> /NEG_6
- U30 pad F11: Net-(TP43-Pad1) -> Net-(TP50-Pad1)
- U30 pad F12: /BUCK_5/Vfb -> /BUCK_6/Vfb
- U30 pad F2: /NEG_5 -> /NEG_6
- U30 pad F3: /NEG_5 -> /NEG_6
- U30 pad F4: /NEG_5 -> /NEG_6
- U30 pad F5: /NEG_5 -> /NEG_6
- U30 pad F6: /NEG_5 -> /NEG_6
- U30 pad F7: /NEG_5 -> /NEG_6
- U30 pad F8: /NEG_5 -> /NEG_6
- U30 pad F9: /NEG_5 -> /NEG_6
- U30 pad G1: /NEG_5 -> /NEG_6
- U30 pad G11: /NEG_5 -> /NEG_6
- U30 pad G12: Net-(TP43-Pad1) -> Net-(TP50-Pad1)
- U30 pad G2: /NEG_5 -> /NEG_6
- U30 pad G3: /NEG_5 -> /NEG_6
- U30 pad G4: /NEG_5 -> /NEG_6
- U30 pad G5: /NEG_5 -> /NEG_6
- U30 pad G6: /NEG_5 -> /NEG_6
- U30 pad G7: /NEG_5 -> /NEG_6
- U30 pad G8: /NEG_5 -> /NEG_6
- U30 pad G9: /NEG_5 -> /NEG_6
- U30 pad H1: /NEG_5 -> /NEG_6
- U30 pad H11: /NEG_5 -> /NEG_6
- U30 pad H12: /NEG_5 -> /NEG_6
- U30 pad H2: /NEG_5 -> /NEG_6
- U30 pad H3: /NEG_5 -> /NEG_6
- U30 pad H4: /NEG_5 -> /NEG_6
- U30 pad H5: /NEG_5 -> /NEG_6
- U30 pad H6: /NEG_5 -> /NEG_6
- U30 pad H7: /NEG_5 -> /NEG_6
- U30 pad H8: /NEG_5 -> /NEG_6
- U30 pad H9: /NEG_5 -> /NEG_6
- U30 pad J1: /NEG_6 -> /NEG_7
- U30 pad J10: /NEG_6 -> /NEG_7
- U30 pad J12: /NEG_6 -> /NEG_7
- U30 pad J2: /NEG_6 -> /NEG_7
- U30 pad J3: /NEG_6 -> /NEG_7
- U30 pad J4: /NEG_6 -> /NEG_7
- U30 pad J5: /NEG_6 -> /NEG_7
- U30 pad J6: /NEG_6 -> /NEG_7
- U30 pad J7: /NEG_6 -> /NEG_7
- U30 pad J8: /NEG_6 -> /NEG_7
- U30 pad J9: /NEG_6 -> /NEG_7
- U30 pad K1: /NEG_6 -> /NEG_7
- U30 pad K10: /NEG_6 -> /NEG_7
- U30 pad K11: /NEG_6 -> /NEG_7
- U30 pad K12: Net-(JP6-Pad1) -> Net-(JP7-Pad1)
- U30 pad K2: /NEG_6 -> /NEG_7
- U30 pad K3: /NEG_6 -> /NEG_7
- U30 pad K4: /NEG_6 -> /NEG_7
- U30 pad K5: /NEG_6 -> /NEG_7
- U30 pad K6: /NEG_6 -> /NEG_7
- U30 pad K7: /NEG_6 -> /NEG_7
- U30 pad K8: /NEG_6 -> /NEG_7
- U30 pad K9: /NEG_6 -> /NEG_7
- U30 pad L1: /NEG_6 -> /NEG_7
- U30 pad L10: /NEG_6 -> /NEG_7
- U30 pad L11: /NEG_6 -> /NEG_7
- U30 pad L12: Net-(JP6-Pad2) -> Net-(JP7-Pad2)
- U30 pad L2: /NEG_6 -> /NEG_7
- U30 pad L3: /NEG_6 -> /NEG_7
- U30 pad L4: /NEG_6 -> /NEG_7
- U30 pad L5: /NEG_6 -> /NEG_7
- U30 pad L6: /NEG_6 -> /NEG_7
- U30 pad L7: /NEG_6 -> /NEG_7
- U30 pad L8: /NEG_6 -> /NEG_7
- U30 pad L9: /NEG_6 -> /NEG_7
- U30 pad M1: /NEG_6 -> /NEG_7
- U30 pad M10: /NEG_6 -> /NEG_7
- U30 pad M11: /NEG_6 -> /NEG_7
- U30 pad M12: /NEG_5 -> /NEG_6
- U30 pad M2: /NEG_6 -> /NEG_7
- U30 pad M3: /NEG_6 -> /NEG_7
- U30 pad M4: /NEG_6 -> /NEG_7
- U30 pad M5: /NEG_6 -> /NEG_7
- U30 pad M6: /NEG_6 -> /NEG_7
- U30 pad M7: /NEG_6 -> /NEG_7
- U30 pad M8: /NEG_6 -> /NEG_7
- U30 pad M9: /NEG_6 -> /NEG_7
- U31 pad 1: /CS5 -> /CS6
- U31 pad 5: /BUCK_5/P0A -> /BUCK_6/P0A
- U31 pad 6: /NEG_5 -> /NEG_6
- U31 pad 7: unconnected-(U27-Pad7) -> unconnected-(U31-Pad7)
- U32 pad 1: /NEG_5 -> /NEG_7
- U32 pad 4: Net-(C95-Pad1) -> Net-(C125-Pad1)
- U32 pad 5: Net-(TP42-Pad1) -> Net-(TP56-Pad1)
- U32 pad 7: unconnected-(U24-Pad7) -> unconnected-(U32-Pad7)
- U32 pad 8: /BUCK_5/+IN -> /BUCK_7/+IN
- U33 pad 10: /BUCK_5/Vin+ -> /BUCK_7/Vin+
- U33 pad 2: +5V -> /SCL
- U33 pad 3: unconnected-(U25-Pad3) -> unconnected-(U33-Pad3)
- U33 pad 8: Net-(TP42-Pad1) -> Net-(TP56-Pad1)
- U33 pad 9: /BUCK_5/Vin- -> /BUCK_7/Vin-
- U34 pad A1: /BUCK_5/BUCK_VIN -> /BUCK_7/BUCK_VIN
- U34 pad A10: /BUCK_5/RUN -> /BUCK_7/RUN
- U34 pad A11: Net-(TP45-Pad1) -> Net-(TP59-Pad1)
- U34 pad A12: unconnected-(U26-PadA12) -> unconnected-(U34-PadA12)
- U34 pad A2: /BUCK_5/BUCK_VIN -> /BUCK_7/BUCK_VIN
- U34 pad A3: /BUCK_5/BUCK_VIN -> /BUCK_7/BUCK_VIN
- U34 pad A4: /BUCK_5/BUCK_VIN -> /BUCK_7/BUCK_VIN
- U34 pad A5: /BUCK_5/BUCK_VIN -> /BUCK_7/BUCK_VIN
- U34 pad A6: /BUCK_5/BUCK_VIN -> /BUCK_7/BUCK_VIN
- U34 pad A7: Net-(TP41-Pad1) -> Net-(TP55-Pad1)
- U34 pad A8: /NEG_5 -> /NEG_7
- U34 pad A9: /BUCK_5/TRACK/SS -> /BUCK_7/TRACK/SS
- U34 pad B1: /BUCK_5/BUCK_VIN -> /BUCK_7/BUCK_VIN
- U34 pad B11: unconnected-(U26-PadB11) -> unconnected-(U34-PadB11)
- U34 pad B12: Net-(TP44-Pad1) -> Net-(TP58-Pad1)
- U34 pad B2: /BUCK_5/BUCK_VIN -> /BUCK_7/BUCK_VIN
- U34 pad B3: /BUCK_5/BUCK_VIN -> /BUCK_7/BUCK_VIN
- U34 pad B4: /BUCK_5/BUCK_VIN -> /BUCK_7/BUCK_VIN
- U34 pad B5: /BUCK_5/BUCK_VIN -> /BUCK_7/BUCK_VIN
- U34 pad B6: /BUCK_5/BUCK_VIN -> /BUCK_7/BUCK_VIN
- U34 pad B7: /NEG_5 -> /NEG_7
- U34 pad B9: /NEG_5 -> /NEG_7
- U34 pad C1: /BUCK_5/BUCK_VIN -> /BUCK_7/BUCK_VIN
- U34 pad C10: unconnected-(U26-PadC10) -> unconnected-(U34-PadC10)
- U34 pad C11: unconnected-(U26-PadC11) -> unconnected-(U34-PadC11)
- U34 pad C12: unconnected-(U26-PadC12) -> unconnected-(U34-PadC12)
- U34 pad C2: /BUCK_5/BUCK_VIN -> /BUCK_7/BUCK_VIN
- U34 pad C3: /BUCK_5/BUCK_VIN -> /BUCK_7/BUCK_VIN
- U34 pad C4: /BUCK_5/BUCK_VIN -> /BUCK_7/BUCK_VIN
- U34 pad C5: /BUCK_5/BUCK_VIN -> /BUCK_7/BUCK_VIN
- U34 pad C6: /BUCK_5/BUCK_VIN -> /BUCK_7/BUCK_VIN
- U34 pad C7: /NEG_5 -> /NEG_7
- U34 pad C9: /NEG_5 -> /NEG_7
- U34 pad D1: /NEG_5 -> /NEG_7
- U34 pad D10: unconnected-(U26-PadD10) -> unconnected-(U34-PadD10)
- U34 pad D11: unconnected-(U26-PadD11) -> unconnected-(U34-PadD11)
- U34 pad D12: unconnected-(U26-PadD12) -> unconnected-(U34-PadD12)
- U34 pad D2: /NEG_5 -> /NEG_7
- U34 pad D3: /NEG_5 -> /NEG_7
- U34 pad D4: /NEG_5 -> /NEG_7
- U34 pad D5: /NEG_5 -> /NEG_7
- U34 pad D6: /NEG_5 -> /NEG_7
- U34 pad D8: /NEG_5 -> /NEG_7
- U34 pad D9: unconnected-(U26-PadD9) -> unconnected-(U34-PadD9)
- U34 pad E1: /NEG_5 -> /NEG_7
- U34 pad E12: unconnected-(U26-PadE12) -> unconnected-(U34-PadE12)
- U34 pad E2: /NEG_5 -> /NEG_7
- U34 pad E3: /NEG_5 -> /NEG_7
- U34 pad E4: /NEG_5 -> /NEG_7
- U34 pad E5: /NEG_5 -> /NEG_7
- U34 pad E6: /NEG_5 -> /NEG_7
- U34 pad E7: /NEG_5 -> /NEG_7
- U34 pad E9: /NEG_5 -> /NEG_7
- U34 pad F1: /NEG_5 -> /NEG_7
- U34 pad F11: Net-(TP43-Pad1) -> Net-(TP57-Pad1)
- U34 pad F12: /BUCK_5/Vfb -> /BUCK_7/Vfb
- U34 pad F2: /NEG_5 -> /NEG_7
- U34 pad F3: /NEG_5 -> /NEG_7
- U34 pad F4: /NEG_5 -> /NEG_7
- U34 pad F5: /NEG_5 -> /NEG_7
- U34 pad F6: /NEG_5 -> /NEG_7
- U34 pad F7: /NEG_5 -> /NEG_7
- U34 pad F8: /NEG_5 -> /NEG_7
- U34 pad F9: /NEG_5 -> /NEG_7
- U34 pad G1: /NEG_5 -> /NEG_7
- U34 pad G11: /NEG_5 -> /NEG_7
- U34 pad G12: Net-(TP43-Pad1) -> Net-(TP57-Pad1)
- U34 pad G2: /NEG_5 -> /NEG_7
- U34 pad G3: /NEG_5 -> /NEG_7
- U34 pad G4: /NEG_5 -> /NEG_7
- U34 pad G5: /NEG_5 -> /NEG_7
- U34 pad G6: /NEG_5 -> /NEG_7
- U34 pad G7: /NEG_5 -> /NEG_7
- U34 pad G8: /NEG_5 -> /NEG_7
- U34 pad G9: /NEG_5 -> /NEG_7
- U34 pad H1: /NEG_5 -> /NEG_7
- U34 pad H11: /NEG_5 -> /NEG_7
- U34 pad H12: /NEG_5 -> /NEG_7
- U34 pad H2: /NEG_5 -> /NEG_7
- U34 pad H3: /NEG_5 -> /NEG_7
- U34 pad H4: /NEG_5 -> /NEG_7
- U34 pad H5: /NEG_5 -> /NEG_7
- U34 pad H6: /NEG_5 -> /NEG_7
- U34 pad H7: /NEG_5 -> /NEG_7
- U34 pad H8: /NEG_5 -> /NEG_7
- U34 pad H9: /NEG_5 -> /NEG_7
- U34 pad J1: /NEG_6 -> /NEG_8
- U34 pad J10: /NEG_6 -> /NEG_8
- U34 pad J12: /NEG_6 -> /NEG_8
- U34 pad J2: /NEG_6 -> /NEG_8
- U34 pad J3: /NEG_6 -> /NEG_8
- U34 pad J4: /NEG_6 -> /NEG_8
- U34 pad J5: /NEG_6 -> /NEG_8
- U34 pad J6: /NEG_6 -> /NEG_8
- U34 pad J7: /NEG_6 -> /NEG_8
- U34 pad J8: /NEG_6 -> /NEG_8
- U34 pad J9: /NEG_6 -> /NEG_8
- U34 pad K1: /NEG_6 -> /NEG_8
- U34 pad K10: /NEG_6 -> /NEG_8
- U34 pad K11: /NEG_6 -> /NEG_8
- U34 pad K12: Net-(JP6-Pad1) -> Net-(JP8-Pad1)
- U34 pad K2: /NEG_6 -> /NEG_8
- U34 pad K3: /NEG_6 -> /NEG_8
- U34 pad K4: /NEG_6 -> /NEG_8
- U34 pad K5: /NEG_6 -> /NEG_8
- U34 pad K6: /NEG_6 -> /NEG_8
- U34 pad K7: /NEG_6 -> /NEG_8
- U34 pad K8: /NEG_6 -> /NEG_8
- U34 pad K9: /NEG_6 -> /NEG_8
- U34 pad L1: /NEG_6 -> /NEG_8
- U34 pad L10: /NEG_6 -> /NEG_8
- U34 pad L11: /NEG_6 -> /NEG_8
- U34 pad L12: Net-(JP6-Pad2) -> Net-(JP8-Pad2)
- U34 pad L2: /NEG_6 -> /NEG_8
- U34 pad L3: /NEG_6 -> /NEG_8
- U34 pad L4: /NEG_6 -> /NEG_8
- U34 pad L5: /NEG_6 -> /NEG_8
- U34 pad L6: /NEG_6 -> /NEG_8
- U34 pad L7: /NEG_6 -> /NEG_8
- U34 pad L8: /NEG_6 -> /NEG_8
- U34 pad L9: /NEG_6 -> /NEG_8
- U34 pad M1: /NEG_6 -> /NEG_8
- U34 pad M10: /NEG_6 -> /NEG_8
- U34 pad M11: /NEG_6 -> /NEG_8
- U34 pad M12: /NEG_5 -> /NEG_7
- U34 pad M2: /NEG_6 -> /NEG_8
- U34 pad M3: /NEG_6 -> /NEG_8
- U34 pad M4: /NEG_6 -> /NEG_8
- U34 pad M5: /NEG_6 -> /NEG_8
- U34 pad M6: /NEG_6 -> /NEG_8
- U34 pad M7: /NEG_6 -> /NEG_8
- U34 pad M8: /NEG_6 -> /NEG_8
- U34 pad M9: /NEG_6 -> /NEG_8
- U35 pad 1: /CS5 -> /CS7
- U35 pad 5: /BUCK_5/P0A -> /BUCK_7/P0A
- U35 pad 6: /NEG_5 -> /NEG_7
- U35 pad 7: unconnected-(U27-Pad7) -> unconnected-(U35-Pad7)
- U36 pad 1: /NEG_5 -> /NEG_8
- U36 pad 4: Net-(C95-Pad1) -> Net-(C140-Pad1)
- U36 pad 5: Net-(TP42-Pad1) -> Net-(TP63-Pad1)
- U36 pad 7: unconnected-(U24-Pad7) -> unconnected-(U36-Pad7)
- U36 pad 8: /BUCK_5/+IN -> /BUCK_8/+IN
- U38 pad A1: /BUCK_5/BUCK_VIN -> /BUCK_8/BUCK_VIN
- U38 pad A10: /BUCK_5/RUN -> /BUCK_8/RUN
- U38 pad A11: Net-(TP45-Pad1) -> Net-(TP66-Pad1)
- U38 pad A12: unconnected-(U26-PadA12) -> unconnected-(U38-PadA12)
- U38 pad A2: /BUCK_5/BUCK_VIN -> /BUCK_8/BUCK_VIN
- U38 pad A3: /BUCK_5/BUCK_VIN -> /BUCK_8/BUCK_VIN
- U38 pad A4: /BUCK_5/BUCK_VIN -> /BUCK_8/BUCK_VIN
- U38 pad A5: /BUCK_5/BUCK_VIN -> /BUCK_8/BUCK_VIN
- U38 pad A6: /BUCK_5/BUCK_VIN -> /BUCK_8/BUCK_VIN
- U38 pad A7: Net-(TP41-Pad1) -> Net-(TP62-Pad1)
- U38 pad A8: /NEG_5 -> /NEG_8
- U38 pad A9: /BUCK_5/TRACK/SS -> /BUCK_8/TRACK/SS
- U38 pad B1: /BUCK_5/BUCK_VIN -> /BUCK_8/BUCK_VIN
- U38 pad B11: unconnected-(U26-PadB11) -> unconnected-(U38-PadB11)
- U38 pad B12: Net-(TP44-Pad1) -> Net-(TP65-Pad1)
- U38 pad B2: /BUCK_5/BUCK_VIN -> /BUCK_8/BUCK_VIN
- U38 pad B3: /BUCK_5/BUCK_VIN -> /BUCK_8/BUCK_VIN
- U38 pad B4: /BUCK_5/BUCK_VIN -> /BUCK_8/BUCK_VIN
- U38 pad B5: /BUCK_5/BUCK_VIN -> /BUCK_8/BUCK_VIN
- U38 pad B6: /BUCK_5/BUCK_VIN -> /BUCK_8/BUCK_VIN
- U38 pad B7: /NEG_5 -> /NEG_8
- U38 pad B9: /NEG_5 -> /NEG_8
- U38 pad C1: /BUCK_5/BUCK_VIN -> /BUCK_8/BUCK_VIN
- U38 pad C10: unconnected-(U26-PadC10) -> unconnected-(U38-PadC10)
- U38 pad C11: unconnected-(U26-PadC11) -> unconnected-(U38-PadC11)
- U38 pad C12: unconnected-(U26-PadC12) -> unconnected-(U38-PadC12)
- U38 pad C2: /BUCK_5/BUCK_VIN -> /BUCK_8/BUCK_VIN
- U38 pad C3: /BUCK_5/BUCK_VIN -> /BUCK_8/BUCK_VIN
- U38 pad C4: /BUCK_5/BUCK_VIN -> /BUCK_8/BUCK_VIN
- U38 pad C5: /BUCK_5/BUCK_VIN -> /BUCK_8/BUCK_VIN
- U38 pad C6: /BUCK_5/BUCK_VIN -> /BUCK_8/BUCK_VIN
- U38 pad C7: /NEG_5 -> /NEG_8
- U38 pad C9: /NEG_5 -> /NEG_8
- U38 pad D1: /NEG_5 -> /NEG_8
- U38 pad D10: unconnected-(U26-PadD10) -> unconnected-(U38-PadD10)
- U38 pad D11: unconnected-(U26-PadD11) -> unconnected-(U38-PadD11)
- U38 pad D12: unconnected-(U26-PadD12) -> unconnected-(U38-PadD12)
- U38 pad D2: /NEG_5 -> /NEG_8
- U38 pad D3: /NEG_5 -> /NEG_8
- U38 pad D4: /NEG_5 -> /NEG_8
- U38 pad D5: /NEG_5 -> /NEG_8
- U38 pad D6: /NEG_5 -> /NEG_8
- U38 pad D8: /NEG_5 -> /NEG_8
- U38 pad D9: unconnected-(U26-PadD9) -> unconnected-(U38-PadD9)
- U38 pad E1: /NEG_5 -> /NEG_8
- U38 pad E12: unconnected-(U26-PadE12) -> unconnected-(U38-PadE12)
- U38 pad E2: /NEG_5 -> /NEG_8
- U38 pad E3: /NEG_5 -> /NEG_8
- U38 pad E4: /NEG_5 -> /NEG_8
- U38 pad E5: /NEG_5 -> /NEG_8
- U38 pad E6: /NEG_5 -> /NEG_8
- U38 pad E7: /NEG_5 -> /NEG_8
- U38 pad E9: /NEG_5 -> /NEG_8
- U38 pad F1: /NEG_5 -> /NEG_8
- U38 pad F11: Net-(TP43-Pad1) -> Net-(TP64-Pad1)
- U38 pad F12: /BUCK_5/Vfb -> /BUCK_8/Vfb
- U38 pad F2: /NEG_5 -> /NEG_8
- U38 pad F3: /NEG_5 -> /NEG_8
- U38 pad F4: /NEG_5 -> /NEG_8
- U38 pad F5: /NEG_5 -> /NEG_8
- U38 pad F6: /NEG_5 -> /NEG_8
- U38 pad F7: /NEG_5 -> /NEG_8
- U38 pad F8: /NEG_5 -> /NEG_8
- U38 pad F9: /NEG_5 -> /NEG_8
- U38 pad G1: /NEG_5 -> /NEG_8
- U38 pad G11: /NEG_5 -> /NEG_8
- U38 pad G12: Net-(TP43-Pad1) -> Net-(TP64-Pad1)
- U38 pad G2: /NEG_5 -> /NEG_8
- U38 pad G3: /NEG_5 -> /NEG_8
- U38 pad G4: /NEG_5 -> /NEG_8
- U38 pad G5: /NEG_5 -> /NEG_8
- U38 pad G6: /NEG_5 -> /NEG_8
- U38 pad G7: /NEG_5 -> /NEG_8
- U38 pad G8: /NEG_5 -> /NEG_8
- U38 pad G9: /NEG_5 -> /NEG_8
- U38 pad H1: /NEG_5 -> /NEG_8
- U38 pad H11: /NEG_5 -> /NEG_8
- U38 pad H12: /NEG_5 -> /NEG_8
- U38 pad H2: /NEG_5 -> /NEG_8
- U38 pad H3: /NEG_5 -> /NEG_8
- U38 pad H4: /NEG_5 -> /NEG_8
- U38 pad H5: /NEG_5 -> /NEG_8
- U38 pad H6: /NEG_5 -> /NEG_8
- U38 pad H7: /NEG_5 -> /NEG_8
- U38 pad H8: /NEG_5 -> /NEG_8
- U38 pad H9: /NEG_5 -> /NEG_8
- U38 pad J1: /NEG_6 -> /NEG_9
- U38 pad J10: /NEG_6 -> /NEG_9
- U38 pad J12: /NEG_6 -> /NEG_9
- U38 pad J2: /NEG_6 -> /NEG_9
- U38 pad J3: /NEG_6 -> /NEG_9
- U38 pad J4: /NEG_6 -> /NEG_9
- U38 pad J5: /NEG_6 -> /NEG_9
- U38 pad J6: /NEG_6 -> /NEG_9
- U38 pad J7: /NEG_6 -> /NEG_9
- U38 pad J8: /NEG_6 -> /NEG_9
- U38 pad J9: /NEG_6 -> /NEG_9
- U38 pad K1: /NEG_6 -> /NEG_9
- U38 pad K10: /NEG_6 -> /NEG_9
- U38 pad K11: /NEG_6 -> /NEG_9
- U38 pad K12: Net-(JP6-Pad1) -> Net-(JP9-Pad1)
- U38 pad K2: /NEG_6 -> /NEG_9
- U38 pad K3: /NEG_6 -> /NEG_9
- U38 pad K4: /NEG_6 -> /NEG_9
- U38 pad K5: /NEG_6 -> /NEG_9
- U38 pad K6: /NEG_6 -> /NEG_9
- U38 pad K7: /NEG_6 -> /NEG_9
- U38 pad K8: /NEG_6 -> /NEG_9
- U38 pad K9: /NEG_6 -> /NEG_9
- U38 pad L1: /NEG_6 -> /NEG_9
- U38 pad L10: /NEG_6 -> /NEG_9
- U38 pad L11: /NEG_6 -> /NEG_9
- U38 pad L12: Net-(JP6-Pad2) -> Net-(JP9-Pad2)
- U38 pad L2: /NEG_6 -> /NEG_9
- U38 pad L3: /NEG_6 -> /NEG_9
- U38 pad L4: /NEG_6 -> /NEG_9
- U38 pad L5: /NEG_6 -> /NEG_9
- U38 pad L6: /NEG_6 -> /NEG_9
- U38 pad L7: /NEG_6 -> /NEG_9
- U38 pad L8: /NEG_6 -> /NEG_9
- U38 pad L9: /NEG_6 -> /NEG_9
- U38 pad M1: /NEG_6 -> /NEG_9
- U38 pad M10: /NEG_6 -> /NEG_9
- U38 pad M11: /NEG_6 -> /NEG_9
- U38 pad M12: /NEG_5 -> /NEG_8
- U38 pad M2: /NEG_6 -> /NEG_9
- U38 pad M3: /NEG_6 -> /NEG_9
- U38 pad M4: /NEG_6 -> /NEG_9
- U38 pad M5: /NEG_6 -> /NEG_9
- U38 pad M6: /NEG_6 -> /NEG_9
- U38 pad M7: /NEG_6 -> /NEG_9
- U38 pad M8: /NEG_6 -> /NEG_9
- U38 pad M9: /NEG_6 -> /NEG_9
- U39 pad 1: /CS5 -> /CS8
- U39 pad 5: /BUCK_5/P0A -> /BUCK_8/P0A
- U39 pad 6: /NEG_5 -> /NEG_8
- U39 pad 7: unconnected-(U27-Pad7) -> unconnected-(U39-Pad7)
- U40 pad 1: /NEG_5 -> /NEG_9
- U40 pad 4: Net-(C95-Pad1) -> Net-(C155-Pad1)
- U40 pad 5: Net-(TP42-Pad1) -> Net-(TP70-Pad1)
- U40 pad 7: unconnected-(U24-Pad7) -> unconnected-(U40-Pad7)
- U40 pad 8: /BUCK_5/+IN -> /BUCK_9/+IN
- U41 pad 1: +5V -> /SDA
- U41 pad 10: /BUCK_5/Vin+ -> /BUCK_9/Vin+
- U41 pad 3: unconnected-(U25-Pad3) -> unconnected-(U41-Pad3)
- U41 pad 8: Net-(TP42-Pad1) -> Net-(TP70-Pad1)
- U41 pad 9: /BUCK_5/Vin- -> /BUCK_9/Vin-
- U42 pad A1: /BUCK_5/BUCK_VIN -> /BUCK_9/BUCK_VIN
- U42 pad A10: /BUCK_5/RUN -> /BUCK_9/RUN
- U42 pad A11: Net-(TP45-Pad1) -> Net-(TP73-Pad1)
- U42 pad A12: unconnected-(U26-PadA12) -> unconnected-(U42-PadA12)
- U42 pad A2: /BUCK_5/BUCK_VIN -> /BUCK_9/BUCK_VIN
- U42 pad A3: /BUCK_5/BUCK_VIN -> /BUCK_9/BUCK_VIN
- U42 pad A4: /BUCK_5/BUCK_VIN -> /BUCK_9/BUCK_VIN
- U42 pad A5: /BUCK_5/BUCK_VIN -> /BUCK_9/BUCK_VIN
- U42 pad A6: /BUCK_5/BUCK_VIN -> /BUCK_9/BUCK_VIN
- U42 pad A7: Net-(TP41-Pad1) -> Net-(TP69-Pad1)
- U42 pad A8: /NEG_5 -> /NEG_9
- U42 pad A9: /BUCK_5/TRACK/SS -> /BUCK_9/TRACK/SS
- U42 pad B1: /BUCK_5/BUCK_VIN -> /BUCK_9/BUCK_VIN
- U42 pad B11: unconnected-(U26-PadB11) -> unconnected-(U42-PadB11)
- U42 pad B12: Net-(TP44-Pad1) -> Net-(TP72-Pad1)
- U42 pad B2: /BUCK_5/BUCK_VIN -> /BUCK_9/BUCK_VIN
- U42 pad B3: /BUCK_5/BUCK_VIN -> /BUCK_9/BUCK_VIN
- U42 pad B4: /BUCK_5/BUCK_VIN -> /BUCK_9/BUCK_VIN
- U42 pad B5: /BUCK_5/BUCK_VIN -> /BUCK_9/BUCK_VIN
- U42 pad B6: /BUCK_5/BUCK_VIN -> /BUCK_9/BUCK_VIN
- U42 pad B7: /NEG_5 -> /NEG_9
- U42 pad B9: /NEG_5 -> /NEG_9
- U42 pad C1: /BUCK_5/BUCK_VIN -> /BUCK_9/BUCK_VIN
- U42 pad C10: unconnected-(U26-PadC10) -> unconnected-(U42-PadC10)
- U42 pad C11: unconnected-(U26-PadC11) -> unconnected-(U42-PadC11)
- U42 pad C12: unconnected-(U26-PadC12) -> unconnected-(U42-PadC12)
- U42 pad C2: /BUCK_5/BUCK_VIN -> /BUCK_9/BUCK_VIN
- U42 pad C3: /BUCK_5/BUCK_VIN -> /BUCK_9/BUCK_VIN
- U42 pad C4: /BUCK_5/BUCK_VIN -> /BUCK_9/BUCK_VIN
- U42 pad C5: /BUCK_5/BUCK_VIN -> /BUCK_9/BUCK_VIN
- U42 pad C6: /BUCK_5/BUCK_VIN -> /BUCK_9/BUCK_VIN
- U42 pad C7: /NEG_5 -> /NEG_9
- U42 pad C9: /NEG_5 -> /NEG_9
- U42 pad D1: /NEG_5 -> /NEG_9
- U42 pad D10: unconnected-(U26-PadD10) -> unconnected-(U42-PadD10)
- U42 pad D11: unconnected-(U26-PadD11) -> unconnected-(U42-PadD11)
- U42 pad D12: unconnected-(U26-PadD12) -> unconnected-(U42-PadD12)
- U42 pad D2: /NEG_5 -> /NEG_9
- U42 pad D3: /NEG_5 -> /NEG_9
- U42 pad D4: /NEG_5 -> /NEG_9
- U42 pad D5: /NEG_5 -> /NEG_9
- U42 pad D6: /NEG_5 -> /NEG_9
- U42 pad D8: /NEG_5 -> /NEG_9
- U42 pad D9: unconnected-(U26-PadD9) -> unconnected-(U42-PadD9)
- U42 pad E1: /NEG_5 -> /NEG_9
- U42 pad E12: unconnected-(U26-PadE12) -> unconnected-(U42-PadE12)
- U42 pad E2: /NEG_5 -> /NEG_9
- U42 pad E3: /NEG_5 -> /NEG_9
- U42 pad E4: /NEG_5 -> /NEG_9
- U42 pad E5: /NEG_5 -> /NEG_9
- U42 pad E6: /NEG_5 -> /NEG_9
- U42 pad E7: /NEG_5 -> /NEG_9
- U42 pad E9: /NEG_5 -> /NEG_9
- U42 pad F1: /NEG_5 -> /NEG_9
- U42 pad F11: Net-(TP43-Pad1) -> Net-(TP71-Pad1)
- U42 pad F12: /BUCK_5/Vfb -> /BUCK_9/Vfb
- U42 pad F2: /NEG_5 -> /NEG_9
- U42 pad F3: /NEG_5 -> /NEG_9
- U42 pad F4: /NEG_5 -> /NEG_9
- U42 pad F5: /NEG_5 -> /NEG_9
- U42 pad F6: /NEG_5 -> /NEG_9
- U42 pad F7: /NEG_5 -> /NEG_9
- U42 pad F8: /NEG_5 -> /NEG_9
- U42 pad F9: /NEG_5 -> /NEG_9
- U42 pad G1: /NEG_5 -> /NEG_9
- U42 pad G11: /NEG_5 -> /NEG_9
- U42 pad G12: Net-(TP43-Pad1) -> Net-(TP71-Pad1)
- U42 pad G2: /NEG_5 -> /NEG_9
- U42 pad G3: /NEG_5 -> /NEG_9
- U42 pad G4: /NEG_5 -> /NEG_9
- U42 pad G5: /NEG_5 -> /NEG_9
- U42 pad G6: /NEG_5 -> /NEG_9
- U42 pad G7: /NEG_5 -> /NEG_9
- U42 pad G8: /NEG_5 -> /NEG_9
- U42 pad G9: /NEG_5 -> /NEG_9
- U42 pad H1: /NEG_5 -> /NEG_9
- U42 pad H11: /NEG_5 -> /NEG_9
- U42 pad H12: /NEG_5 -> /NEG_9
- U42 pad H2: /NEG_5 -> /NEG_9
- U42 pad H3: /NEG_5 -> /NEG_9
- U42 pad H4: /NEG_5 -> /NEG_9
- U42 pad H5: /NEG_5 -> /NEG_9
- U42 pad H6: /NEG_5 -> /NEG_9
- U42 pad H7: /NEG_5 -> /NEG_9
- U42 pad H8: /NEG_5 -> /NEG_9
- U42 pad H9: /NEG_5 -> /NEG_9
- U42 pad J1: /NEG_6 -> /POS_9
- U42 pad J10: /NEG_6 -> /POS_9
- U42 pad J12: /NEG_6 -> /POS_9
- U42 pad J2: /NEG_6 -> /POS_9
- U42 pad J3: /NEG_6 -> /POS_9
- U42 pad J4: /NEG_6 -> /POS_9
- U42 pad J5: /NEG_6 -> /POS_9
- U42 pad J6: /NEG_6 -> /POS_9
- U42 pad J7: /NEG_6 -> /POS_9
- U42 pad J8: /NEG_6 -> /POS_9
- U42 pad J9: /NEG_6 -> /POS_9
- U42 pad K1: /NEG_6 -> /POS_9
- U42 pad K10: /NEG_6 -> /POS_9
- U42 pad K11: /NEG_6 -> /POS_9
- U42 pad K12: Net-(JP6-Pad1) -> Net-(JP10-Pad1)
- U42 pad K2: /NEG_6 -> /POS_9
- U42 pad K3: /NEG_6 -> /POS_9
- U42 pad K4: /NEG_6 -> /POS_9
- U42 pad K5: /NEG_6 -> /POS_9
- U42 pad K6: /NEG_6 -> /POS_9
- U42 pad K7: /NEG_6 -> /POS_9
- U42 pad K8: /NEG_6 -> /POS_9
- U42 pad K9: /NEG_6 -> /POS_9
- U42 pad L1: /NEG_6 -> /POS_9
- U42 pad L10: /NEG_6 -> /POS_9
- U42 pad L11: /NEG_6 -> /POS_9
- U42 pad L12: Net-(JP6-Pad2) -> Net-(JP10-Pad2)
- U42 pad L2: /NEG_6 -> /POS_9
- U42 pad L3: /NEG_6 -> /POS_9
- U42 pad L4: /NEG_6 -> /POS_9
- U42 pad L5: /NEG_6 -> /POS_9
- U42 pad L6: /NEG_6 -> /POS_9
- U42 pad L7: /NEG_6 -> /POS_9
- U42 pad L8: /NEG_6 -> /POS_9
- U42 pad L9: /NEG_6 -> /POS_9
- U42 pad M1: /NEG_6 -> /POS_9
- U42 pad M10: /NEG_6 -> /POS_9
- U42 pad M11: /NEG_6 -> /POS_9
- U42 pad M12: /NEG_5 -> /NEG_9
- U42 pad M2: /NEG_6 -> /POS_9
- U42 pad M3: /NEG_6 -> /POS_9
- U42 pad M4: /NEG_6 -> /POS_9
- U42 pad M5: /NEG_6 -> /POS_9
- U42 pad M6: /NEG_6 -> /POS_9
- U42 pad M7: /NEG_6 -> /POS_9
- U42 pad M8: /NEG_6 -> /POS_9
- U42 pad M9: /NEG_6 -> /POS_9
- U43 pad 1: /CS5 -> /CS9
- U43 pad 5: /BUCK_5/P0A -> /BUCK_9/P0A
- U43 pad 6: /NEG_5 -> /NEG_9
- U43 pad 7: unconnected-(U27-Pad7) -> unconnected-(U43-Pad7)
Routing:
- net /SCL: track 889.4 -> 485.9 mm
- net /SDA: track 830.6 -> 522.6 mm, vias 10 -> 7
- net /NEG_5: track 154.2 -> 35.5 mm, vias 20 -> 4
- net Net-(TP42-Pad1): track 139.2 -> 28.3 mm, vias 1 -> 0
- net Net-(JP6-Pad2): track 90.2 -> 18.0 mm, vias 10 -> 2
- net Net-(TP43-Pad1): track 71.9 -> 14.4 mm, vias 10 -> 2
- net Net-(JP6-Pad1): track 60.6 -> 12.1 mm, vias 10 -> 2
- net /BUCK_5/Vin-: track 52.2 -> 10.4 mm
- net /BUCK_5/+IN: track 46.1 -> 9.23 mm
- net /NEG_7: track 0.00 -> 36.2 mm, vias 0 -> 4
- net /NEG_9: track 0.00 -> 35.7 mm, vias 0 -> 4
- net /BUCK_5/BUCK_VIN: track 42.0 -> 8.40 mm
- net Net-(TP63-Pad1): track 0.00 -> 31.6 mm
- net Net-(TP56-Pad1): track 0.00 -> 30.7 mm
- net /BUCK_5/Vin+: track 38.1 -> 7.62 mm
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- added copper zone on F.Cu, net /BUCK_6/BUCK_VIN
- added copper zone on F.Cu, net /BUCK_7/BUCK_VIN
- added copper zone on F.Cu, net /BUCK_8/BUCK_VIN
- added copper zone on F.Cu, net /BUCK_9/BUCK_VIN
- added copper zone on F.Cu, net /NEG_6
- added copper zone on F.Cu, net /NEG_7
- added copper zone on F.Cu, net /NEG_8
- added copper zone on F.Cu, net /NEG_9
- added copper zone on F.Cu, net /PV_POS_6
- added copper zone on F.Cu, net /PV_POS_7
- added copper zone on F.Cu, net /PV_POS_8
- added copper zone on F.Cu, net /PV_POS_9
Other:
- board text added: "INA226 decoupling cap moet ff bij allen GOED gedaan worden"
- board text removed: "misschien een fout: wrm willen de LTM4611's aan de rechterkant allemaal NEG_5?"

Commit message: Change routing of bypass caps, routed 3.3v to micro.
Parts:
- moved J11 209.6 mm to (150.2, 28.5), turned to 180 degrees
- moved U2 190.1 mm to (137.6, 50.9), turned to 0 degrees
- moved R2 147.5 mm to (154.3, 58.6), turned to 180 degrees
- moved D1 141.7 mm to (140.3, 68.1), turned to 0 degrees
- moved TP3 131.1 mm to (150.3, 61.5), turned to 180 degrees
- moved R1 123.3 mm to (136.6, 66.6)
- moved C9 120.2 mm to (143.4, 59.5), turned to 0 degrees
- moved TP2 120.2 mm to (139.7, 61.6), turned to 180 degrees
- moved C10 117.4 mm to (149.0, 67.9), turned to 0 degrees
- moved U1 94.8 mm to (144.9, 64.7), turned to -90 degrees
- moved J12 79.2 mm to (160.1, 66.7), turned to 0 degrees
- moved D2 73.8 mm to (143.5, 94.7)
- moved R4 73.8 mm to (143.5, 91.7)
- moved C156 68.6 mm to (231.5, 92.0), turned to 90 degrees
- moved C141 68.5 mm to (231.2, 128.5), turned to 90 degrees
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Routing:
- net /SDA: track 522.6 -> 11.8 mm, vias 7 -> 0
- net /SCL: track 485.9 -> 6.81 mm
- net +3.3V: track 2.53 -> 76.1 mm, vias 0 -> 3
- net GND: track 190.8 -> 122.8 mm, vias 33 -> 68
- net Net-(TP63-Pad1): track 31.6 -> 22.0 mm
- net /NRST: track 0.00 -> 9.45 mm
- net Net-(TP56-Pad1): track 30.7 -> 21.8 mm
- net Net-(R2-Pad1): track 0.00 -> 7.95 mm
- net Net-(TP42-Pad1): track 28.3 -> 20.8 mm
- net Net-(TP70-Pad1): track 28.8 -> 21.8 mm
- net Net-(TP14-Pad1): track 29.2 -> 22.4 mm, vias 1 -> 0
- net Net-(TP7-Pad1): track 28.7 -> 22.5 mm, vias 1 -> 0
- net Net-(TP21-Pad1): track 27.4 -> 21.7 mm, vias 1 -> 0
- net /SWDIO: track 19.4 -> 14.1 mm
- net Net-(TP49-Pad1): track 26.6 -> 21.8 mm
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Other:
- board text added: "To do: - 3V3 regulator met componenten plaatsen - 5V converter plaatsen - mounting hole in het midden - SDA, SCL - SCK, SDIO - SC met pull-up"
- board text removed: "INA226 decoupling cap moet ff bij allen GOED gedaan worden"
