File: KiCAD/Quest_39/BUCK_0.kicad_sch (KiCad schematic)
At the start: 34 parts, among them U4 AD626ANZ, U5 INA226, U6 LTM4611EV-PBF, U7 MCP4151-502E/SN

Commit message: Added all the SolidWorks files, edited README
Other:
- title: BUCK_0 -> (none)
Changed lines of the file:
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@@
   (paper "A3")
   (title_block
-    (title "BUCK_0")
-    (date "2022-12-05")
-    (rev "0.1")
+    (date "2023-01-31")
+    (rev "1.0")
   )
   (junction (at 25.4 80.01) (diameter 0) (color 0 0 0 0)
